File: mcu.kicad_sch (KiCad schematic)
At the start: 45 parts, among them U9 NUCLEOH723ZG

Commit message: Simplifying the design
Parts:
- added Q1, Q2, Q3, Q4, Q5: IRL6283M, Package_DirectFET:DirectFET_MD, symbol Transistor_FET:IRL6283M
- added R162, R163, R164, R165, R172, R173, R174, R175, R176, R177, R178, R179, R74: 10kR, Resistor_SMD:R_0402_1005Metric_Pad0.72x0.64mm_HandSolder, symbol Device:R
- added R166, R167, R168, R169, R170, R171, R182, R73, R75, R77, R78, R79, R80, R81, R82: 33R, Resistor_SMD:R_0402_1005Metric_Pad0.72x0.64mm_HandSolder, symbol Device:R
- added R183, R184, R185, R186, R187: 470R, symbol Device:R
- added R188, R193, R194, R195, R196: 10k, symbol Device:R
- R123: value 33R -> 10kR
Connections:
- net +3V3: now also R123.1, R162.1, R163.2, R164.2, R165.2, R172.2, R173.1, R174.1, R175.2, R176.2, R177.2, R178.2, R179.2, R74.2
- net GND: now also U9.CN10_17 (GND_CN10), U9.CN10_22 (GND_CN10), U9.CN10_27 (GND_CN10), U9.CN10_3 (AGND_CN10), U9.CN10_5 (GND_CN10), U9.CN7_8 (GND_CN7), R188.2, R193.2, R194.2, R195.2, R196.2
- net at U9.CN7_17 (D24/SPI_B_NSS): now also R182.1
- net GPIO_PD15: now reaches U9.CN7_18 (D9/TIMER_B_PWM2)
- net GPIO_PD15: now also R173.2
- net at U9.CN9_10 (D55/USART_B_CTS): now also R169.2
- net CH2_ATTEN_MCU: now reaches U9.CN9_13 (D72/COMP1_INP)
- net CH2_ATTEN_MCU: now also R186.2
- net at U9.CN9_16 (D57/SAI_A_FS): now also R75.2
- net at U9.CN9_18 (D58/SAI_A_SCK): now also R77.2
- net at U9.CN9_2 (D51/USART_B_SCLK): now also R170.2
- net at U9.CN9_20 (D59/SAI_A_SD): now also R78.2
- net AD_DC_MCU: now reaches U9.CN9_26 (D62/SAI_B_MCLK)
- net AD_DC_MCU: now also R187.2
- net TRIGG_2_MCU: now reaches U9.CN9_29 (D65/IO)
- net TRIGG_2_MCU: now also R184.2
- net TRIGG_1_MCU: now reaches U9.CN9_30 (D64/IO)
- net TRIGG_1_MCU: now also R183.2
- net at U9.CN9_4 (D52/USART_B_RX): now also R171.2
- net at U9.CN9_6 (D53/USART_B_TX): now also R167.2
- net at U9.CN9_8 (D54/USART_B_RTS): now also R168.2
- net at U9.CN10_28 (D38/TIMER_A_BKIN2): no longer R123.2
- net at U9.CN8_12 (D48/SDMMC_CMD): now also R166.2, R174.2
- net at U9.CN10_10 (D3/TIMER_A_PWM3): now also R81.2
- net at U9.CN10_33 (D34/TIMER_B_ETR): now also R73.1, R74.1
- net at U9.CN10_4 (D6/TIMER_A_PWM1): now also R79.2
- net at U9.CN10_6 (D5/TIMER_A_PWM2): now also R80.2
- net at U9.CN10_8 (D4/IO): now also R172.1, R82.1
- net GPIO_10 renamed GPIO_PE7
- net GPIO_11 renamed GPIO_PE8
- net GPIO_20 renamed GPIO_4
- net GPIO_4: no longer R157.2
- net GPIO_21 renamed GPIO_3
- net GPIO_3: no longer R158.2
- net GPIO_22 renamed GPIO_2
- net GPIO_23 renamed GPIO_1
- net GPIO_6 renamed GPIO_PE15
- net GPIO_7 renamed GPIO_PE11
- net GPIO_PE11: now also R80.1; no longer R123.1
- net GPIO_8 renamed GPIO_PE12
- net GPIO_9 renamed GPIO_PE10
- net QSPI_CLK/GPIO_1 renamed QSPI_CLK
- net QSPI_CS/GPIO_0 renamed QSPI_CS
- net QSPI_IO0/GPIO_2 renamed QSPI_IO0/GPIO_PD11
- net QSPI_IO1/GPIO_3 renamed QSPI_IO1/GPIO_PD12
- net QSPI_IO2/GPIO_4 renamed QSPI_IO2/GPIO_PE2
- net QSPI_IO3/GPIO_5 renamed QSPI_IO3/GPIO_PD13
- new net: Q2.3 (S), R193.1
- new net: Q2.2 (G), R184.1
- new net: Q3.2 (G), R185.1
- new net: Q3.3 (S), R194.1
- new net: Q1.3 (S), R188.1
- new net: Q5.3 (S), R195.1
- new net: Q1.2 (G), R183.1
- new net: Q4.3 (S), R196.1
- new net: Q5.2 (G), R187.1
- new net: Q4.2 (G), R186.1
- new net AD_DC: Q5.1 (D)
- new net CH1_ATTEN: Q3.1 (D)
- new net CH1_ATTEN_MCU: R185.2
- new net CH2_ATTEN: Q4.1 (D)
- new net DAC1: R182.2
- new net GPIO_0: R82.2
- new net GPIO_PD0: R158.2
- new net GPIO_PD1: R157.2
- new net GPIO_PD2: R166.1
- new net GPIO_PD3: R169.1, R177.1
- new net GPIO_PD4: R168.1, R176.1
- new net GPIO_PD5: R167.1, R175.1
- new net GPIO_PD6: R171.1, R179.1
- new net GPIO_PD7: R170.1, R178.1
- new net GPIO_PE0: R73.2
- new net GPIO_PE13: R123.2, R81.1
- new net GPIO_PE4: R165.1, R75.1
- new net GPIO_PE5: R163.1, R77.1
- new net GPIO_PE6: R164.1, R78.1
- new net GPIO_PE9: R162.2, R79.1
- new net TRIGG_1: Q1.1 (D)
- new net TRIGG_2: Q2.1 (D)
Other:
- moved on the sheet: R120, R121, R122, R124, R125, R126, R127, R128, R129, R130, R131, R132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
