File: analog_inputs_sch.kicad_sch (KiCad schematic)
At the start: 135 parts, among them J1 Conn_Coaxial, J2 Conn_Coaxial, J7 Conn_Coaxial, K1 G2RL-1, K10 G2RL-2, K2 G2RL-1, K8 G2RL-2, K9 G2RL-2, U1 OPA656U, U11 AD8045ACPZ-R2, U12 OPA2277, U13 OPA2277, U14 AD8045ACPZ-R2, U2 LTC6754xSC6, U8 OPA656U

Commit message: Almost finishing schematic
Parts:
- removed C5, C9: C 2.0 - 6.0 pF, symbol Device:C_Variable
- removed C59: DNP, symbol Device:C
- removed C7: C 360 pF, symbol Device:C
- removed K1, K2: G2RL-1, Relay_THT:Relay_SPDT_Omron_G2RL-1, symbol Relay:G2RL-1
- removed K10, K8, K9: G2RL-2, Relay_THT:Relay_DPDT_Omron_G2RL-2, symbol Relay:G2RL-2
- removed U2: LTC6754xSC6, Package_TO_SOT_SMD:SOT-363_SC-70-6, symbol Comparator:LTC6754xSC6
- added C11, C84: 12pF, symbol Device:C
- added C12, C13: C, symbol Device:C
- added C130, C132, C73, C76, C80, C81, C86, C89, C92, C95: 1uF, symbol Device:C
- added C131, C14, C72, C75, C79, C85, C90, C91, C96: 100nF, symbol Device:C
- added C133, C134, C74, C77, C82, C83, C87, C88, C93, C94: 10uF, symbol Device:C
- added C135: 22nF, symbol Device:C
- added C136, C137, C138, C139, C5: DNP, symbol Device:C
- added C59: C 2.0 - 6.0 pF, symbol Device:C_Variable
- added C7: C 2.0 - 10.0 pF, symbol Device:C_Variable
- added C9: C 390 pF, symbol Device:C
- added D1, D2: BAV199DW, Package_TO_SOT_SMD:SOT-363_SC-70-6, symbol Diode:BAV199DW
- added K3, K4, K6, K7, K8: TQ2-L2-5V, RELAY_TQ2_2C_PAN, symbol 2025-10-25_18-45-48:TQ2-L2-5V
- added L19, L21, L23, L24, L27, L30, L31, L34, L55, L57: LCBB-601, symbol Device:L
- added L20, L22, L25, L26, L28, L29, L32, L33, L56, L58: 0.68uH, 0.8Ohm, symbol Device:L
- added R17, R199, R32, R36, R4, R43, R5, R7: 25R, Resistor_SMD:R_1206_3216Metric, symbol Device:R
- added R18, R198: 33 R, Resistor_SMD:R_1206_3216Metric, symbol Device:R
- added R19, R35: R, Resistor_SMD:R_1206_3216Metric, symbol Device:R
- added R200, R44: 49.9 R, Resistor_SMD:R_1206_3216Metric, symbol Device:R
- added R21, R22, R24, R25, R26, R27, R6, R69: 499R, Resistor_SMD:R_1206_3216Metric, symbol Device:R
- added R28, R29, R30, R31: 100 R, Resistor_SMD:R_1206_3216Metric, symbol Device:R
- added R70, R71: DNP, Resistor_SMD:R_1206_3216Metric, symbol Device:R
- added TP19, TP20, TP21, TP22, TP23, TP24, TP25, TP26: TestPoint, Connector_PinHeader_2.54mm:PinHeader_1x01_P2.54mm_Vertical, symbol Connector:TestPoint
- added U17: AD8611ARZ, R_8_ADI, symbol 2025-10-25_17-44-45:AD8611ARZ
- added U3, U5: AD8337BCPZ-REEL-ND, footprints:CP_8_2_ADI, symbol 2025-07-13_23-24-37:AD8337BCPZ-REEL-ND
- added U4, U6: AD8138ARZ, R_8_ADI, symbol 2025-10-25_19-35-02:AD8138ARZ
- C127: value 1uF -> 100nF
- C8: value C 390 pF -> C 360 pF
- R12: value R 47k -> 33R
- R13: value 33R -> R 9.53 kΩ
- R16: value 33 R -> 33R
- R20, R34: value DNP -> 10k
- R23, R33: value R -> 10k
- R9: value R 22.2k -> R 9.53 kΩ
Connections:
- net +3V3 is gone; now on net GND: C127.2
- net +5V: now also D1.2 (K2), D2.2 (K2), K4.1, K4.10, K8.1, L28.1, L29.1, L56.1
- net -5V: now also D1.1 (A1), D2.1 (A1), L32.1, L33.1, L58.1
- net AN_TRIGGER_CH1: now also K4.2, R17.1
- net AN_TRIGGER_CH2: now also K4.4, R7.1
- net AN_TRIGGER_N: now also R34.1, TP17.1, U17.8 (OUT*); no longer R20.1, TP18.1
- net AN_TRIGGER_P: now also R20.1, TP18.1, U17.7 (OUT); no longer R34.1, TP17.1
- net GND: now also C8.2, R13.2, C12.2, C13.2, C130.1, C131.2, C132.1, C133.1, C134.1, C14.2, C59.2, C72.2, C73.1, C74.1, C75.2, C76.1, C77.1, C79.2, C80.1, C81.1, C82.1, C83.1, C85.2, C86.1, C87.1, C88.1, C89.1, C90.2, C91.2, C92.1, C93.1, C94.1, C95.1, C96.2, R18.2, R19.2, R198.2, R200.2, R29.2, R31.2, R35.2, R44.2, U17.5 (LATCH), U17.6 (GND), U3.HTAB (EPAD), U5.HTAB (EPAD); no longer C127.1, R12.2
- net TRIGG_1: now also K4.5
- net TRIGG_2: now also K4.6
- net at R23.1, R34.2: now also U17.3 (-IN)
- net at R3.2: now also C8.1, R13.1, C5.2, C7.2, K3.9; no longer R12.1
- net at TP2.1: now also C1.1, R2.2, K7.8; no longer R2.1
- net at J2.1 (In): now also R12.1; no longer R13.1
- net at R16.1: now also K3.8; no longer TP8.1
- net at C10.1, R16.2: now also TP8.1, K7.3
- net at C4.1, R10.1: now also K6.4
- net at C3.1, C4.2, C57.1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: now also K6.7
- net at R20.2, R33.1: now also U17.2 (+IN)
- net at R33.2, TP15.1: now also C135.2, K8.4
- net at R14.1: now also C9.1, K3.4; no longer C8.1
- net at C58.1, R14.2, R15.1: now also C59.1, C9.2, K3.7; no longer C8.2
- net at C10.2, TP9.1, U8.3 (POS): now also D2.6 (K3A4), K7.4
- net at C2.1, C56.2, C6.2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: now also K6.9
- net at TP7.1: now also R12.2, K3.3; no longer R13.2
- net at C1.2, TP3.1, U1.3 (POS): now also D1.6 (K3A4), K7.7
- net at C56.1, C6.1, R8.1: now also K6.2
- net at R1.2, TP1.1: now also K6.3
- net at R3.1: now also C5.1, C7.1, K3.2
- net CH1_VGA: no longer names the net of R46.2, R59.2, TP6.1, U14.7 (OUTPUT)
- net CH1_VGA: now also R200.1, U5.3 (INPP)
- net CH2_VGA: no longer names the net of R63.2, R64.2, TP14.1, U11.7 (OUTPUT)
- net CH2_VGA: now also R44.1, U3.3 (INPP)
- net TRIGGER_LEVEL renamed EXT_TRIGGER_LEVEL
- net EXT_TRIGGER_LEVEL: now also K4.7
- new net: R17.2, R198.1, R6.2, TP22.1, U5.1 (VOUT)
- new net: R28.1, R29.1, U5.2 (VCOM), U5.4 (INPN)
- new net: R28.2, U5.5 (PRAO)
- new net: C91.1, C92.2, C93.2, L31.2, U5.6 (VNEG)
- new net: R43.1, TP19.1, U5.7 (GAIN)
- new net: C85.1, C86.2, C87.2, L27.2, U5.8 (VPOS)
- new net: C137.1, R24.2, R6.1, U6.8 (+IN)
- new net: C137.2, R24.1, R5.2, TP25.1, U6.4 (+OUT)
- new net: L24.1, L26.2
- new net: C79.1, C81.2, C83.2, L24.2, U4.6 (V-)
- new net: C75.1, C76.2, C77.2, L21.2, U6.6 (V-)
- new net: R18.1, R21.2, R7.2, TP21.1, U3.1 (VOUT)
- new net: L29.2, L30.1
- new net: C94.2, C95.2, C96.1, L34.2, U3.6 (VNEG)
- new net: C138.1, R22.1, R27.2, U4.1 (-IN)
- new net: C14.1, C80.2, C82.2, L23.2, U4.3 (V+)
- new net: C139.2, R26.1, R32.2, TP23.1, U4.4 (+OUT)
- new net: C138.2, R27.1, R36.2, TP24.1, U4.5 (-OUT)
- new net: C139.1, R21.1, R26.2, U4.8 (+IN)
- new net: C72.1, C73.2, C74.2, L19.2, U6.3 (V+)
- new net: C136.1, R25.2, R69.1, U6.1 (-IN)
- new net: R35.1, R69.2
- new net: L21.1, L22.2
- new net: L55.1, L56.2
- new net: K4.3, K4.9
- new net: C135.1, K4.8, K8.3
- new net: K6.8, R2.1
- new net: C127.1, C130.2, C134.2, L55.2, U17.1 (V+)
- new net: C88.2, C89.2, C90.1, L30.2, U3.8 (VPOS)
- new net: C131.1, C132.2, C133.2, L57.2, U17.4 (V-)
- new net: C136.2, R25.1, R4.2, TP26.1, U6.5 (-OUT)
- new net: L33.2, L34.1
- new net: R30.1, R31.1, U3.2 (VCOM), U3.4 (INPN)
- new net: L27.1, L28.2
- new net: L31.1, L32.2
- new net: L19.1, L20.2
- new net: R30.2, U3.5 (PRAO)
- new net: L57.1, L58.2
- new net: L23.1, L25.2
- new net: R19.1, R22.2
- new net: R199.1, TP20.1, U3.7 (GAIN)
- new net +1V5: C12.1, C13.1, U4.2 (VOCM), U6.2 (VOCM)
- new net +5V_EXT: K3.1, K3.10, K6.1, K6.10, K7.1, K7.10
- new net +6V5: L20.1, L25.1
- new net -3V5: L22.1, L26.1
- new net AC_DC_CH1: K7.6
- new net AC_DC_CH2: K7.5
- new net CH1_ATTEN_A: K6.5
- new net CH1_ATTEN_B: K6.6
- new net CH1_CH+: C11.1, R5.1, R71.1
- new net CH1_CH-: C11.2, R4.1, R71.2
- new net CH1_GAIN_DAC: R43.2
- new net CH2_ATTEN_A: K3.5
- new net CH2_ATTEN_B: K3.6
- new net CH2_CH+: C84.1, R32.1, R70.1
- new net CH2_CH-: C84.2, R36.1, R70.2
- new net CH2_GAIN_DAC: R199.2
- new net TRIGGER_AC_DC: K8.5
- no-connect marks 6 -> 14
Other:
- note added: "~ 1 : 100"
- note removed: "sbaa343a"
- note removed: "~ 1 : 44"
- moved on the sheet: C1, C100, C101, C102, C103, C104, C105, C106, C107, C108, C109, C110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

Commit message: Save work before deleting amps from DAC to offset
Parts:
- removed C100, C109, C112, C97: 100nF, symbol Device:C
- removed C101, C110, C113, C98: 1uF, symbol Device:C
- removed C102, C111, C114, C99: 10uF, symbol Device:C
- removed L35, L37, L43, L45: LCBB-601, symbol Device:L
- removed L36, L38, L44, L46: 0.68uH, 0.8Ohm, symbol Device:L
- removed R46, R54, R60, R63: 10k, Resistor_SMD:R_1206_3216Metric, symbol Device:R
- removed R59, R64: 0R, Resistor_SMD:R_1206_3216Metric, symbol Device:R
- removed TP14, TP6: TestPoint, Connector_PinHeader_2.54mm:PinHeader_1x01_P2.54mm_Vertical, symbol Connector:TestPoint
- removed U11, U14: AD8045ACPZ-R2, footprints:CP_8_2_ADI, symbol 2025-07-01_23-44-10:AD8045ACPZ-R2
- R45: value 10k -> 33R
Connections:
- net +5V: no longer K4.1, K4.10, K8.1
- net +5V_EXT: now also K4.1, K4.10, K8.1
- net GND: no longer R38.1, R45.1
- net at R45.2: now also R37.1, U1.6 (OUTPUT)
- net at R37.2, TP4.1: now also R200.1, U5.3 (INPP); no longer R38.2, R39.1
- net at R41.1, U8.6 (OUTPUT): now also R38.1; no longer U8.2 (NEG)
- net at R41.2, TP13.1: now also R44.1, U3.3 (INPP); no longer R53.1
- net DAC1 renamed TRIGGER_THRESHOLD
- new net: R38.2, R53.1, U8.2 (NEG)
- new net: R39.1, R45.1, U1.2 (NEG)
- no-connect marks 14 -> 10
Other:
- moved on the sheet: C103, C104, C105, C106, C107, C108, C115, C116, C117, C118, C119, C120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
