File: DigitalOsciloscope.kicad_pcb (KiCad board)
At the start: 2 copper layers, 10 parts, among them U11 SN75160BDW, U12 SN75160BDW, U13 SN75160BDW, U14 SN75160BDW, U16 DAC80504, U17 CYPD3177-24LQ, U2 LTC6754xSC6, U4 LMH6551MA, U6 LTC2299xUP, U7 LMH6551MA

Commit message: PCB edge, initial work on assigning footprints
Parts:
- added D10: 1N5822, Diode_THT:D_DO-201AD_P15.24mm_Horizontal, F.Cu at (173.2, -85.9)
- added D2: 1N5822, Diode_THT:D_DO-201AD_P15.24mm_Horizontal, F.Cu at (173.2, -119.6)
- added D6: 1N5822, Diode_THT:D_DO-201AD_P15.24mm_Horizontal, F.Cu at (173.2, -112.9)
- added D7: 1N5822, Diode_THT:D_DO-201AD_P15.24mm_Horizontal, F.Cu at (173.2, -106.1)
- added D8: 1N5400, Diode_THT:D_DO-201AD_P15.24mm_Horizontal, F.Cu at (173.2, -99.4)
- added D9: 1N5400, Diode_THT:D_DO-201AD_P15.24mm_Horizontal, F.Cu at (173.2, -92.6)
- added J1: Conn_Coaxial, Connector_Coaxial:BNC_TEConnectivity_1478035_Horizontal, F.Cu at (38.5, 44.5)
- added J2: Conn_Coaxial, Connector_Coaxial:BNC_TEConnectivity_1478035_Horizontal, F.Cu at (38.5, 72.5)
- added J7: Conn_Coaxial, Connector_Coaxial:BNC_TEConnectivity_1478035_Horizontal, F.Cu at (38.5, 100.5)
- added K10: G2RL-2, Relay_THT:Relay_DPDT_Omron_G2RL-2, F.Cu at (202.6, -76.1)
- added K8: G2RL-2, Relay_THT:Relay_DPDT_Omron_G2RL-2, F.Cu at (263.8, -75.0)
- added K9: G2RL-2, Relay_THT:Relay_DPDT_Omron_G2RL-2, F.Cu at (264.5, -39.0)
- added Q1: 2N7002, Package_TO_SOT_SMD:SOT-23, F.Cu at (211.0, -120.6)
- added Q2: DMP3099L, Package_TO_SOT_SMD:SOT-23, F.Cu at (211.0, -116.0)
- added Q3: DMP3099L, Package_TO_SOT_SMD:SOT-23, F.Cu at (211.0, -111.3)
- added U1: OPA656U, OPA656U:SOIC127P599X175-8N, F.Cu at (59.5, 44.6)
- added U19: LM2596S-ADJ, Package_TO_SOT_SMD:TO-263-5_TabPin3, F.Cu at (201.5, -116.8)
- added U20: INA180A3, Package_TO_SOT_SMD:SOT-23-5, F.Cu at (193.4, -83.5)
- added U21: LM2596S-5, Package_TO_SOT_SMD:TO-263-5_TabPin3, F.Cu at (201.5, -104.5)
- added U22: LM2596S-5, Package_TO_SOT_SMD:TO-263-5_TabPin3, F.Cu at (201.5, -92.1)
- added U23: AP1117-ADJ, Package_TO_SOT_SMD:SOT-223-3_TabPin2, F.Cu at (220.3, -118.8)
- added U24: AP1117-ADJ, Package_TO_SOT_SMD:SOT-223-3_TabPin2, F.Cu at (220.3, -110.5)
- added U25: AP1117-ADJ, Package_TO_SOT_SMD:SOT-223-3_TabPin2, F.Cu at (220.3, -102.2)
- added U26: AP1117-ADJ, Package_TO_SOT_SMD:SOT-223-3_TabPin2, F.Cu at (220.3, -93.8)
- added U27: AP1117-ADJ, Package_TO_SOT_SMD:SOT-223-3_TabPin2, F.Cu at (220.3, -85.5)
- added U8: OPA656U, OPA656U:SOIC127P599X175-8N, F.Cu at (60.0, 74.1)
- moved U11 154.4 mm to (46.3, -91.3)
- moved U12 154.4 mm to (59.2, -91.3)
- moved U13 154.4 mm to (72.2, -91.3)
- moved U14 154.4 mm to (85.1, -91.3)
- moved U16 154.4 mm to (74.6, -79.5)
- moved U17 154.4 mm to (108.7, -78.5)
- moved U2 154.4 mm to (74.1, -72.8)
- moved U4 154.4 mm to (44.1, -78.8)
- moved U6 154.4 mm to (56.0, -76.5)
- moved U7 154.4 mm to (44.1, -72.2)
Connections:
- U17 pad 10: Net-(U17-FLIP) -> I2C1_SCL
- U17 pad 11: unconnected-(U17-VDC_OUT-Pad11) -> Net-(Q3-D)
- U17 pad 12: I2C1_SDA -> I2C1_SCL
- U17 pad 23: unconnected-(U17-VDDD-Pad23) -> +3V3_PD_AON
- U17 pad 24: unconnected-(U17-VCCD-Pad24) -> +1V8_PD_AON
- U17 pad 3: unconnected-(U17-VBUS_FET_EN-Pad3) -> Net-(U17-VBUS_FET_EN)
- U17 pad 9: unconnected-(U17-FAULT-Pad9) -> USB_PD_FAULT
Other:
- board outline added: 160 x 100 mm

Commit message: Link up ADC to FPGA
Parts:
- added R100: 33R, Resistor_SMD:R_0402_1005Metric_Pad0.72x0.64mm_HandSolder, F.Cu at (125.1, 68.8)
- added R101: 33R, Resistor_SMD:R_0402_1005Metric_Pad0.72x0.64mm_HandSolder, F.Cu at (125.1, 67.5)
- added R102: 33R, Resistor_SMD:R_0402_1005Metric_Pad0.72x0.64mm_HandSolder, F.Cu at (125.1, 66.2)
- added R103: 33R, Resistor_SMD:R_0402_1005Metric_Pad0.72x0.64mm_HandSolder, F.Cu at (125.1, 58.5)
- added R104: 33R, Resistor_SMD:R_0402_1005Metric_Pad0.72x0.64mm_HandSolder, F.Cu at (125.1, 57.2)
- added R105: 33R, Resistor_SMD:R_0402_1005Metric_Pad0.72x0.64mm_HandSolder, F.Cu at (125.1, 56.0)
- added R106: 33R, Resistor_SMD:R_0402_1005Metric_Pad0.72x0.64mm_HandSolder, F.Cu at (125.1, 54.8)
- added R107: 33R, Resistor_SMD:R_0402_1005Metric_Pad0.72x0.64mm_HandSolder, F.Cu at (125.5, 107.2)
- added R108: 33R, Resistor_SMD:R_0402_1005Metric_Pad0.72x0.64mm_HandSolder, F.Cu at (125.5, 105.8)
- added R109: 33R, Resistor_SMD:R_0402_1005Metric_Pad0.72x0.64mm_HandSolder, F.Cu at (125.5, 104.4)
- added R110: 33R, Resistor_SMD:R_0402_1005Metric_Pad0.72x0.64mm_HandSolder, F.Cu at (125.5, 103.0)
- added R111: 33R, Resistor_SMD:R_0402_1005Metric_Pad0.72x0.64mm_HandSolder, F.Cu at (125.5, 101.6)
- added R112: 33R, Resistor_SMD:R_0402_1005Metric_Pad0.72x0.64mm_HandSolder, F.Cu at (125.5, 100.2)
- added R113: 33R, Resistor_SMD:R_0402_1005Metric_Pad0.72x0.64mm_HandSolder, F.Cu at (125.5, 98.8)
- added R114: 33R, Resistor_SMD:R_0402_1005Metric_Pad0.72x0.64mm_HandSolder, F.Cu at (125.5, 97.4)
- added R115: 33R, Resistor_SMD:R_0402_1005Metric_Pad0.72x0.64mm_HandSolder, F.Cu at (125.2, 92.0)
- added R116: 33R, Resistor_SMD:R_0402_1005Metric_Pad0.72x0.64mm_HandSolder, F.Cu at (125.2, 90.5)
- added R117: 33R, Resistor_SMD:R_0402_1005Metric_Pad0.72x0.64mm_HandSolder, F.Cu at (125.2, 89.2)
- added R118: 33R, Resistor_SMD:R_0402_1005Metric_Pad0.72x0.64mm_HandSolder, F.Cu at (125.2, 88.0)
- added R95: 33R, Resistor_SMD:R_0402_1005Metric_Pad0.72x0.64mm_HandSolder, F.Cu at (125.1, 75.0)
- added R96: 33R, Resistor_SMD:R_0402_1005Metric_Pad0.72x0.64mm_HandSolder, F.Cu at (125.1, 73.8)
- added R97: 33R, Resistor_SMD:R_0402_1005Metric_Pad0.72x0.64mm_HandSolder, F.Cu at (125.1, 72.5)
- added R98: 33R, Resistor_SMD:R_0402_1005Metric_Pad0.72x0.64mm_HandSolder, F.Cu at (125.1, 71.2)
- added R99: 33R, Resistor_SMD:R_0402_1005Metric_Pad0.72x0.64mm_HandSolder, F.Cu at (125.1, 70.0)
- added TR1: Wuerth_749013011A, Transformer_SMD:Transformer_Ethernet_Wuerth_749013011A, F.Cu at (79.0, 179.0)
- added U10: P0082_BOTTOMMOUNT, P0082_BOTTOMMOUNT:MODULE_P0082_BOTTOMMOUNT, F.Cu at (161.0, 73.0)
- added U28: STM32H723ZGIx, Package_BGA:UFBGA-144_7x7mm_Layout12x12_P0.5mm, F.Cu at (77.9, 191.2)
- added U29: LAN8742A, Package_DFN_QFN:VQFN-24-1EP_4x4mm_P0.5mm_EP2.5x2.5mm_ThermalVias, F.Cu at (76.0, 199.3)
- added U9: NUCLEOH723ZG, NUCLEOH723ZG:MODULE_NUCLEOH723ZG, F.Cu at (204.5, 251.6)
- moved U13 198.9 mm to (115.3, 102.9), turned to 180 degrees
- moved U14 181.3 mm to (115.2, 87.5), turned to 180 degrees
- moved U11 176.0 mm to (115.1, 70.7), turned to 180 degrees
- moved U6 159.7 mm to (95.2, 78.3)
- moved U12 155.7 mm to (115.2, 54.0), turned to 180 degrees
Connections:
- net /adc/D_ADC_A_0 renamed /adc/D_ADC_A0
- net /adc/D_ADC_A_1 renamed /adc/D_ADC_A1
- net /adc/D_ADC_A_10 renamed /adc/D_ADC_A10
- net /adc/D_ADC_A_11 renamed /adc/D_ADC_A11
- net /adc/D_ADC_A_2 renamed /adc/D_ADC_A2
- net /adc/D_ADC_A_3 renamed /adc/D_ADC_A3
- net /adc/D_ADC_A_4 renamed /adc/D_ADC_A4
- net /adc/D_ADC_A_5 renamed /adc/D_ADC_A5
- net /adc/D_ADC_A_6 renamed /adc/D_ADC_A6
- net /adc/D_ADC_A_7 renamed /adc/D_ADC_A7
- net /adc/D_ADC_A_8 renamed /adc/D_ADC_A8
- net /adc/D_ADC_A_9 renamed /adc/D_ADC_A9
- net /adc/D_ADC_B_0 renamed /adc/D_ADC_B0
- net /adc/D_ADC_B_1 renamed /adc/D_ADC_B1
- net /adc/D_ADC_B_10 renamed /adc/D_ADC_B10
- net /adc/D_ADC_B_11 renamed /adc/D_ADC_B11
- net /adc/D_ADC_B_2 renamed /adc/D_ADC_B2
- net /adc/D_ADC_B_3 renamed /adc/D_ADC_B3
- net /adc/D_ADC_B_4 renamed /adc/D_ADC_B4
- net /adc/D_ADC_B_5 renamed /adc/D_ADC_B5
- net /adc/D_ADC_B_6 renamed /adc/D_ADC_B6
- net /adc/D_ADC_B_7 renamed /adc/D_ADC_B7
- net /adc/D_ADC_B_8 renamed /adc/D_ADC_B8
- net /adc/D_ADC_B_9 renamed /adc/D_ADC_B9
- net /fpga/D_ADC0 renamed /fpga/D_ADC_A0
- net /fpga/D_ADC1 renamed /fpga/D_ADC_A1
- net /fpga/D_ADC2 renamed /fpga/D_ADC_A2
- net /fpga/D_ADC3 renamed /fpga/D_ADC_A3
- net /fpga/D_ADC4 renamed /fpga/D_ADC_A4
- net /fpga/D_ADC5 renamed /fpga/D_ADC_A5
- net /fpga/D_ADC6 renamed /fpga/D_ADC_A6
- net /fpga/D_ADC7 renamed /fpga/D_ADC_A7
- U11 pad 2: unconnected-(U11-B1-Pad2) -> Net-(U11-B1)
- U11 pad 3: unconnected-(U11-B2-Pad3) -> Net-(U11-B2)
- U11 pad 4: unconnected-(U11-B3-Pad4) -> Net-(U11-B3)
- U11 pad 5: unconnected-(U11-B4-Pad5) -> Net-(U11-B4)
- U11 pad 6: unconnected-(U11-B5-Pad6) -> Net-(U11-B5)
- U11 pad 7: unconnected-(U11-B6-Pad7) -> Net-(U11-B6)
- U11 pad 8: unconnected-(U11-B7-Pad8) -> Net-(U11-B7)
- U11 pad 9: unconnected-(U11-B8-Pad9) -> Net-(U11-B8)
- U12 pad 16: unconnected-(U12-D4-Pad16) -> /fpga/D_ADC_A11
- U12 pad 17: unconnected-(U12-D3-Pad17) -> /fpga/D_ADC_A10
- U12 pad 18: unconnected-(U12-D2-Pad18) -> /fpga/D_ADC_A9
- U12 pad 19: unconnected-(U12-D1-Pad19) -> /fpga/D_ADC_A8
- U12 pad 2: unconnected-(U12-B1-Pad2) -> Net-(U12-B1)
- U12 pad 3: unconnected-(U12-B2-Pad3) -> Net-(U12-B2)
- U12 pad 4: unconnected-(U12-B3-Pad4) -> Net-(U12-B3)
- U12 pad 5: unconnected-(U12-B4-Pad5) -> Net-(U12-B4)
- U13 pad 12: unconnected-(U13-D8-Pad12) -> /fpga/D_ADC_B7
- U13 pad 13: unconnected-(U13-D7-Pad13) -> /fpga/D_ADC_B6
- U13 pad 14: unconnected-(U13-D6-Pad14) -> /fpga/D_ADC_B5
- U13 pad 15: unconnected-(U13-D5-Pad15) -> /fpga/D_ADC_B4
- U13 pad 16: unconnected-(U13-D4-Pad16) -> /fpga/D_ADC_B3
- U13 pad 17: unconnected-(U13-D3-Pad17) -> /fpga/D_ADC_B2
- U13 pad 18: unconnected-(U13-D2-Pad18) -> /fpga/D_ADC_B1
- U13 pad 19: unconnected-(U13-D1-Pad19) -> /fpga/D_ADC_B0
- U13 pad 2: unconnected-(U13-B1-Pad2) -> Net-(U13-B1)
- U13 pad 3: unconnected-(U13-B2-Pad3) -> Net-(U13-B2)
- U13 pad 4: unconnected-(U13-B3-Pad4) -> Net-(U13-B3)
- U13 pad 5: unconnected-(U13-B4-Pad5) -> Net-(U13-B4)
- U13 pad 6: unconnected-(U13-B5-Pad6) -> Net-(U13-B5)
- U13 pad 7: unconnected-(U13-B6-Pad7) -> Net-(U13-B6)
- U13 pad 8: unconnected-(U13-B7-Pad8) -> Net-(U13-B7)
- U13 pad 9: unconnected-(U13-B8-Pad9) -> Net-(U13-B8)
- U14 pad 16: unconnected-(U14-D4-Pad16) -> /fpga/D_ADC_B11
- U14 pad 17: unconnected-(U14-D3-Pad17) -> /fpga/D_ADC_B10
- U14 pad 18: unconnected-(U14-D2-Pad18) -> /fpga/D_ADC_B9
- U14 pad 19: unconnected-(U14-D1-Pad19) -> /fpga/D_ADC_B8
- U14 pad 2: unconnected-(U14-B1-Pad2) -> Net-(U14-B1)
- U14 pad 3: unconnected-(U14-B2-Pad3) -> Net-(U14-B2)
- U14 pad 4: unconnected-(U14-B3-Pad4) -> Net-(U14-B3)
- U14 pad 5: unconnected-(U14-B4-Pad5) -> Net-(U14-B4)

Commit message: Simplifying the design
Parts:
- removed D10, D2, D6, D7: 1N5822, Diode_THT:D_DO-201AD_P15.24mm_Horizontal
- removed D8, D9: 1N5400, Diode_THT:D_DO-201AD_P15.24mm_Horizontal
- removed Q1: 2N7002, Package_TO_SOT_SMD:SOT-23
- removed Q2, Q3: DMP3099L, Package_TO_SOT_SMD:SOT-23
- removed TR1: Wuerth_749013011A, Transformer_SMD:Transformer_Ethernet_Wuerth_749013011A
- removed U12, U13: SN75160BDW, Package_SO:SOIC-20W_7.5x12.8mm_P1.27mm
- removed U17: CYPD3177-24LQ, Package_DFN_QFN:QFN-24-1EP_4x4mm_P0.5mm_EP2.75x2.75mm
- removed U19: LM2596S-ADJ, Package_TO_SOT_SMD:TO-263-5_TabPin3
- removed U20: INA180A3, Package_TO_SOT_SMD:SOT-23-5
- removed U21, U22: LM2596S-5, Package_TO_SOT_SMD:TO-263-5_TabPin3
- removed U28: STM32H723ZGIx, Package_BGA:UFBGA-144_7x7mm_Layout12x12_P0.5mm
- removed U29: LAN8742A, Package_DFN_QFN:VQFN-24-1EP_4x4mm_P0.5mm_EP2.5x2.5mm_ThermalVias
- added C11: 12pF, Capacitor_SMD:C_0603_1608Metric_Pad1.08x0.95mm_HandSolder, F.Cu at (25.5, 8.71)
- added C12: 12pF, Capacitor_SMD:C_0603_1608Metric_Pad1.08x0.95mm_HandSolder, F.Cu at (25.5, 11.2)
- added R119: 10kR, Resistor_SMD:R_0402_1005Metric_Pad0.72x0.64mm_HandSolder, F.Cu at (375.3, -49.5)
- added R120: 33R, Resistor_SMD:R_0402_1005Metric_Pad0.72x0.64mm_HandSolder, F.Cu at (375.3, -47.5)
- added R121: 33R, Resistor_SMD:R_0402_1005Metric_Pad0.72x0.64mm_HandSolder, F.Cu at (375.3, -45.5)
- added R122: 33R, Resistor_SMD:R_0402_1005Metric_Pad0.72x0.64mm_HandSolder, F.Cu at (375.3, -43.5)
- added R123: 33R, Resistor_SMD:R_0402_1005Metric_Pad0.72x0.64mm_HandSolder, F.Cu at (375.3, -41.5)
- added R124: 33R, Resistor_SMD:R_0402_1005Metric_Pad0.72x0.64mm_HandSolder, F.Cu at (375.3, -39.5)
- added R125: 33R, Resistor_SMD:R_0402_1005Metric_Pad0.72x0.64mm_HandSolder, F.Cu at (375.3, -37.5)
- added R126: 33R, Resistor_SMD:R_0402_1005Metric_Pad0.72x0.64mm_HandSolder, F.Cu at (375.3, -35.5)
- added R127: 33R, Resistor_SMD:R_0402_1005Metric_Pad0.72x0.64mm_HandSolder, F.Cu at (375.3, -33.5)
- added R128: 10kR, Resistor_SMD:R_0402_1005Metric_Pad0.72x0.64mm_HandSolder, F.Cu at (378.6, -49.5)
- added R129: 10kR, Resistor_SMD:R_0402_1005Metric_Pad0.72x0.64mm_HandSolder, F.Cu at (378.6, -47.5)
- added R130: 10kR, Resistor_SMD:R_0402_1005Metric_Pad0.72x0.64mm_HandSolder, F.Cu at (378.6, -45.5)
- added R131: 10kR, Resistor_SMD:R_0402_1005Metric_Pad0.72x0.64mm_HandSolder, F.Cu at (378.6, -43.5)
- added R132: 10kR, Resistor_SMD:R_0402_1005Metric_Pad0.72x0.64mm_HandSolder, F.Cu at (378.6, -41.5)
- added R133: 10kR, Resistor_SMD:R_0402_1005Metric_Pad0.72x0.64mm_HandSolder, F.Cu at (378.6, -39.5)
- added R134: 10kR, Resistor_SMD:R_0402_1005Metric_Pad0.72x0.64mm_HandSolder, F.Cu at (378.6, -37.5)
- added R135: 10kR, Resistor_SMD:R_0402_1005Metric_Pad0.72x0.64mm_HandSolder, F.Cu at (378.6, -35.5)
- added R136: 10kR, Resistor_SMD:R_0402_1005Metric_Pad0.72x0.64mm_HandSolder, F.Cu at (378.6, -33.5)
- added R137: 10kR, Resistor_SMD:R_0402_1005Metric_Pad0.72x0.64mm_HandSolder, F.Cu at (381.8, -49.5)
- added R138: 10kR, Resistor_SMD:R_0402_1005Metric_Pad0.72x0.64mm_HandSolder, F.Cu at (381.8, -47.5)
- added R139: 10kR, Resistor_SMD:R_0402_1005Metric_Pad0.72x0.64mm_HandSolder, F.Cu at (381.8, -45.5)
- added R140: 10kR, Resistor_SMD:R_0402_1005Metric_Pad0.72x0.64mm_HandSolder, F.Cu at (381.8, -43.5)
- added R141: 33R, Resistor_SMD:R_0402_1005Metric_Pad0.72x0.64mm_HandSolder, F.Cu at (381.8, -41.5)
- added R142: 33R, Resistor_SMD:R_0402_1005Metric_Pad0.72x0.64mm_HandSolder, F.Cu at (381.8, -39.5)
- added R143: 33R, Resistor_SMD:R_0402_1005Metric_Pad0.72x0.64mm_HandSolder, F.Cu at (381.8, -37.5)
- added R144: 33R, Resistor_SMD:R_0402_1005Metric_Pad0.72x0.64mm_HandSolder, F.Cu at (381.8, -35.5)
- added R145: 33R, Resistor_SMD:R_0402_1005Metric_Pad0.72x0.64mm_HandSolder, F.Cu at (381.8, -33.5)
- added R146: 33R, Resistor_SMD:R_0402_1005Metric_Pad0.72x0.64mm_HandSolder, F.Cu at (385.1, -49.5)
- added R147: 10kR, Resistor_SMD:R_0402_1005Metric_Pad0.72x0.64mm_HandSolder, F.Cu at (385.1, -47.5)
- added R148: 33R, Resistor_SMD:R_0402_1005Metric_Pad0.72x0.64mm_HandSolder, F.Cu at (385.1, -45.5)
- added R149: 33R, Resistor_SMD:R_0402_1005Metric_Pad0.72x0.64mm_HandSolder, F.Cu at (385.1, -43.5)
- added R150: 33R, Resistor_SMD:R_0402_1005Metric_Pad0.72x0.64mm_HandSolder, F.Cu at (385.1, -41.5)
- added R151: 10kR, Resistor_SMD:R_0402_1005Metric_Pad0.72x0.64mm_HandSolder, F.Cu at (385.1, -39.5)
- added R152: 33R, Resistor_SMD:R_0402_1005Metric_Pad0.72x0.64mm_HandSolder, F.Cu at (385.1, -37.5)
- added R153: 10kR, Resistor_SMD:R_0402_1005Metric_Pad0.72x0.64mm_HandSolder, F.Cu at (385.1, -35.5)
- added R154: 10kR, Resistor_SMD:R_0402_1005Metric_Pad0.72x0.64mm_HandSolder, F.Cu at (385.1, -33.5)
- added R155: 10kR, Resistor_SMD:R_0402_1005Metric_Pad0.72x0.64mm_HandSolder, F.Cu at (388.4, -49.5)
- added R156: 10kR, Resistor_SMD:R_0402_1005Metric_Pad0.72x0.64mm_HandSolder, F.Cu at (388.4, -47.5)
- added R157: 33R, Resistor_SMD:R_0402_1005Metric_Pad0.72x0.64mm_HandSolder, F.Cu at (388.4, -45.5)
- added R158: 33R, Resistor_SMD:R_0402_1005Metric_Pad0.72x0.64mm_HandSolder, F.Cu at (388.4, -43.5)
- added R189: 10kR, Resistor_SMD:R_0402_1005Metric_Pad0.72x0.64mm_HandSolder, F.Cu at (388.4, -41.5)
- added R190: 10kR, Resistor_SMD:R_0402_1005Metric_Pad0.72x0.64mm_HandSolder, F.Cu at (388.4, -39.5)
- added R191: 10kR, Resistor_SMD:R_0402_1005Metric_Pad0.72x0.64mm_HandSolder, F.Cu at (388.4, -37.5)
- added R192: 10kR, Resistor_SMD:R_0402_1005Metric_Pad0.72x0.64mm_HandSolder, F.Cu at (388.4, -35.5)
- added R21: 25R, Resistor_SMD:R_0402_1005Metric_Pad0.72x0.64mm_HandSolder, F.Cu at (25.0, 4.47)
- added R22: 25R, Resistor_SMD:R_0402_1005Metric_Pad0.72x0.64mm_HandSolder, F.Cu at (25.0, 6.46)
- added R4: 25R, Resistor_SMD:R_0402_1005Metric_Pad0.72x0.64mm_HandSolder, F.Cu at (25.0, 0.49)
- added R5: 25R, Resistor_SMD:R_0402_1005Metric_Pad0.72x0.64mm_HandSolder, F.Cu at (25.0, 2.48)
- added R55: 0R, Resistor_SMD:R_0402_1005Metric_Pad0.72x0.64mm_HandSolder, F.Cu at (375.3, -29.6)
- added R56: 0R, Resistor_SMD:R_0402_1005Metric_Pad0.72x0.64mm_HandSolder, F.Cu at (375.3, -27.6)
- added R57: 0R, Resistor_SMD:R_0402_1005Metric_Pad0.72x0.64mm_HandSolder, F.Cu at (375.3, -25.6)
- added R58: 0R, Resistor_SMD:R_0402_1005Metric_Pad0.72x0.64mm_HandSolder, F.Cu at (375.3, -23.6)
- added U3: AD8337BCPZ-REEL-ND, footprints:CP_8_2_ADI, F.Cu at (20.6, 2.26)
- added U5: AD8337BCPZ-REEL-ND, footprints:CP_8_2_ADI, F.Cu at (20.6, 7.78)
- U11, U14: value SN75160BDW -> AD8045ACPZ-R2; footprint Package_SO:SOIC-20W_7.5x12.8mm_P1.27mm -> footprints:CP_8_2_ADI
- moved U9 224.1 mm to (359.4, 89.7), turned to 0 degrees
- moved U10 123.8 mm to (284.5, 63.5)
- moved U14 114.7 mm to (20.6, 22.8), turned to 0 degrees
- moved U11 108.6 mm to (20.6, 17.2), turned to 0 degrees
- moved U2 101.6 mm to (25.5, 16.5)
- moved R107 28.0 mm to (97.7, 103.4)
- moved R108 28.0 mm to (97.7, 102.0)
- moved R113 28.0 mm to (97.7, 95.0)
- moved R114 28.0 mm to (97.7, 93.6)
- moved R100 28.0 mm to (97.4, 64.9)
- moved R101 28.0 mm to (97.4, 63.7)
- moved R102 28.0 mm to (97.4, 62.4)
- moved R103 28.0 mm to (97.4, 54.7)
- moved R104 28.0 mm to (97.4, 53.4)
- moved R105 28.0 mm to (97.4, 52.2)
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Connections:
- R100 pad 1: Net-(U11-B6) -> /adc/D_ADC_A5
- R101 pad 1: Net-(U11-B7) -> /adc/D_ADC_A6
- R102 pad 1: Net-(U11-B8) -> /adc/D_ADC_A7
- R103 pad 1: Net-(U12-B1) -> /adc/D_ADC_A8
- R104 pad 1: Net-(U12-B2) -> /adc/D_ADC_A9
- R105 pad 1: Net-(U12-B3) -> /adc/D_ADC_A10
- R106 pad 1: Net-(U12-B4) -> /adc/D_ADC_A11
- R107 pad 1: Net-(U13-B1) -> /adc/D_ADC_B0
- R108 pad 1: Net-(U13-B2) -> /adc/D_ADC_B1
- R109 pad 1: Net-(U13-B3) -> /adc/D_ADC_B2
- R110 pad 1: Net-(U13-B4) -> /adc/D_ADC_B3
- R111 pad 1: Net-(U13-B5) -> /adc/D_ADC_B4
- R112 pad 1: Net-(U13-B6) -> /adc/D_ADC_B5
- R113 pad 1: Net-(U13-B7) -> /adc/D_ADC_B6
- R114 pad 1: Net-(U13-B8) -> /adc/D_ADC_B7
- R115 pad 1: Net-(U14-B1) -> /adc/D_ADC_B8
- R116 pad 1: Net-(U14-B2) -> /adc/D_ADC_B9
- R117 pad 1: Net-(U14-B3) -> /adc/D_ADC_B10
- R118 pad 1: Net-(U14-B4) -> /adc/D_ADC_B11
- R95 pad 1: Net-(U11-B1) -> /adc/D_ADC_A0
- R96 pad 1: Net-(U11-B2) -> /adc/D_ADC_A1
- R97 pad 1: Net-(U11-B3) -> /adc/D_ADC_A2
- R98 pad 1: Net-(U11-B4) -> /adc/D_ADC_A3
- R99 pad 1: Net-(U11-B5) -> /adc/D_ADC_A4
- U10 pad JP1_10: unconnected-(U10A-GPIO_07-PadJP1_10) -> GPIO_23
- U10 pad JP1_11: unconnected-(U10A-GPIO-0_VCC_SYS-PadJP1_11) -> Net-(U10A-GPIO-0_VCC_SYS)
- U10 pad JP1_12: Net-(U10A-GPIO-0_GND-PadJP1_12) -> GND
- U10 pad JP1_17: unconnected-(U10A-GPIO_012-PadJP1_17) -> GPIO_6
- U10 pad JP1_18: unconnected-(U10A-GPIO_013-PadJP1_18) -> QSPI_CS/GPIO_0
- U10 pad JP1_19: unconnected-(U10A-GPIO_014-PadJP1_19) -> GPIO_7
- U10 pad JP1_20: unconnected-(U10A-GPIO_015-PadJP1_20) -> QSPI_CLK/GPIO_1
- U10 pad JP1_21: unconnected-(U10A-GPIO_016-PadJP1_21) -> GPIO_8
- U10 pad JP1_22: unconnected-(U10A-GPIO_017-PadJP1_22) -> QSPI_IO0/GPIO_2
- U10 pad JP1_23: unconnected-(U10A-GPIO_018-PadJP1_23) -> GPIO_9
- U10 pad JP1_24: unconnected-(U10A-GPIO_019-PadJP1_24) -> QSPI_IO1/GPIO_3
- U10 pad JP1_25: unconnected-(U10A-GPIO_020-PadJP1_25) -> GPIO_10
- U10 pad JP1_26: unconnected-(U10A-GPIO_021-PadJP1_26) -> QSPI_IO2/GPIO_4
- U10 pad JP1_27: unconnected-(U10A-GPIO_022-PadJP1_27) -> GPIO_11
- U10 pad JP1_28: unconnected-(U10A-GPIO_023-PadJP1_28) -> QSPI_IO3/GPIO_5
- U10 pad JP1_29: unconnected-(U10A-GPIO-0_VCC3P3-PadJP1_29) -> Net-(U10A-GPIO-0_VCC3P3)
- U10 pad JP1_30: Net-(U10A-GPIO-0_GND-PadJP1_12) -> GND
- U10 pad JP1_4: unconnected-(U10A-GPIO_01-PadJP1_4) -> GPIO_20
- U10 pad JP1_6: unconnected-(U10A-GPIO_03-PadJP1_6) -> GPIO_21
- U10 pad JP1_7: unconnected-(U10A-GPIO_04-PadJP1_7) -> USART_1_RX
- U10 pad JP1_8: unconnected-(U10A-GPIO_05-PadJP1_8) -> GPIO_22
- U10 pad JP1_9: unconnected-(U10A-GPIO_06-PadJP1_9) -> USART_1_TX
- U10 pad JP2_11: unconnected-(U10B-GPIO-1_VCC_SYS-PadJP2_11) -> Net-(U10B-GPIO-1_VCC_SYS)
- U10 pad JP2_12: Net-(U10B-GPIO-1_GND-PadJP2_12) -> GND
- U10 pad JP2_29: unconnected-(U10B-GPIO-1_VCC3P3-PadJP2_29) -> Net-(U10B-GPIO-1_VCC3P3)
- U10 pad JP2_30: Net-(U10B-GPIO-1_GND-PadJP2_12) -> GND
- U11 pad 2: Net-(U11-B1) -> Net-(U11-FEEDBACK)
- U11 pad 3: Net-(U11-B2) -> CH2_VGA
- U11 pad 4: Net-(U11-B3) -> Net-(U11-+IN)
- U11 pad 5: Net-(U11-B4) -> unconnected-(U11--VS-Pad5)
- U11 pad 6: Net-(U11-B5) -> unconnected-(U11-NC-Pad6)
- U11 pad 7: Net-(U11-B6) -> CH2_VGA
- U11 pad 8: Net-(U11-B7) -> unconnected-(U11-+VS-Pad8)
- U14 pad 2: Net-(U14-B1) -> Net-(U14-FEEDBACK)
- U14 pad 3: Net-(U14-B2) -> Net-(U14--IN)
- U14 pad 4: Net-(U14-B3) -> Net-(U14-+IN)
- U14 pad 5: Net-(U14-B4) -> unconnected-(U14--VS-Pad5)
- U14 pad 7: unconnected-(U14-B6-Pad7) -> CH1_VGA
- U16 pad 1: unconnected-(U16-REF-Pad1) -> Net-(U16-REF)
- U16 pad 10: unconnected-(U16-REFDIV-Pad10) -> GND
- U16 pad 11: unconnected-(U16-~{LDAC}-Pad11) -> GND
- U16 pad 12: unconnected-(U16-~{CS}-Pad12) -> SPI_1_CS
- U16 pad 13: unconnected-(U16-SCLK-Pad13) -> SPI_1_SCK
- U16 pad 14: unconnected-(U16-SDI-Pad14) -> SPI_1_MOSI
- U16 pad 15: unconnected-(U16-SDO/~{ALARM}-Pad15) -> SPI_1_MISO
- U16 pad 16: unconnected-(U16-VIO-Pad16) -> +3V3
- U16 pad 17: unconnected-(U16-EP-Pad17) -> GND
- U16 pad 6: unconnected-(U16-GND-Pad6) -> GND
- U16 pad 7: unconnected-(U16-VDD-Pad7) -> +5V
- U16 pad 8: unconnected-(U16-GAIN-Pad8) -> GND
- U16 pad 9: unconnected-(U16-RSTSEL-Pad9) -> GND
- U4 pad 2: CH2_COMMON -> +1V5
- U6 pad 20: CH2_COMMON -> +1V5
- U6 pad 61: CH1_COMMON -> +1V5
- U7 pad 2: CH1_COMMON -> +1V5
- U9 pad CN10_13: unconnected-(U9F-D26/QSPI_CS-PadCN10_13) -> Net-(U9F-D26/QSPI_CS)
- U9 pad CN10_14: unconnected-(U9F-D1/USART_A_TX-PadCN10_14) -> Net-(U9F-D1/USART_A_TX)
- U9 pad CN10_15: unconnected-(U9F-D27/QSPI_CLK-PadCN10_15) -> Net-(U9F-D27/QSPI_CLK)
- U9 pad CN10_16: unconnected-(U9F-D0/USART_A_RX-PadCN10_16) -> Net-(U9F-D0/USART_A_RX)
- U9 pad CN10_18: unconnected-(U9F-D42/TIMER_A_PWM1N-PadCN10_18) -> Net-(U9F-D42/TIMER_A_PWM1N)
- U9 pad CN10_19: unconnected-(U9F-D28/QSPI_BK1_IO3-PadCN10_19) -> Net-(U9F-D28/QSPI_BK1_IO3)
- U9 pad CN10_20: unconnected-(U9F-D41/TIMER_A_ETR-PadCN10_20) -> Net-(U9F-D41/TIMER_A_ETR)
- U9 pad CN10_21: unconnected-(U9F-D29/QSPI_BK1_IO1-PadCN10_21) -> Net-(U9F-D29/QSPI_BK1_IO1)
- U9 pad CN10_23: unconnected-(U9F-D30/QSPI_BK1_IO0-PadCN10_23) -> Net-(U9F-D30/QSPI_BK1_IO0)
- U9 pad CN10_24: unconnected-(U9F-D40/TIMER_A_PWM2N-PadCN10_24) -> Net-(U9F-D40/TIMER_A_PWM2N)
- U9 pad CN10_25: unconnected-(U9F-D31/QSPI_BK1_IO2-PadCN10_25) -> Net-(U9F-D31/QSPI_BK1_IO2)
- U9 pad CN10_26: unconnected-(U9F-D39/TIMER_A_PWM3N-PadCN10_26) -> Net-(U9F-D39/TIMER_A_PWM3N)
- U9 pad CN10_28: unconnected-(U9F-D38/TIMER_A_BKIN2-PadCN10_28) -> Net-(U9F-D38/TIMER_A_BKIN2)
- U9 pad CN10_29: unconnected-(U9F-D32/TIMER_C_PWM1-PadCN10_29) -> Net-(U9F-D32/TIMER_C_PWM1)
- U9 pad CN10_30: unconnected-(U9F-D37/TIMER_A_BKIN1-PadCN10_30) -> Net-(U9F-D37/TIMER_A_BKIN1)
- U9 pad CN10_31: unconnected-(U9F-D33/TIMER_D_PWM1-PadCN10_31) -> Net-(U9F-D33/TIMER_D_PWM1)
- U9 pad CN10_32: unconnected-(U9F-D36/TIMER_C_PWM2-PadCN10_32) -> Net-(U9F-D36/TIMER_C_PWM2)
- U9 pad CN10_34: unconnected-(U9F-D35/TIMER_C_PWM3-PadCN10_34) -> Net-(U9F-D35/TIMER_C_PWM3)
- U9 pad CN7_10: unconnected-(U9E-D13/SPI_A_SCK-PadCN7_10) -> SPI_1_SCK
- U9 pad CN7_12: unconnected-(U9E-D12/SPI_A_MISO-PadCN7_12) -> SPI_1_MISO
- U9 pad CN7_14: unconnected-(U9E-D11/SPI_A_MOSI/TIM_E_PWM1-PadCN7_14) -> SPI_1_MOSI
- U9 pad CN7_16: unconnected-(U9E-D10/SPI_A_CS/TIM_B_PWM3-PadCN7_16) -> SPI_1_CS
- U9 pad CN8_11: Net-(U9C-GND_CN8-PadCN8_11) -> GND
- U9 pad CN8_13: Net-(U9C-GND_CN8-PadCN8_11) -> GND
- U9 pad CN8_5: unconnected-(U9C-NRST_CN8-PadCN8_5) -> NRST
- U9 pad CN8_9: unconnected-(U9C-5V_CN8-PadCN8_9) -> +5V
- U9 pad CN9_12: Net-(U9D-GND_CN9-PadCN9_12) -> GND
- U9 pad CN9_23: Net-(U9D-GND_CN9-PadCN9_12) -> GND
- U9 pad CN9_25: unconnected-(U9D-D67/CAN_RX-PadCN9_25) -> Net-(U9D-D67/CAN_RX)
- U9 pad CN9_27: unconnected-(U9D-D66/CAN_TX-PadCN9_27) -> Net-(U9D-D66/CAN_TX)

Commit message: Mostly finished schematics, without decoupling and power
Parts:
- removed U6: LTC2299xUP, Package_DFN_QFN:QFN-64-1EP_9x9mm_P0.5mm_EP7.15x7.15mm
- added K1: G2RL-1, Relay_THT:Relay_SPDT_Omron_G2RL-1, F.Cu at (100.5, 88.8)
- added K2: G2RL-1, Relay_THT:Relay_SPDT_Omron_G2RL-1, F.Cu at (132.0, 88.8)
- added Q1: IRL6283M, Package_DirectFET:DirectFET_MD, F.Cu at (29.4, -229.8)
- added Q2: IRL6283M, Package_DirectFET:DirectFET_MD, F.Cu at (29.4, -223.3)
- added Q3: IRL6283M, Package_DirectFET:DirectFET_MD, F.Cu at (29.4, -216.9)
- added Q4: IRL6283M, Package_DirectFET:DirectFET_MD, F.Cu at (29.4, -210.4)
- added Q5: IRL6283M, Package_DirectFET:DirectFET_MD, F.Cu at (29.4, -204.0)
- added R1: 33R, Resistor_SMD:R_1206_3216Metric, F.Cu at (42.2, 34.2)
- added R10: R 49.9k, Resistor_SMD:R_1206_3216Metric, F.Cu at (27.8, -240.0)
- added R11: R 953k, Resistor_SMD:R_1206_3216Metric, F.Cu at (27.8, -236.7)
- added R12: R 47k, Resistor_SMD:R_1206_3216Metric, F.Cu at (33.4, -256.5)
- added R13: 33R, Resistor_SMD:R_1206_3216Metric, F.Cu at (33.4, -253.2)
- added R14: R 49.9k, Resistor_SMD:R_1206_3216Metric, F.Cu at (33.4, -249.9)
- added R15: R 953k, Resistor_SMD:R_1206_3216Metric, F.Cu at (33.4, -246.6)
- added R159: 33R, Resistor_SMD:R_1206_3216Metric, F.Cu at (92.3, -226.7)
- added R16: 33 R, Resistor_SMD:R_1206_3216Metric, F.Cu at (33.4, -243.3)
- added R160: 33R, Resistor_SMD:R_1206_3216Metric, F.Cu at (92.3, -223.4)
- added R161: 33R, Resistor_SMD:R_1206_3216Metric, F.Cu at (92.3, -220.1)
- added R162: 10kR, Resistor_SMD:R_1206_3216Metric, F.Cu at (42.3, -221.4)
- added R163: 10kR, Resistor_SMD:R_1206_3216Metric, F.Cu at (42.3, -218.1)
- added R164: 10kR, Resistor_SMD:R_1206_3216Metric, F.Cu at (42.3, -214.8)
- added R165: 10kR, Resistor_SMD:R_1206_3216Metric, F.Cu at (42.3, -211.5)
- added R166: 33R, Resistor_SMD:R_1206_3216Metric, F.Cu at (42.3, -208.2)
- added R167: 33R, Resistor_SMD:R_1206_3216Metric, F.Cu at (47.9, -231.3)
- added R168: 33R, Resistor_SMD:R_1206_3216Metric, F.Cu at (47.9, -228.0)
- added R169: 33R, Resistor_SMD:R_1206_3216Metric, F.Cu at (47.9, -224.7)
- added R17: 25R, Resistor_SMD:R_1206_3216Metric, F.Cu at (71.9, -227.6)
- added R170: 33R, Resistor_SMD:R_1206_3216Metric, F.Cu at (47.9, -221.4)
- added R171: 33R, Resistor_SMD:R_1206_3216Metric, F.Cu at (47.9, -218.1)
- added R172: 10kR, Resistor_SMD:R_1206_3216Metric, F.Cu at (47.9, -214.8)
- added R173: 10kR, Resistor_SMD:R_1206_3216Metric, F.Cu at (47.9, -211.5)
- added R174: 10kR, Resistor_SMD:R_1206_3216Metric, F.Cu at (47.9, -208.2)
- added R175: 10kR, Resistor_SMD:R_1206_3216Metric, F.Cu at (53.5, -231.3)
- added R176: 10kR, Resistor_SMD:R_1206_3216Metric, F.Cu at (53.5, -228.0)
- added R177: 10kR, Resistor_SMD:R_1206_3216Metric, F.Cu at (53.5, -224.7)
- added R178: 10kR, Resistor_SMD:R_1206_3216Metric, F.Cu at (53.5, -221.4)
- added R179: 10kR, Resistor_SMD:R_1206_3216Metric, F.Cu at (53.5, -218.1)
- added R18: 360R, Resistor_SMD:R_1206_3216Metric, F.Cu at (71.9, -224.2)
- added R180: 33R, Resistor_SMD:R_1206_3216Metric, F.Cu at (92.3, -216.8)
- added R181: 33R, Resistor_SMD:R_1206_3216Metric, F.Cu at (92.3, -213.5)
- added R182: 33R, Resistor_SMD:R_1206_3216Metric, F.Cu at (53.5, -214.8)
- added R183: 470R, Resistor_SMD:R_1206_3216Metric, F.Cu at (53.5, -211.5)
- added R184: 470R, Resistor_SMD:R_1206_3216Metric, F.Cu at (53.5, -208.2)
- added R185: 470R, Resistor_SMD:R_1206_3216Metric, F.Cu at (59.1, -231.3)
- added R186: 470R, Resistor_SMD:R_1206_3216Metric, F.Cu at (59.1, -228.0)
- added R187: 470R, Resistor_SMD:R_1206_3216Metric, F.Cu at (59.1, -224.7)
- added R188: 10k, Resistor_SMD:R_1206_3216Metric, F.Cu at (59.1, -221.4)
- added R19: 360R, Resistor_SMD:R_1206_3216Metric, F.Cu at (71.9, -220.9)
- added R193: 10k, Resistor_SMD:R_1206_3216Metric, F.Cu at (59.1, -218.1)
- added R194: 10k, Resistor_SMD:R_1206_3216Metric, F.Cu at (59.1, -214.8)
- added R195: 10k, Resistor_SMD:R_1206_3216Metric, F.Cu at (59.1, -211.5)
- added R196: 10k, Resistor_SMD:R_1206_3216Metric, F.Cu at (59.1, -208.2)
- added R197: 33 R, Resistor_SMD:R_1206_3216Metric, F.Cu at (83.1, -227.6)
- added R198: 33 R, Resistor_SMD:R_1206_3216Metric, F.Cu at (83.1, -224.2)
- added R199: 25R, Resistor_SMD:R_1206_3216Metric, F.Cu at (83.1, -220.9)
- added R2: 33R, Resistor_SMD:R_1206_3216Metric, F.Cu at (27.8, -253.2)
- added R20: DNP, Resistor_SMD:R_1206_3216Metric, F.Cu at (33.4, -240.0)
- added R200: 49.9 R, Resistor_SMD:R_1206_3216Metric, F.Cu at (83.1, -217.6)
- added R23: R, Resistor_SMD:R_1206_3216Metric, F.Cu at (33.4, -236.7)
- added R24: 360R, Resistor_SMD:R_1206_3216Metric, F.Cu at (71.9, -217.6)
- added R25: 360R, Resistor_SMD:R_1206_3216Metric, F.Cu at (71.9, -214.3)
- added R26: 72 R, Resistor_SMD:R_1206_3216Metric, F.Cu at (71.9, -211.0)
- added R27: 72R, Resistor_SMD:R_1206_3216Metric, F.Cu at (77.5, -234.2)
- added R28: 100 R, Resistor_SMD:R_1206_3216Metric, F.Cu at (77.5, -230.9)
- added R29: 100 R, Resistor_SMD:R_1206_3216Metric, F.Cu at (77.5, -227.6)
- added R3: R 953k, Resistor_SMD:R_1206_3216Metric, F.Cu at (27.8, -249.9)
- added R30: 100 R, Resistor_SMD:R_1206_3216Metric, F.Cu at (77.5, -224.2)
- added R31: 100 R, Resistor_SMD:R_1206_3216Metric, F.Cu at (77.5, -220.9)
- added R32: 25R, Resistor_SMD:R_1206_3216Metric, F.Cu at (77.5, -217.6)
- added R33: R, Resistor_SMD:R_1206_3216Metric, F.Cu at (39.0, -256.5)
- added R34: DNP, Resistor_SMD:R_1206_3216Metric, F.Cu at (39.0, -253.2)
- added R35: R, Resistor_SMD:R_1206_3216Metric, F.Cu at (77.5, -214.3)
- added R36: 33 R, Resistor_SMD:R_1206_3216Metric, F.Cu at (77.5, -211.0)
- added R37: 33R, Resistor_SMD:R_1206_3216Metric, F.Cu at (39.0, -249.9)
- added R38: 10k, Resistor_SMD:R_1206_3216Metric, F.Cu at (39.0, -246.6)
- added R39: 10k, Resistor_SMD:R_1206_3216Metric, F.Cu at (39.0, -243.3)
- added R40: 16k, Resistor_SMD:R_1206_3216Metric, F.Cu at (39.0, -240.0)
- added R41: 33R, Resistor_SMD:R_1206_3216Metric, F.Cu at (39.0, -236.7)
- added R42: 8k, Resistor_SMD:R_1206_3216Metric, F.Cu at (44.6, -256.5)
- added R43: 25R, Resistor_SMD:R_1206_3216Metric, F.Cu at (83.1, -234.2)
- added R44: 49.9 R, Resistor_SMD:R_1206_3216Metric, F.Cu at (83.1, -230.9)
- added R45: 10k, Resistor_SMD:R_1206_3216Metric, F.Cu at (44.6, -253.2)
- added R46: 10k, Resistor_SMD:R_1206_3216Metric, F.Cu at (44.6, -249.9)
- added R47: 16k, Resistor_SMD:R_1206_3216Metric, F.Cu at (44.6, -246.6)
- added R48: 16k, Resistor_SMD:R_1206_3216Metric, F.Cu at (44.6, -243.3)
- added R49: 8k, Resistor_SMD:R_1206_3216Metric, F.Cu at (44.6, -240.0)
- added R50: 120, Resistor_SMD:R_1206_3216Metric, F.Cu at (81.8, -287.0)
- added R51: 16k, Resistor_SMD:R_1206_3216Metric, F.Cu at (44.6, -236.7)
- added R52: 560, Resistor_SMD:R_1206_3216Metric, F.Cu at (81.8, -283.7)
- added R53: 10k, Resistor_SMD:R_1206_3216Metric, F.Cu at (50.2, -256.5)
- added R54: 10k, Resistor_SMD:R_1206_3216Metric, F.Cu at (50.2, -253.2)
- added R59: 0R, Resistor_SMD:R_1206_3216Metric, F.Cu at (50.2, -249.9)
- added R6: 72R, Resistor_SMD:R_1206_3216Metric, F.Cu at (71.9, -234.2)
- added R60: 10k, Resistor_SMD:R_1206_3216Metric, F.Cu at (50.2, -246.6)
- added R61: 5K1, Resistor_SMD:R_1206_3216Metric, F.Cu at (81.8, -280.4)
- added R62: 5K1, Resistor_SMD:R_1206_3216Metric, F.Cu at (81.8, -277.1)
- added R63: 10k, Resistor_SMD:R_1206_3216Metric, F.Cu at (50.2, -243.3)
- added R64: 0R, Resistor_SMD:R_1206_3216Metric, F.Cu at (50.2, -240.0)
- added R65: R, Resistor_SMD:R_1206_3216Metric, F.Cu at (81.8, -273.7)
- added R66: R, Resistor_SMD:R_1206_3216Metric, F.Cu at (87.4, -287.0)
- added R67: R, Resistor_SMD:R_1206_3216Metric, F.Cu at (87.4, -283.7)
- added R68: R, Resistor_SMD:R_1206_3216Metric, F.Cu at (87.4, -280.4)
- added R69: R, Resistor_SMD:R_1206_3216Metric, F.Cu at (87.4, -277.1)
- added R7: 72R, Resistor_SMD:R_1206_3216Metric, F.Cu at (71.9, -230.9)
- added R70: R, Resistor_SMD:R_1206_3216Metric, F.Cu at (87.4, -273.7)
- added R71: R, Resistor_SMD:R_1206_3216Metric, F.Cu at (93.0, -287.0)
- added R72: R, Resistor_SMD:R_1206_3216Metric, F.Cu at (93.0, -283.7)
- added R73: 33R, Resistor_SMD:R_1206_3216Metric, F.Cu at (36.7, -231.3)
- added R74: 10kR, Resistor_SMD:R_1206_3216Metric, F.Cu at (36.7, -228.0)
- added R75: 33R, Resistor_SMD:R_1206_3216Metric, F.Cu at (36.7, -224.7)
- added R76: 12K, Resistor_SMD:R_1206_3216Metric, F.Cu at (93.0, -280.4)
- added R77: 33R, Resistor_SMD:R_1206_3216Metric, F.Cu at (36.7, -221.4)
- added R78: 33R, Resistor_SMD:R_1206_3216Metric, F.Cu at (36.7, -218.1)
- added R79: 33R, Resistor_SMD:R_1206_3216Metric, F.Cu at (36.7, -214.8)
- added R8: R 953k, Resistor_SMD:R_1206_3216Metric, F.Cu at (21.0, -79.3)
- added R80: 33R, Resistor_SMD:R_1206_3216Metric, F.Cu at (36.7, -211.5)
- added R81: 33R, Resistor_SMD:R_1206_3216Metric, F.Cu at (36.7, -208.2)
- added R82: 33R, Resistor_SMD:R_1206_3216Metric, F.Cu at (42.3, -231.3)
- added R83: 33R, Resistor_SMD:R_1206_3216Metric, F.Cu at (92.3, -230.1)
- added R84: 120, Resistor_SMD:R_1206_3216Metric, F.Cu at (100.6, -287.0)
- added R85: 560, Resistor_SMD:R_1206_3216Metric, F.Cu at (100.6, -283.7)
- added R86: R, Resistor_SMD:R_1206_3216Metric, F.Cu at (100.6, -280.4)
- added R87: R, Resistor_SMD:R_1206_3216Metric, F.Cu at (100.6, -277.1)
- added R88: R, Resistor_SMD:R_1206_3216Metric, F.Cu at (100.6, -273.7)
- added R89: R, Resistor_SMD:R_1206_3216Metric, F.Cu at (100.6, -270.4)
- added R9: R 22.2k, Resistor_SMD:R_1206_3216Metric, F.Cu at (21.0, -76.0)
- added R90: R, Resistor_SMD:R_1206_3216Metric, F.Cu at (100.6, -267.1)
- added R91: R, Resistor_SMD:R_1206_3216Metric, F.Cu at (100.6, -263.8)
- added R92: R, Resistor_SMD:R_1206_3216Metric, F.Cu at (100.6, -260.5)
- added R93: R, Resistor_SMD:R_1206_3216Metric, F.Cu at (100.6, -257.2)
- added R94: 33R, Resistor_SMD:R_1206_3216Metric, F.Cu at (50.2, -236.7)
- added TP1: TestPoint, Connector_PinHeader_2.54mm:PinHeader_1x01_P2.54mm_Vertical, F.Cu at (55.6, -286.3)
- added TP10: TestPoint, Connector_PinHeader_2.54mm:PinHeader_1x01_P2.54mm_Vertical, F.Cu at (60.2, -272.6)
- added TP11: TestPoint, Connector_PinHeader_2.54mm:PinHeader_1x01_P2.54mm_Vertical, F.Cu at (60.2, -268.0)
- added TP12: TestPoint, Connector_PinHeader_2.54mm:PinHeader_1x01_P2.54mm_Vertical, F.Cu at (60.2, -263.4)
- added TP13: TestPoint, Connector_PinHeader_2.54mm:PinHeader_1x01_P2.54mm_Vertical, F.Cu at (64.8, -286.3)
- added TP14: TestPoint, Connector_PinHeader_2.54mm:PinHeader_1x01_P2.54mm_Vertical, F.Cu at (64.8, -281.8)
- added TP15: TestPoint, Connector_PinHeader_2.54mm:PinHeader_1x01_P2.54mm_Vertical, F.Cu at (64.8, -277.2)
- added TP16: TestPoint, Connector_PinHeader_2.54mm:PinHeader_1x01_P2.54mm_Vertical, F.Cu at (64.8, -272.6)
- added TP17: TestPoint, Connector_PinHeader_2.54mm:PinHeader_1x01_P2.54mm_Vertical, F.Cu at (64.8, -268.0)
- added TP18: TestPoint, Connector_PinHeader_2.54mm:PinHeader_1x01_P2.54mm_Vertical, F.Cu at (64.8, -263.4)
- added TP19: TestPoint, Connector_PinHeader_2.54mm:PinHeader_1x01_P2.54mm_Vertical, F.Cu at (71.4, -242.7)
- added TP2: TestPoint, Connector_PinHeader_2.54mm:PinHeader_1x01_P2.54mm_Vertical, F.Cu at (55.6, -281.8)
- added TP20: TestPoint, Connector_PinHeader_2.54mm:PinHeader_1x01_P2.54mm_Vertical, F.Cu at (71.4, -238.1)
- added TP21: TestPoint, Connector_PinHeader_2.54mm:PinHeader_1x01_P2.54mm_Vertical, F.Cu at (76.0, -242.7)
- added TP22: TestPoint, Connector_PinHeader_2.54mm:PinHeader_1x01_P2.54mm_Vertical, F.Cu at (76.0, -238.1)
- added TP23: TestPoint, Connector_PinHeader_2.54mm:PinHeader_1x01_P2.54mm_Vertical, F.Cu at (80.6, -242.7)
- added TP24: TestPoint, Connector_PinHeader_2.54mm:PinHeader_1x01_P2.54mm_Vertical, F.Cu at (80.6, -238.1)
- added TP25: TestPoint, Connector_PinHeader_2.54mm:PinHeader_1x01_P2.54mm_Vertical, F.Cu at (85.2, -242.7)
- added TP26: TestPoint, Connector_PinHeader_2.54mm:PinHeader_1x01_P2.54mm_Vertical, F.Cu at (85.2, -238.1)
- added TP3: TestPoint, Connector_PinHeader_2.54mm:PinHeader_1x01_P2.54mm_Vertical, F.Cu at (55.6, -277.2)
- added TP4: TestPoint, Connector_PinHeader_2.54mm:PinHeader_1x01_P2.54mm_Vertical, F.Cu at (55.6, -272.6)
- added TP5: TestPoint, Connector_PinHeader_2.54mm:PinHeader_1x01_P2.54mm_Vertical, F.Cu at (55.6, -268.0)
- added TP6: TestPoint, Connector_PinHeader_2.54mm:PinHeader_1x01_P2.54mm_Vertical, F.Cu at (55.6, -263.4)
- added TP7: TestPoint, Connector_PinHeader_2.54mm:PinHeader_1x01_P2.54mm_Vertical, F.Cu at (60.2, -286.3)
- added TP8: TestPoint, Connector_PinHeader_2.54mm:PinHeader_1x01_P2.54mm_Vertical, F.Cu at (60.2, -281.8)
- added TP9: TestPoint, Connector_PinHeader_2.54mm:PinHeader_1x01_P2.54mm_Vertical, F.Cu at (60.2, -277.2)
- added U15: AP1117-ADJ, Package_TO_SOT_SMD:SOT-223-3_TabPin2, F.Cu at (74.0, -284.4)
- added U17: AP1117-ADJ, Package_TO_SOT_SMD:SOT-223-3_TabPin2, F.Cu at (74.0, -276.1)
- added U18: AP1117-ADJ, Package_TO_SOT_SMD:SOT-223-3_TabPin2, F.Cu at (74.0, -267.8)
- added U19: AP1117-ADJ, Package_TO_SOT_SMD:SOT-223-3_TabPin2, F.Cu at (74.0, -259.5)
- added U20: AP1117-ADJ, Package_TO_SOT_SMD:SOT-223-3_TabPin2, F.Cu at (74.0, -251.1)
- added U21: LTC2299xUP, Package_DFN_QFN:QFN-64-1EP_9x9mm_P0.5mm_EP7.15x7.15mm, F.Cu at (123.2, 57.9)
- R100, R101, R102, R103, R104, R105, R106, R107, R108, R109, R110, R111, R112, R113, R114, R115, R116, R117, R118, R119, R120, R121, R122, R124, R125, R126, R127, R128, R129, R130, R131, R132, R133, R134, R135, R136, R137, R138, R139, R140, R141, R142, R143, R144, R145, R146, R147, R148, R149, R150, R151, R152, R153, R154, R155, R156, R157, R158, R189, R190, R191, R192, R21, R22, R4, R5, R55, R56, R57, R58, R95, R96, R97, R98, R99: footprint Resistor_SMD:R_0402_1005Metric_Pad0.72x0.64mm_HandSolder -> Resistor_SMD:R_1206_3216Metric
- R123: value 33R -> 10kR; footprint Resistor_SMD:R_0402_1005Metric_Pad0.72x0.64mm_HandSolder -> Resistor_SMD:R_1206_3216Metric
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Connections:
- K10 pad A1: unconnected-(K10-PadA1) -> +5V
- K10 pad A2: unconnected-(K10-PadA2) -> AD_DC
- K8 pad A1: unconnected-(K8-PadA1) -> +5V
- K8 pad A2: unconnected-(K8-PadA2) -> CH1_ATTEN
- K9 pad A1: unconnected-(K9-PadA1) -> +5V
- K9 pad A2: unconnected-(K9-PadA2) -> CH2_ATTEN
- R119 pad 2: GPIO_7 -> GPIO_PE11
- R122 pad 1: GPIO_6 -> GPIO_PE15
- R123 pad 1: GPIO_7 -> +3V3
- R123 pad 2: Net-(U9F-D38/TIMER_A_BKIN2) -> GPIO_PE13
- R124 pad 1: GPIO_8 -> GPIO_PE12
- R125 pad 1: GPIO_9 -> GPIO_PE10
- R126 pad 1: GPIO_10 -> GPIO_PE7
- R127 pad 1: GPIO_11 -> GPIO_PE8
- R128 pad 2: GPIO_8 -> GPIO_PE12
- R129 pad 2: GPIO_6 -> GPIO_PE15
- R130 pad 2: GPIO_9 -> GPIO_PE10
- R131 pad 2: GPIO_10 -> GPIO_PE7
- R132 pad 2: GPIO_11 -> GPIO_PE8
- R141 pad 2: QSPI_CS/GPIO_0 -> QSPI_CS
- R142 pad 2: QSPI_CLK/GPIO_1 -> QSPI_CLK
- R143 pad 2: QSPI_IO0/GPIO_2 -> QSPI_IO0/GPIO_PD11
- R144 pad 2: QSPI_IO1/GPIO_3 -> QSPI_IO1/GPIO_PD12
- R145 pad 2: QSPI_IO2/GPIO_4 -> QSPI_IO2/GPIO_PE2
- R146 pad 2: QSPI_IO3/GPIO_5 -> QSPI_IO3/GPIO_PD13
- R148 pad 2: GPIO_20 -> GPIO_4
- R149 pad 2: GPIO_21 -> GPIO_3
- R150 pad 2: GPIO_22 -> GPIO_2
- R152 pad 2: GPIO_23 -> GPIO_1
- R157 pad 2: GPIO_20 -> GPIO_PD1
- R158 pad 2: GPIO_21 -> GPIO_PD0
- U10 pad JP1_13: unconnected-(U10A-GPIO_08-PadJP1_13) -> OE_A
- U10 pad JP1_15: unconnected-(U10A-GPIO_010-PadJP1_15) -> OE_B
- U10 pad JP1_31: unconnected-(U10A-GPIO_024-PadJP1_31) -> Net-(U10A-GPIO_024)
- U10 pad JP1_33: unconnected-(U10A-GPIO_026-PadJP1_33) -> Net-(U10A-GPIO_026)
- U10 pad JP1_5: unconnected-(U10A-GPIO_02-PadJP1_5) -> CLIPPING
- U10 pad JP2_27: unconnected-(U10B-GPIO_122-PadJP2_27) -> ADC_B_12
- U10 pad JP2_31: unconnected-(U10B-GPIO_124-PadJP2_31) -> ADC_B_13
- U10 pad JP2_37: unconnected-(U10B-GPIO_130-PadJP2_37) -> ADC_A_13
- U10 pad JP2_39: unconnected-(U10B-GPIO_132-PadJP2_39) -> ADC_A_12
- U11 pad 3: CH2_VGA -> Net-(U11--IN)
- U11 pad 5: unconnected-(U11--VS-Pad5) -> -5V
- U11 pad 8: unconnected-(U11-+VS-Pad8) -> +5V
- U14 pad 8: unconnected-(U14-+VS-Pad8) -> +5V
- U9 pad CN10_10: unconnected-(U9F-D3/TIMER_A_PWM3-PadCN10_10) -> Net-(U9F-D3/TIMER_A_PWM3)
- U9 pad CN10_17: Net-(U9F-GND_CN10-PadCN10_17) -> GND
- U9 pad CN10_22: Net-(U9F-GND_CN10-PadCN10_17) -> GND
- U9 pad CN10_27: Net-(U9F-GND_CN10-PadCN10_17) -> GND
- U9 pad CN10_28: Net-(U9F-D38/TIMER_A_BKIN2) -> unconnected-(U9F-D38/TIMER_A_BKIN2-PadCN10_28)
- U9 pad CN10_3: unconnected-(U9F-AGND_CN10-PadCN10_3) -> GND
- U9 pad CN10_33: unconnected-(U9F-D34/TIMER_B_ETR-PadCN10_33) -> Net-(U9F-D34/TIMER_B_ETR)
- U9 pad CN10_4: unconnected-(U9F-D6/TIMER_A_PWM1-PadCN10_4) -> Net-(U9F-D6/TIMER_A_PWM1)
- U9 pad CN10_5: Net-(U9F-GND_CN10-PadCN10_17) -> GND
- U9 pad CN10_6: unconnected-(U9F-D5/TIMER_A_PWM2-PadCN10_6) -> Net-(U9F-D5/TIMER_A_PWM2)
- U9 pad CN10_8: unconnected-(U9F-D4/IO-PadCN10_8) -> Net-(U9F-D4/IO)
- U9 pad CN7_17: unconnected-(U9E-D24/SPI_B_NSS-PadCN7_17) -> Net-(U9E-D24/SPI_B_NSS)
- U9 pad CN7_18: unconnected-(U9E-D9/TIMER_B_PWM2-PadCN7_18) -> GPIO_PD15
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Other:
- board size 160 x 100 mm -> 160 x 149.3 mm
