File: DigitalOsciloscope.kicad_pcb (KiCad board)
At the start: 2 copper layers, 160 x 149.3 mm, 264 parts, among them J1 Conn_Coaxial, J2 Conn_Coaxial, J7 Conn_Coaxial, K1 G2RL-1, K10 G2RL-2, K2 G2RL-1, K8 G2RL-2, K9 G2RL-2, Q1 IRL6283M, Q2 IRL6283M, Q3 IRL6283M, Q4 IRL6283M, Q5 IRL6283M, U1 OPA656U, U10 P0082_BOTTOMMOUNT, U11 AD8045ACPZ-R2, U14 AD8045ACPZ-R2, U15 AP1117-ADJ, U16 DAC80504, U17 AP1117-ADJ, U18 AP1117-ADJ, U19 AP1117-ADJ, U2 LTC6754xSC6, U20 AP1117-ADJ, U21 LTC2299xUP, U23 AP1117-ADJ, U24 AP1117-ADJ, U25 AP1117-ADJ, U26 AP1117-ADJ, U27 AP1117-ADJ, U3 AD8337BCPZ-REEL-ND, U4 LMH6551MA, U5 AD8337BCPZ-REEL-ND, U7 LMH6551MA, U8 OPA656U, U9 NUCLEOH723ZG

Commit message: Finished schematic?
Parts:
- removed R65, R66, R69, R70, R71, R72, R86, R87, R88, R89, R90, R91, R92, R93: R, Resistor_SMD:R_1206_3216Metric
- removed R84: 120, Resistor_SMD:R_1206_3216Metric
- removed R85: 560, Resistor_SMD:R_1206_3216Metric
- removed U17, U19, U20, U23, U24, U25, U26, U27: AP1117-ADJ, Package_TO_SOT_SMD:SOT-223-3_TabPin2
- added R203: 240, Resistor_SMD:R_1206_3216Metric, F.Cu at (12.2, 7.78)
- added R204: 430, Resistor_SMD:R_1206_3216Metric, F.Cu at (12.2, 11.1)
- added U22: AP1117-ADJ, Package_TO_SOT_SMD:SOT-223-3_TabPin2, F.Cu at (4.42, 12.0)
- R56, R58: value 0R -> DNP
- R67: value R -> 120
- R68: value R -> 200
- moved R67 294.6 mm to (12.2, 1.16)
- moved R68 294.6 mm to (12.2, 4.46)
- moved U18 280.3 mm to (4.42, 3.70)
- moved R15 54.5 mm to (23.8, -192.9)
- moved R38 54.5 mm to (29.4, -192.9)
- moved R47 54.5 mm to (35.0, -192.9)
- moved R50 54.5 mm to (72.2, -233.3)
- moved R52 54.5 mm to (72.2, -230.0)
- moved R60 54.5 mm to (40.6, -192.9)
- moved R61 54.5 mm to (72.2, -226.7)
- moved R62 54.5 mm to (72.2, -223.4)
- moved R76 54.5 mm to (83.4, -226.7)
- moved TP11 54.5 mm to (50.6, -214.3)
- moved TP15 54.5 mm to (55.2, -223.5)
- moved TP17 54.5 mm to (55.2, -214.3)
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Connections:
- R50 pad 1: Net-(U15-VO) -> +6V5
- R67 pad 1: Net-(U18-VO) -> +3V3
- U1 pad 4: -5V -> Net-(U1--VS)
- U1 pad 7: +5V -> Net-(U1-+VS)
- U11 pad 5: -5V -> Net-(U11--VS)
- U11 pad 8: +5V -> Net-(U11-+VS)
- U14 pad 5: unconnected-(U14--VS-Pad5) -> Net-(U14--VS)
- U14 pad 8: +5V -> Net-(U14-+VS)
- U15 pad 2: Net-(U15-VO) -> +6V5
- U15 pad 3: +9V -> Net-(U15-VI)
- U18 pad 2: Net-(U18-VO) -> +3V3
- U18 pad 3: +5V -> Net-(U18-VI)
- U21 pad 10: +3V3 -> Net-(J5-Pin_1)
- U21 pad 18: +3V3 -> Net-(C39-Pad1)
- U21 pad 21: +3V3 -> Net-(J5-Pin_1)
- U21 pad 32: +1V2 -> Net-(C46-Pad1)
- U21 pad 49: +1V2 -> Net-(C19-Pad1)
- U21 pad 63: +3V3 -> Net-(C39-Pad1)
- U21 pad 7: +3V3 -> Net-(J5-Pin_1)
- U3 pad 6: -5V -> Net-(U3-VNEG)
- U3 pad 8: +5V -> Net-(U3-VPOS)
- U4 pad 3: +6V5 -> Net-(U4-V+)
- U4 pad 6: -3V5 -> Net-(U4-V-)
- U5 pad 6: -5V -> Net-(U5-VNEG)
- U5 pad 8: +5V -> Net-(U5-VPOS)
- U7 pad 3: +6V5 -> Net-(U7-V+)
- U7 pad 6: -3V5 -> Net-(U7-V-)
- U8 pad 4: -5V -> Net-(U8--VS)
- U8 pad 7: +5V -> Net-(U8-+VS)

Commit message: Added first dirty BOM
Parts:
- removed K1, K2: G2RL-1, Relay_THT:Relay_SPDT_Omron_G2RL-1
- removed K10, K9: G2RL-2, Relay_THT:Relay_DPDT_Omron_G2RL-2
- removed Q1, Q2, Q3, Q4, Q5: IRL6283M, Package_DirectFET:DirectFET_MD
- removed R109, R110, R111, R112, R113, R114, R115, R116, R117, R118, R159, R160, R161, R182: 33R, Resistor_SMD:R_1206_3216Metric
- removed R184, R185, R186, R187: 470R, Resistor_SMD:R_1206_3216Metric
- removed R193, R194, R195, R196: 10k, Resistor_SMD:R_1206_3216Metric
- removed R197: 33 R, Resistor_SMD:R_1206_3216Metric
- removed R203: 240, Resistor_SMD:R_1206_3216Metric
- removed R204: 430, Resistor_SMD:R_1206_3216Metric
- removed U16: DAC80504, Package_DFN_QFN:Texas_RTE0016D_WQFN-16-1EP_3x3mm_P0.5mm_EP0.8x0.8mm_ThermalVias
- removed U22: AP1117-ADJ, Package_TO_SOT_SMD:SOT-223-3_TabPin2
- removed U4, U7: LMH6551MA, Package_SO:SOIC-8_3.9x4.9mm_P1.27mm
- added C1: 22nF, Capacitor_SMD:C_0805_2012Metric, F.Cu at (39.0, -140.0)
- added C10: 22nF, Capacitor_SMD:C_0805_2012Metric, F.Cu at (39.0, -112.9)
- added C100: 0.1uF, Capacitor_SMD:C_0805_2012Metric, F.Cu at (85.7, -78.1)
- added C101: 100pF, Capacitor_SMD:C_0805_2012Metric, F.Cu at (90.2, -90.1)
- added C102: 1uF, Capacitor_SMD:C_0805_2012Metric, F.Cu at (90.2, -87.1)
- added C103: 100nF, Capacitor_SMD:C_0805_2012Metric, F.Cu at (56.8, -140.0)
- added C104: 1uF, Capacitor_SMD:C_0805_2012Metric, F.Cu at (56.8, -137.0)
- added C105: 10uF, Capacitor_SMD:C_0805_2012Metric, F.Cu at (56.8, -134.0)
- added C106: 100nF, Capacitor_SMD:C_0805_2012Metric, F.Cu at (56.8, -131.0)
- added C107: 1uF, Capacitor_SMD:C_0805_2012Metric, F.Cu at (56.8, -128.0)
- added C108: 10uF, Capacitor_SMD:C_0805_2012Metric, F.Cu at (56.8, -125.0)
- added C109: 0.1uF, Capacitor_SMD:C_0805_2012Metric, F.Cu at (90.2, -84.1)
- added C110: 100pF, Capacitor_SMD:C_0805_2012Metric, F.Cu at (90.2, -81.1)
- added C111: 0.1uF, Capacitor_SMD:C_0805_2012Metric, F.Cu at (90.2, -78.1)
- added C112: 1uF, Capacitor_SMD:C_0805_2012Metric, F.Cu at (94.6, -90.1)
- added C113: 100pF, Capacitor_SMD:C_0805_2012Metric, F.Cu at (94.6, -87.1)
- added C114: 0.1uF, Capacitor_SMD:C_0805_2012Metric, F.Cu at (94.6, -84.1)
- added C115: 100nF, Capacitor_SMD:C_0805_2012Metric, F.Cu at (56.8, -121.9)
- added C116: 1uF, Capacitor_SMD:C_0805_2012Metric, F.Cu at (56.8, -118.9)
- added C117: 10uF, Capacitor_SMD:C_0805_2012Metric, F.Cu at (56.8, -115.9)
- added C118: 100nF, Capacitor_SMD:C_0805_2012Metric, F.Cu at (56.8, -112.9)
- added C119: 1uF, Capacitor_SMD:C_0805_2012Metric, F.Cu at (56.8, -109.9)
- added C120: 10uF, Capacitor_SMD:C_0805_2012Metric, F.Cu at (56.8, -106.9)
- added C121: 100nF, Capacitor_SMD:C_0805_2012Metric, F.Cu at (61.2, -140.0)
- added C122: 1uF, Capacitor_SMD:C_0805_2012Metric, F.Cu at (61.2, -137.0)
- added C123: 10uF, Capacitor_SMD:C_0805_2012Metric, F.Cu at (61.2, -134.0)
- added C124: 100nF, Capacitor_SMD:C_0805_2012Metric, F.Cu at (61.2, -131.0)
- added C125: 1uF, Capacitor_SMD:C_0805_2012Metric, F.Cu at (61.2, -128.0)
- added C126: 10uF, Capacitor_SMD:C_0805_2012Metric, F.Cu at (61.2, -125.0)
- added C127: 100nF, Capacitor_SMD:C_0805_2012Metric, F.Cu at (61.2, -121.9)
- added C128: 1uF, Capacitor_SMD:C_0805_2012Metric, F.Cu at (94.6, -81.1)
- added C129: 10uF, Capacitor_SMD:C_0805_2012Metric, F.Cu at (124.1, -149.6)
- added C13: C, Capacitor_SMD:C_0805_2012Metric, F.Cu at (43.4, -140.0)
- added C130: 1uF, Capacitor_SMD:C_0805_2012Metric, F.Cu at (61.2, -118.9)
- added C131: 100nF, Capacitor_SMD:C_0805_2012Metric, F.Cu at (61.2, -115.9)
- added C132: 1uF, Capacitor_SMD:C_0805_2012Metric, F.Cu at (61.2, -112.9)
- added C133: 10uF, Capacitor_SMD:C_0805_2012Metric, F.Cu at (61.2, -109.9)
- added C134: 10uF, Capacitor_SMD:C_0805_2012Metric, F.Cu at (61.2, -106.9)
- added C135: 22nF, Capacitor_SMD:C_0805_2012Metric, F.Cu at (65.7, -140.0)
- added C136: DNP, Capacitor_SMD:C_0805_2012Metric, F.Cu at (65.7, -137.0)
- added C137: DNP, Capacitor_SMD:C_0805_2012Metric, F.Cu at (65.7, -134.0)
- added C138: DNP, Capacitor_SMD:C_0805_2012Metric, F.Cu at (65.7, -131.0)
- added C139: DNP, Capacitor_SMD:C_0805_2012Metric, F.Cu at (65.7, -128.0)
- added C14: 100nF, Capacitor_SMD:C_0805_2012Metric, F.Cu at (43.4, -137.0)
- added C140: 10nF, Capacitor_SMD:C_0805_2012Metric, F.Cu at (114.3, -63.8)
- added C141: 100nF, Capacitor_SMD:C_0805_2012Metric, F.Cu at (124.1, -146.6)
- added C15: 2.2uF, Capacitor_SMD:C_0805_2012Metric, F.Cu at (85.7, -73.1)
- added C16: 2.2uF, Capacitor_SMD:C_0805_2012Metric, F.Cu at (85.7, -70.1)
- added C17: 0.1uF, Capacitor_SMD:C_0805_2012Metric, F.Cu at (85.7, -67.1)
- added C18: 2.2uF, Capacitor_SMD:C_0805_2012Metric, F.Cu at (85.7, -64.1)
- added C19: 100nF, Capacitor_SMD:C_0805_2012Metric, F.Cu at (85.7, -61.0)
- added C2: C 360 pF, Capacitor_SMD:C_0805_2012Metric, F.Cu at (39.0, -137.0)
- added C20: 1uF, Capacitor_SMD:C_0805_2012Metric, F.Cu at (85.7, -58.0)
- added C21: 22pF, Capacitor_SMD:C_0805_2012Metric, F.Cu at (43.4, -134.0)
- added C22: 22pF, Capacitor_SMD:C_0805_2012Metric, F.Cu at (43.4, -131.0)
- added C23: DNP, Capacitor_SMD:C_0805_2012Metric, F.Cu at (43.4, -128.0)
- added C24: 10uF, Capacitor_SMD:C_0805_2012Metric, F.Cu at (110.8, -155.7)
- added C25: 10uF, Capacitor_SMD:C_0805_2012Metric, F.Cu at (110.8, -152.6)
- added C26: DNP, Capacitor_SMD:C_0805_2012Metric, F.Cu at (43.4, -125.0)
- added C27: 100nF, Capacitor_SMD:C_0805_2012Metric, F.Cu at (110.8, -149.6)
- added C28: DNP, Capacitor_SMD:C_0805_2012Metric, F.Cu at (43.4, -121.9)
- added C29: DNP, Capacitor_SMD:C_0805_2012Metric, F.Cu at (43.4, -118.9)
- added C3: C 2.0 - 6.0 pF, Capacitor_SMD:C_0805_2012Metric, F.Cu at (39.0, -134.0)
- added C30: 10uF, Capacitor_SMD:C_0805_2012Metric, F.Cu at (110.8, -146.6)
- added C31: 10uF, Capacitor_SMD:C_0805_2012Metric, F.Cu at (110.8, -143.6)
- added C32: 10uF, Capacitor_SMD:C_0805_2012Metric, F.Cu at (110.8, -140.6)
- added C33: 10uF, Capacitor_SMD:C_0805_2012Metric, F.Cu at (85.7, -55.0)
- added C34: 10uF, Capacitor_SMD:C_0805_2012Metric, F.Cu at (90.2, -73.1)
- added C35: 1uF, Capacitor_SMD:C_0805_2012Metric, F.Cu at (90.2, -70.1)
- added C36: 1uF, Capacitor_SMD:C_0805_2012Metric, F.Cu at (90.2, -67.1)
- added C37: 100nF, Capacitor_SMD:C_0805_2012Metric, F.Cu at (90.2, -64.1)
- added C38: 100nF, Capacitor_SMD:C_0805_2012Metric, F.Cu at (90.2, -61.0)
- added C39: 10uF, Capacitor_SMD:C_0805_2012Metric, F.Cu at (90.2, -58.0)
- added C4: C 390 pF, Capacitor_SMD:C_0805_2012Metric, F.Cu at (39.0, -131.0)
- added C40: 10uF, Capacitor_SMD:C_0805_2012Metric, F.Cu at (90.2, -55.0)
- added C41: 1uF, Capacitor_SMD:C_0805_2012Metric, F.Cu at (94.6, -73.1)
- added C42: 1uF, Capacitor_SMD:C_0805_2012Metric, F.Cu at (94.6, -70.1)
- added C43: 100nF, Capacitor_SMD:C_0805_2012Metric, F.Cu at (94.6, -67.1)
- added C44: 100nF, Capacitor_SMD:C_0805_2012Metric, F.Cu at (94.6, -64.1)
- added C45: 10uF, Capacitor_SMD:C_0805_2012Metric, F.Cu at (94.6, -61.0)
- added C46: 100nF, Capacitor_SMD:C_0805_2012Metric, F.Cu at (94.6, -58.0)
- added C47: 1uF, Capacitor_SMD:C_0805_2012Metric, F.Cu at (94.6, -55.0)
- added C48: 10uF, Capacitor_SMD:C_0805_2012Metric, F.Cu at (110.8, -137.6)
- added C49: 100nF, Capacitor_SMD:C_0805_2012Metric, F.Cu at (115.2, -155.7)
- added C5: DNP, Capacitor_SMD:C_0805_2012Metric, F.Cu at (39.0, -128.0)
- added C50: 100nF, Capacitor_SMD:C_0805_2012Metric, F.Cu at (115.2, -152.6)
- added C51: 10uF, Capacitor_SMD:C_0805_2012Metric, F.Cu at (115.2, -149.6)
- added C52: 10uF, Capacitor_SMD:C_0805_2012Metric, F.Cu at (115.2, -146.6)
- added C53: 100nF, Capacitor_SMD:C_0805_2012Metric, F.Cu at (115.2, -143.6)
- added C54: 2.2uF, Capacitor_SMD:C_0805_2012Metric, F.Cu at (99.1, -73.1)
- added C55: 0.1uF, Capacitor_SMD:C_0805_2012Metric, F.Cu at (99.1, -70.1)
- added C56: DNP, Capacitor_SMD:C_0805_2012Metric, F.Cu at (43.4, -115.9)
- added C57: DNP, Capacitor_SMD:C_0805_2012Metric, F.Cu at (43.4, -112.9)
- added C58: DNP, Capacitor_SMD:C_0805_2012Metric, F.Cu at (43.4, -109.9)
- added C59: C 2.0 - 6.0 pF, Capacitor_SMD:C_0805_2012Metric, F.Cu at (43.4, -106.9)
- added C6: C 2.0 - 10.0 pF, Capacitor_SMD:C_0805_2012Metric, F.Cu at (39.0, -125.0)
- added C60: 10uF, Capacitor_SMD:C_0805_2012Metric, F.Cu at (115.2, -140.6)
- added C61: 100nF, Capacitor_SMD:C_0805_2012Metric, F.Cu at (115.2, -137.6)
- added C62: 10uF, Capacitor_SMD:C_0805_2012Metric, F.Cu at (119.7, -155.7)
- added C63: 100nF, Capacitor_SMD:C_0805_2012Metric, F.Cu at (119.7, -152.6)
- added C64: 100nF, Capacitor_SMD:C_0805_2012Metric, F.Cu at (119.7, -149.6)
- added C65: 10uF, Capacitor_SMD:C_0805_2012Metric, F.Cu at (119.7, -146.6)
- added C66: 10uF, Capacitor_SMD:C_0805_2012Metric, F.Cu at (119.7, -143.6)
- added C67: 100nF, Capacitor_SMD:C_0805_2012Metric, F.Cu at (119.7, -140.6)
- added C68: 10uF, Capacitor_SMD:C_0805_2012Metric, F.Cu at (119.7, -137.6)
- added C69: 100nF, Capacitor_SMD:C_0805_2012Metric, F.Cu at (124.1, -155.7)
- added C7: C 2.0 - 10.0 pF, Capacitor_SMD:C_0805_2012Metric, F.Cu at (39.0, -121.9)
- added C70: 10uF, Capacitor_SMD:C_0805_2012Metric, F.Cu at (124.1, -152.6)
- added C71: 10uF, Capacitor_SMD:C_0805_2012Metric, F.Cu at (99.1, -67.1)
- added C72: 100nF, Capacitor_SMD:C_0805_2012Metric, F.Cu at (47.9, -140.0)
- added C73: 1uF, Capacitor_SMD:C_0805_2012Metric, F.Cu at (47.9, -137.0)
- added C74: 10uF, Capacitor_SMD:C_0805_2012Metric, F.Cu at (47.9, -134.0)
- added C75: 100nF, Capacitor_SMD:C_0805_2012Metric, F.Cu at (47.9, -131.0)
- added C76: 1uF, Capacitor_SMD:C_0805_2012Metric, F.Cu at (47.9, -128.0)
- added C77: 10uF, Capacitor_SMD:C_0805_2012Metric, F.Cu at (47.9, -125.0)
- added C78: 100pF, Capacitor_SMD:C_0805_2012Metric, F.Cu at (85.7, -90.1)
- added C79: 100nF, Capacitor_SMD:C_0805_2012Metric, F.Cu at (47.9, -121.9)
- added C8: C 360 pF, Capacitor_SMD:C_0805_2012Metric, F.Cu at (39.0, -118.9)
- added C80: 1uF, Capacitor_SMD:C_0805_2012Metric, F.Cu at (47.9, -118.9)
- added C81: 1uF, Capacitor_SMD:C_0805_2012Metric, F.Cu at (47.9, -115.9)
- added C82: 10uF, Capacitor_SMD:C_0805_2012Metric, F.Cu at (47.9, -112.9)
- added C83: 10uF, Capacitor_SMD:C_0805_2012Metric, F.Cu at (47.9, -109.9)
- added C84: 12pF, Capacitor_SMD:C_0805_2012Metric, F.Cu at (47.9, -106.9)
- added C85: 100nF, Capacitor_SMD:C_0805_2012Metric, F.Cu at (52.3, -140.0)
- added C86: 1uF, Capacitor_SMD:C_0805_2012Metric, F.Cu at (52.3, -137.0)
- added C87: 10uF, Capacitor_SMD:C_0805_2012Metric, F.Cu at (52.3, -134.0)
- added C88: 10uF, Capacitor_SMD:C_0805_2012Metric, F.Cu at (52.3, -131.0)
- added C89: 1uF, Capacitor_SMD:C_0805_2012Metric, F.Cu at (52.3, -128.0)
- added C9: C 390 pF, Capacitor_SMD:C_0805_2012Metric, F.Cu at (39.0, -115.9)
- added C90: 100nF, Capacitor_SMD:C_0805_2012Metric, F.Cu at (52.3, -125.0)
- added C91: 100nF, Capacitor_SMD:C_0805_2012Metric, F.Cu at (52.3, -121.9)
- added C92: 1uF, Capacitor_SMD:C_0805_2012Metric, F.Cu at (52.3, -118.9)
- added C93: 10uF, Capacitor_SMD:C_0805_2012Metric, F.Cu at (52.3, -115.9)
- added C94: 10uF, Capacitor_SMD:C_0805_2012Metric, F.Cu at (52.3, -112.9)
- added C95: 1uF, Capacitor_SMD:C_0805_2012Metric, F.Cu at (52.3, -109.9)
- added C96: 100nF, Capacitor_SMD:C_0805_2012Metric, F.Cu at (52.3, -106.9)
- added C97: 330pF, Capacitor_SMD:C_0805_2012Metric, F.Cu at (85.7, -87.1)
- added C98: 150nF, Capacitor_SMD:C_0805_2012Metric, F.Cu at (85.7, -84.1)
- added C99: 1uF, Capacitor_SMD:C_0805_2012Metric, F.Cu at (85.7, -81.1)
- added D1: BAV199DW, Package_TO_SOT_SMD:SOT-363_SC-70-6, F.Cu at (44.4, -103.4)
- added D10: 1N4001, Diode_THT:D_DO-41_SOD81_P10.16mm_Horizontal, F.Cu at (69.5, -72.5)
- added D11: 1N4001, Diode_THT:D_DO-41_SOD81_P10.16mm_Horizontal, F.Cu at (69.5, -68.3)
- added D12: 1N4001, Diode_THT:D_DO-41_SOD81_P10.16mm_Horizontal, F.Cu at (69.5, -64.0)
- added D13: 1N4001, Diode_THT:D_DO-41_SOD81_P10.16mm_Horizontal, F.Cu at (69.5, -59.8)
- added D14: 1N4001, Diode_THT:D_DO-41_SOD81_P10.16mm_Horizontal, F.Cu at (69.5, -55.5)
- added D15: LED, LED_SMD:LED_0805_2012Metric, F.Cu at (124.0, -125.4)
- added D16: LED, LED_SMD:LED_0805_2012Metric, F.Cu at (124.0, -122.4)
- added D17: LED, LED_SMD:LED_0805_2012Metric, F.Cu at (124.0, -119.4)
- added D18: LED, LED_SMD:LED_0805_2012Metric, F.Cu at (124.0, -116.3)
- added D19: LED, LED_SMD:LED_0805_2012Metric, F.Cu at (124.0, -113.3)
- added D2: BAV199DW, Package_TO_SOT_SMD:SOT-363_SC-70-6, F.Cu at (44.4, -99.5)
- added D3: LED, LED_SMD:LED_0805_2012Metric, F.Cu at (124.0, -134.6)
- added D4: LED, LED_SMD:LED_0805_2012Metric, F.Cu at (124.0, -131.5)
- added D5: LED, LED_SMD:LED_0805_2012Metric, F.Cu at (124.0, -128.5)
- added D6: 1N4001, Diode_THT:D_DO-41_SOD81_P10.16mm_Horizontal, F.Cu at (69.5, -89.5)
- added D7: 1N4001, Diode_THT:D_DO-41_SOD81_P10.16mm_Horizontal, F.Cu at (69.5, -85.3)
- added D8: 1N4001, Diode_THT:D_DO-41_SOD81_P10.16mm_Horizontal, F.Cu at (69.5, -81.0)
- added D9: 1N4001, Diode_THT:D_DO-41_SOD81_P10.16mm_Horizontal, F.Cu at (69.5, -76.8)
- added K3: TQ2-L2-5V, TQ2:RELAY_TQ2_2C_PAN, F.Cu at (53.8, 55.9)
- added K4: TQ2-L2-5V, TQ2:RELAY_TQ2_2C_PAN, F.Cu at (64.4, 83.9)
- added K6: TQ2-L2-5V, TQ2:RELAY_TQ2_2C_PAN, F.Cu at (53.8, 28.9)
- added K7: TQ2-L2-5V, TQ2:RELAY_TQ2_2C_PAN, F.Cu at (86.8, 43.9)
- added R65: 120, Resistor_SMD:R_0805_2012Metric, F.Cu at (110.8, -116.9)
- added R66: 560, Resistor_SMD:R_0805_2012Metric, F.Cu at (115.2, -134.6)
- added R69: 499R, Resistor_SMD:R_0805_2012Metric, F.Cu at (92.1, -140.0)
- added R70: DNP, Resistor_SMD:R_0805_2012Metric, F.Cu at (92.1, -137.1)
- added R71: DNP, Resistor_SMD:R_0805_2012Metric, F.Cu at (92.1, -134.1)
- added R72: DNP, Resistor_SMD:R_0805_2012Metric, F.Cu at (109.9, -61.3)
- added R84: DNP, Resistor_SMD:R_0805_2012Metric, F.Cu at (103.5, -70.2)
- added R85: 10k, Resistor_SMD:R_0805_2012Metric, F.Cu at (38.9, -60.7)
- added R86: 220R, Resistor_SMD:R_0805_2012Metric, F.Cu at (38.9, -57.7)
- added R87: 10k, Resistor_SMD:R_0805_2012Metric, F.Cu at (38.9, -54.8)
- added R88: 220R, Resistor_SMD:R_0805_2012Metric, F.Cu at (43.3, -90.2)
- added R89: 10k, Resistor_SMD:R_0805_2012Metric, F.Cu at (43.3, -87.2)
- added R90: 220R, Resistor_SMD:R_0805_2012Metric, F.Cu at (43.3, -84.3)
- added R91: 10k, Resistor_SMD:R_0805_2012Metric, F.Cu at (43.3, -81.3)
- added R92: 220R, Resistor_SMD:R_0805_2012Metric, F.Cu at (43.3, -78.4)
- added R93: 10k, Resistor_SMD:R_0805_2012Metric, F.Cu at (43.3, -75.4)
- added TP27: TestPoint, Connector_PinHeader_2.54mm:PinHeader_1x01_P2.54mm_Vertical, F.Cu at (99.2, -80.2)
- added Y1: XLL735080.000000I, KiCad:XLL735080000000I, F.Cu at (117.2, -69.9)
- C11: footprint Capacitor_SMD:C_0603_1608Metric_Pad1.08x0.95mm_HandSolder -> Capacitor_SMD:C_0805_2012Metric
- C12: value 12pF -> C; footprint Capacitor_SMD:C_0603_1608Metric_Pad1.08x0.95mm_HandSolder -> Capacitor_SMD:C_0805_2012Metric
- K8: value G2RL-2 -> TQ2-L2-5V; footprint Relay_THT:Relay_DPDT_Omron_G2RL-2 -> TQ2:RELAY_TQ2_2C_PAN
- R1, R10, R11, R119, R120, R121, R122, R123, R124, R125, R126, R127, R128, R129, R130, R131, R132, R133, R134, R135, R136, R137, R138, R139, R14, R140, R141, R142, R143, R144, R145, R146, R147, R148, R149, R15, R150, R151, R152, R153, R154, R155, R156, R157, R158, R162, R163, R164, R165, R166, R167, R168, R169, R17, R170, R171, R172, R173, R174, R175, R176, R177, R178, R179, R180, R181, R188, R189, R190, R191, R192, R198, R199, R2, R200, R28, R29, R3, R30, R31, R32, R35, R37, R38, R39, R4, R40, R41, R42, R43, R44, R47, R48, R49, R5, R50, R51, R53, R55, R56, R57, R58, R67, R68, R73, R74, R75, R77, R78, R79, R8, R80, R81, R82, R94: footprint Resistor_SMD:R_1206_3216Metric -> Resistor_SMD:R_0805_2012Metric
- R100, R101, R96, R98: value 33R -> 10k; footprint Resistor_SMD:R_1206_3216Metric -> Resistor_SMD:R_0805_2012Metric
- R102: value 33R -> 220; footprint Resistor_SMD:R_1206_3216Metric -> Resistor_SMD:R_0805_2012Metric
- R103: value 33R -> 120; footprint Resistor_SMD:R_1206_3216Metric -> Resistor_SMD:R_0805_2012Metric
- R104: value 33R -> 1k2; footprint Resistor_SMD:R_1206_3216Metric -> Resistor_SMD:R_0805_2012Metric
- R105: value 33R -> 800; footprint Resistor_SMD:R_1206_3216Metric -> Resistor_SMD:R_0805_2012Metric
- R106: value 33R -> 600; footprint Resistor_SMD:R_1206_3216Metric -> Resistor_SMD:R_0805_2012Metric
- R107, R108: value 33R -> 300; footprint Resistor_SMD:R_1206_3216Metric -> Resistor_SMD:R_0805_2012Metric
- R12: value R 47k -> 33R; footprint Resistor_SMD:R_1206_3216Metric -> Resistor_SMD:R_0805_2012Metric
- R13: value 33R -> R 9.53 kΩ; footprint Resistor_SMD:R_1206_3216Metric -> Resistor_SMD:R_0805_2012Metric
- R16: value 33 R -> 33R; footprint Resistor_SMD:R_1206_3216Metric -> Resistor_SMD:R_0805_2012Metric
- R18: value 360R -> 33 R; footprint Resistor_SMD:R_1206_3216Metric -> Resistor_SMD:R_0805_2012Metric
- R183: value 470R -> 220R; footprint Resistor_SMD:R_1206_3216Metric -> Resistor_SMD:R_0805_2012Metric
- R19: value 360R -> R; footprint Resistor_SMD:R_1206_3216Metric -> Resistor_SMD:R_0805_2012Metric
- R20, R34: value DNP -> 10k; footprint Resistor_SMD:R_1206_3216Metric -> Resistor_SMD:R_0805_2012Metric
- R21, R22: value 25R -> 499R; footprint Resistor_SMD:R_1206_3216Metric -> Resistor_SMD:R_0805_2012Metric
- R23, R33: value R -> 10k; footprint Resistor_SMD:R_1206_3216Metric -> Resistor_SMD:R_0805_2012Metric
- R24, R25: value 360R -> 499R; footprint Resistor_SMD:R_1206_3216Metric -> Resistor_SMD:R_0805_2012Metric
- R26: value 72 R -> 499R; footprint Resistor_SMD:R_1206_3216Metric -> Resistor_SMD:R_0805_2012Metric
- R27, R6: value 72R -> 499R; footprint Resistor_SMD:R_1206_3216Metric -> Resistor_SMD:R_0805_2012Metric
- R36: value 33 R -> 25R; footprint Resistor_SMD:R_1206_3216Metric -> Resistor_SMD:R_0805_2012Metric
- R45: value 10k -> 33R; footprint Resistor_SMD:R_1206_3216Metric -> Resistor_SMD:R_0805_2012Metric
- R46, R54: value 10k -> DNP; footprint Resistor_SMD:R_1206_3216Metric -> Resistor_SMD:R_0805_2012Metric
- R52: value 560 -> 1k; footprint Resistor_SMD:R_1206_3216Metric -> Resistor_SMD:R_0805_2012Metric
- R59: value 0R -> DNP; footprint Resistor_SMD:R_1206_3216Metric -> Resistor_SMD:R_0805_2012Metric
- R60: value 10k -> 360; footprint Resistor_SMD:R_1206_3216Metric -> Resistor_SMD:R_0805_2012Metric
- R61, R62: value 5K1 -> 1k2; footprint Resistor_SMD:R_1206_3216Metric -> Resistor_SMD:R_0805_2012Metric
- R63: value 10k -> 120; footprint Resistor_SMD:R_1206_3216Metric -> Resistor_SMD:R_0805_2012Metric
- R64: value 0R -> 220R; footprint Resistor_SMD:R_1206_3216Metric -> Resistor_SMD:R_0805_2012Metric
- R7: value 72R -> 25R; footprint Resistor_SMD:R_1206_3216Metric -> Resistor_SMD:R_0805_2012Metric
- R76: value 12K -> 600; footprint Resistor_SMD:R_1206_3216Metric -> Resistor_SMD:R_0805_2012Metric
- R83: value 33R -> DNP; footprint Resistor_SMD:R_1206_3216Metric -> Resistor_SMD:R_0805_2012Metric
- R9: value R 22.2k -> R 9.53 kΩ; footprint Resistor_SMD:R_1206_3216Metric -> Resistor_SMD:R_0805_2012Metric
- R95, R97, R99: value 33R -> 220R; footprint Resistor_SMD:R_1206_3216Metric -> Resistor_SMD:R_0805_2012Metric
- U11, U14: value AD8045ACPZ-R2 -> LM337_SOT223; footprint footprints:CP_8_2_ADI -> Package_TO_SOT_SMD:SOT-223-3_TabPin2
- U2: value LTC6754xSC6 -> AP1117-ADJ; footprint Package_TO_SOT_SMD:SOT-363_SC-70-6 -> Package_TO_SOT_SMD:SOT-223-3_TabPin2
- moved R108 456.9 mm to (119.6, -125.8)
- moved R95 446.3 mm to (43.3, -72.5)
- moved R101 445.4 mm to (92.1, -128.2)
- moved R96 443.6 mm to (43.3, -69.5)
- moved R97 440.9 mm to (43.3, -66.6)
- moved R98 438.3 mm to (43.3, -63.6)
- moved R99 435.6 mm to (43.3, -60.7)
- moved R100 433.0 mm to (43.3, -57.7)
- moved R102 425.5 mm to (115.2, -122.8)
- moved R105 423.9 mm to (119.6, -134.6)
- moved R106 420.6 mm to (119.6, -131.7)
- moved R103 417.2 mm to (115.2, -119.9)
- moved R104 414.0 mm to (115.2, -116.9)
- moved U15 375.9 mm to (93.0, 144.0), turned to 90 degrees
- moved R155 332.1 mm to (56.6, -63.6)
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Connections:
- net DAC1 renamed TRIGGER_THRESHOLD
- C11 pad 1: CH1_CH- -> CH1_CH+
- C11 pad 2: CH1_CH+ -> CH1_CH-
- C12 pad 1: CH2_CH- -> +1V5
- C12 pad 2: CH2_CH+ -> GND
- R1 pad 2: Net-(K8-Pad21) -> Net-(K6-Pad3)
- R100 pad 1: /adc/D_ADC_A5 -> Net-(Q13-G)
- R100 pad 2: ADC_A_5 -> GND
- R101 pad 1: /adc/D_ADC_A6 -> unconnected-(R101-Pad1)
- R101 pad 2: ADC_A_6 -> unconnected-(R101-Pad2)
- R102 pad 1: /adc/D_ADC_A7 -> GND
- R102 pad 2: ADC_A_7 -> Net-(U11-ADJ)
- R103 pad 1: /adc/D_ADC_A8 -> Net-(U11-ADJ)
- R103 pad 2: ADC_A_8 -> -3V5
- R104 pad 1: /adc/D_ADC_A9 -> Net-(D15-K)
- R104 pad 2: ADC_A_9 -> GND
- R105 pad 1: /adc/D_ADC_A10 -> Net-(D16-K)
- R105 pad 2: ADC_A_10 -> GND
- R106 pad 1: /adc/D_ADC_A11 -> Net-(D17-K)
- R106 pad 2: ADC_A_11 -> -5V
- R107 pad 1: /adc/D_ADC_B0 -> Net-(D18-K)
- R107 pad 2: ADC_B_0 -> GND
- R108 pad 1: /adc/D_ADC_B1 -> Net-(D19-K)
- R108 pad 2: ADC_B_1 -> -3V5
- R12 pad 1: Net-(C5-Pad2) -> Net-(J2-In)
- R12 pad 2: GND -> Net-(K3-Pad3)
- R13 pad 1: Net-(J2-In) -> Net-(C5-Pad2)
- R13 pad 2: Net-(K9-Pad21) -> GND
- R16 pad 1: Net-(K9-Pad11) -> Net-(K3-Pad8)
- R18 pad 1: Net-(R18-Pad1) -> Net-(U3-VOUT)
- R18 pad 2: Net-(U3-VOUT) -> GND
- R188 pad 1: Net-(Q1-S) -> Net-(Q1-G)
- R19 pad 2: Net-(R19-Pad2) -> GND
- R2 pad 1: Net-(K8-Pad11) -> Net-(K6-Pad8)
- R20 pad 1: AN_TRIGGER_N -> AN_TRIGGER_P
- R20 pad 2: Net-(U2--) -> Net-(U17-+IN)
- R200 pad 1: CH1_VGA -> Net-(U5-INPP)
- R21 pad 1: CH2_CH- -> Net-(U4-+IN)
- R21 pad 2: Net-(R21-Pad2) -> Net-(U3-VOUT)
- R22 pad 1: CH2_CH+ -> Net-(U4--IN)
- R22 pad 2: Net-(R22-Pad2) -> Net-(R19-Pad1)
- R23 pad 1: Net-(U2-+) -> Net-(U17--IN)
- R24 pad 1: Net-(R24-Pad1) -> Net-(U6-+OUT)
- R24 pad 2: Net-(R24-Pad2) -> Net-(U6-+IN)
- R25 pad 1: Net-(R25-Pad1) -> Net-(U6--OUT)
- R25 pad 2: Net-(U5-VOUT) -> Net-(U6--IN)
- R26 pad 1: Net-(R21-Pad2) -> Net-(U4-+OUT)
- R26 pad 2: Net-(R18-Pad1) -> Net-(U4-+IN)
- R27 pad 1: Net-(R22-Pad2) -> Net-(U4--OUT)
- R27 pad 2: Net-(R19-Pad1) -> Net-(U4--IN)
- R32 pad 1: AN_TRIGGER_CH2 -> CH2_CH+
- R32 pad 2: Net-(U3-VOUT) -> Net-(U4-+OUT)
- R33 pad 1: Net-(U2--) -> Net-(U17-+IN)
- R33 pad 2: Net-(K2-Pad11) -> Net-(C135-Pad2)
- R34 pad 1: AN_TRIGGER_P -> AN_TRIGGER_N
- R34 pad 2: Net-(U2-+) -> Net-(U17--IN)
- R35 pad 1: Net-(R24-Pad2) -> Net-(R35-Pad1)
- R36 pad 1: Net-(R19-Pad2) -> CH2_CH-
- R36 pad 2: GND -> Net-(U4--OUT)
- R37 pad 1: Net-(U1-NEG) -> Net-(U1-OUTPUT)
- R37 pad 2: Net-(U14-+IN) -> Net-(U5-INPP)
- R38 pad 1: GND -> Net-(U8-OUTPUT)
- R38 pad 2: Net-(U14-+IN) -> Net-(U8-NEG)
- R39 pad 1: Net-(U14-+IN) -> Net-(U1-NEG)
- R4 pad 1: CH1_CH+ -> CH1_CH-
- R4 pad 2: Net-(R4-Pad2) -> Net-(U6--OUT)
- R41 pad 1: Net-(U8-NEG) -> Net-(U8-OUTPUT)
- R41 pad 2: Net-(U11-+IN) -> Net-(U3-INPP)
- R44 pad 1: CH2_VGA -> Net-(U3-INPP)
- R45 pad 1: GND -> Net-(U1-NEG)
- R45 pad 2: Net-(U14--IN) -> Net-(U1-OUTPUT)
- R46 pad 1: Net-(U14--IN) -> Net-(U7-OUT6)
- R46 pad 2: CH1_VGA -> unconnected-(R46-Pad2)
- R5 pad 1: CH1_CH- -> CH1_CH+
- R5 pad 2: Net-(R5-Pad2) -> Net-(U6-+OUT)
- R53 pad 1: Net-(U11-+IN) -> Net-(U8-NEG)
- R54 pad 1: GND -> Net-(U7-OUT5)
- R54 pad 2: Net-(U11-+IN) -> unconnected-(R54-Pad2)
- R59 pad 1: Net-(U14-FEEDBACK) -> Net-(U7-OUT7)
- R59 pad 2: CH1_VGA -> unconnected-(R59-Pad2)
- R6 pad 1: Net-(R5-Pad2) -> Net-(U6-+IN)
- R6 pad 2: Net-(R25-Pad1) -> Net-(U5-VOUT)
- R60 pad 2: Net-(U11--IN) -> Net-(U14-ADJ)
- R61 pad 2: -5V -> -8V
- R63 pad 1: Net-(U11--IN) -> Net-(U14-ADJ)
- R63 pad 2: CH2_VGA -> -5V
- R64 pad 1: Net-(U11-FEEDBACK) -> Net-(Q6-G)
- R64 pad 2: CH2_VGA -> TRIGG_2_MCU
- R7 pad 1: Net-(R4-Pad2) -> AN_TRIGGER_CH2
- R7 pad 2: Net-(R24-Pad1) -> Net-(U3-VOUT)
- R83 pad 1: /adc/D_ADC_A12 -> CLK_FPGA_PLL_50MHz
- R83 pad 2: ADC_A_12 -> CLOCK_80MHz
- R94 pad 2: TRIGGER_LEVEL -> EXT_TRIGGER_LEVEL
- R95 pad 1: /adc/D_ADC_A0 -> Net-(Q11-G)
- R95 pad 2: ADC_A_0 -> CH2_ATTEN_B_MCU
- R96 pad 1: /adc/D_ADC_A1 -> Net-(Q11-G)
- R96 pad 2: ADC_A_1 -> GND
- R97 pad 1: /adc/D_ADC_A2 -> Net-(Q12-G)
- R97 pad 2: ADC_A_2 -> AC_DC_CH1_MCU
- R98 pad 1: /adc/D_ADC_A3 -> Net-(Q12-G)
- R98 pad 2: ADC_A_3 -> GND
- R99 pad 1: /adc/D_ADC_A4 -> Net-(Q13-G)
- R99 pad 2: ADC_A_4 -> AC_DC_CH2_MCU
- TP1 pad 1: Net-(K8-Pad21) -> Net-(K6-Pad3)
- TP13 pad 1: Net-(U11-+IN) -> Net-(U3-INPP)
- TP14 pad 1: CH2_VGA -> Net-(U7-OUT6)
- TP15 pad 1: Net-(K2-Pad11) -> Net-(C135-Pad2)
- TP17 pad 1: AN_TRIGGER_P -> AN_TRIGGER_N
- TP18 pad 1: AN_TRIGGER_N -> AN_TRIGGER_P
- TP2 pad 1: Net-(K8-Pad11) -> Net-(C1-Pad1)
- TP23 pad 1: Net-(R21-Pad2) -> Net-(U4-+OUT)
- TP24 pad 1: Net-(R22-Pad2) -> Net-(U4--OUT)
- TP25 pad 1: Net-(R5-Pad2) -> Net-(U6-+OUT)
- TP26 pad 1: Net-(R4-Pad2) -> Net-(U6--OUT)
- TP4 pad 1: Net-(U14-+IN) -> Net-(U5-INPP)
- TP6 pad 1: CH1_VGA -> Net-(U7-OUT5)
- TP7 pad 1: Net-(K9-Pad21) -> Net-(K3-Pad3)
- TP8 pad 1: Net-(K9-Pad11) -> Net-(C10-Pad1)
- U1 pad 6: Net-(U1-NEG) -> Net-(U1-OUTPUT)
- U10 pad JP2_1: ADC_B_0 -> CLOCK_80MHz
- U10 pad JP2_13: ADC_B_5 -> ADC_B_3
- U10 pad JP2_15: ADC_B_6 -> ADC_B_4
- U10 pad JP2_17: ADC_B_7 -> ADC_B_5
- U10 pad JP2_19: ADC_B_8 -> ADC_B_6
- U10 pad JP2_21: ADC_B_9 -> ADC_B_7
- U10 pad JP2_23: ADC_B_10 -> ADC_B_8
- U10 pad JP2_25: ADC_B_11 -> ADC_B_9
- U10 pad JP2_27: ADC_B_12 -> ADC_B_10
- U10 pad JP2_3: ADC_B_1 -> unconnected-(U10B-GPIO_1_IN1-PadJP2_3)
- U10 pad JP2_31: ADC_B_13 -> ADC_B_11
- U10 pad JP2_33: unconnected-(U10B-GPIO_126-PadJP2_33) -> ADC_B_10
- U10 pad JP2_35: unconnected-(U10B-GPIO_128-PadJP2_35) -> ADC_B_11
- U10 pad JP2_5: ADC_B_2 -> ADC_B_0
- U10 pad JP2_7: ADC_B_3 -> ADC_B_1
- U10 pad JP2_9: ADC_B_4 -> ADC_B_2
- U11 pad 1: unconnected-(U11-NC-Pad1) -> Net-(U11-ADJ)
- U11 pad 2: Net-(U11-FEEDBACK) -> Net-(U11-VI)
- U11 pad 3: Net-(U11--IN) -> -3V5
- U14 pad 1: unconnected-(U14-NC-Pad1) -> Net-(U14-ADJ)
- U14 pad 2: Net-(U14-FEEDBACK) -> Net-(U14-VI)
- U14 pad 3: Net-(U14--IN) -> -5V
- U2 pad 1: AN_TRIGGER_P -> Net-(U2-ADJ)
- U2 pad 2: GND -> +5V
- U2 pad 3: Net-(U2-+) -> Net-(U2-VI)
- U21 pad 24: /adc/D_ADC_B0 -> ADC_B_0
- U21 pad 25: /adc/D_ADC_B1 -> ADC_B_1
- U21 pad 26: /adc/D_ADC_B2 -> ADC_B_2
- U21 pad 27: /adc/D_ADC_B3 -> ADC_B_3
- U21 pad 28: /adc/D_ADC_B4 -> ADC_B_4
- U21 pad 29: /adc/D_ADC_B5 -> ADC_B_5
- U21 pad 30: /adc/D_ADC_B6 -> ADC_B_6
- U21 pad 33: /adc/D_ADC_B7 -> ADC_B_7
- U21 pad 34: /adc/D_ADC_B8 -> ADC_B_8
- U21 pad 35: /adc/D_ADC_B9 -> ADC_B_9
- U21 pad 36: /adc/D_ADC_B10 -> ADC_B_10
- U21 pad 37: /adc/D_ADC_B11 -> ADC_B_11
- U21 pad 41: /adc/D_ADC_A0 -> ADC_A_0
- U21 pad 42: /adc/D_ADC_A1 -> ADC_A_1
- U21 pad 43: /adc/D_ADC_A2 -> ADC_A_2
- U21 pad 44: /adc/D_ADC_A3 -> ADC_A_3
- U21 pad 45: /adc/D_ADC_A4 -> ADC_A_4
- U21 pad 46: /adc/D_ADC_A5 -> ADC_A_5
- U21 pad 47: /adc/D_ADC_A6 -> ADC_A_6
- U21 pad 48: /adc/D_ADC_A7 -> ADC_A_7
- U21 pad 51: /adc/D_ADC_A8 -> ADC_A_8
- U21 pad 52: /adc/D_ADC_A9 -> ADC_A_9
- U21 pad 53: /adc/D_ADC_A10 -> ADC_A_10
- U21 pad 54: /adc/D_ADC_A11 -> ADC_A_11
- U21 pad 55: /adc/D_ADC_A12 -> ADC_A_12
- U21 pad 56: /adc/D_ADC_A13 -> ADC_A_13
- U21 pad 8: CLK_FPGA_PLL_50MHz -> CLOCK_80MHz
- U21 pad 9: CLK_FPGA_PLL_50MHz -> CLOCK_80MHz
- U3 pad 3: CH2_VGA -> Net-(U3-INPP)
- U5 pad 3: CH1_VGA -> Net-(U5-INPP)
- U8 pad 6: Net-(U8-NEG) -> Net-(U8-OUTPUT)
- U9 pad CN7_11: unconnected-(U9E-D21/I2S_B_MCK-PadCN7_11) -> AC_DC_CH2_MCU
- U9 pad CN7_13: unconnected-(U9E-D22/I2S_B_SD/SPI_B_MOSI-PadCN7_13) -> CH1_ATTEN_B_MCU
- U9 pad CN7_15: unconnected-(U9E-D23/I2S_B_CK/SPI_B_SCK-PadCN7_15) -> CH2_ATTEN_A_MCU
- U9 pad CN7_17: Net-(U9E-D24/SPI_B_NSS) -> CH2_ATTEN_B_MCU
- U9 pad CN7_19: unconnected-(U9E-D25/SPI_B_MISO-PadCN7_19) -> AC_DC_CH1_MCU
- U9 pad CN9_13: CH2_ATTEN_MCU -> TRIGGER_AC_DC_MCU
- U9 pad CN9_17: unconnected-(U9D-D70/I2C_B_SMBA-PadCN9_17) -> DAC_ALM
- U9 pad CN9_19: unconnected-(U9D-D69/I2C_B_SCL-PadCN9_19) -> DAC_TEMP
- U9 pad CN9_24: unconnected-(U9D-D61/SAI_B_SCK-PadCN9_24) -> DAC_RST
- U9 pad CN9_26: AD_DC_MCU -> CH1_ATTEN_A_MCU
- U9 pad CN9_28: unconnected-(U9D-D63/SAI_B_FS-PadCN9_28) -> DAC_CLR
Other:
- board size 160 x 149.3 mm -> 159 x 149.3 mm
