File: DigitalOsciloscope.kicad_pcb (KiCad board)
At the start: 2 copper layers, 159 x 149.3 mm, 385 parts, among them J1 Conn_Coaxial, J2 Conn_Coaxial, J7 Conn_Coaxial, K3 TQ2-L2-5V, K4 TQ2-L2-5V, K6 TQ2-L2-5V, K7 TQ2-L2-5V, K8 TQ2-L2-5V, U1 OPA656U, U10 P0082_BOTTOMMOUNT, U11 LM337_SOT223, U14 LM337_SOT223, U15 AP1117-ADJ, U18 AP1117-ADJ, U2 AP1117-ADJ, U21 LTC2299xUP, U3 AD8337BCPZ-REEL-ND, U5 AD8337BCPZ-REEL-ND, U8 OPA656U, U9 NUCLEOH723ZG, Y1 XLL735080.000000I

Commit message: Remove the stage between DAC and FET buffer
Parts:
- removed C1, C10, C135: 22nF, Capacitor_SMD:C_0805_2012Metric
- removed C100, C109, C111, C114, C17, C55: 0.1uF, Capacitor_SMD:C_0805_2012Metric
- removed C101, C110, C113, C78: 100pF, Capacitor_SMD:C_0805_2012Metric
- removed C102, C104, C107, C112, C116, C119, C122, C125, C128, C130, C132, C20, C35, C36, C41, C42, C47, C73, C76, C80, C81, C86, C89, C92, C95, C99: 1uF, Capacitor_SMD:C_0805_2012Metric
- removed C103, C106, C115, C118, C121, C124, C127, C131, C14, C141, C19, C27, C37, C38, C43, C44, C46, C49, C50, C53, C61, C63, C64, C67, C69, C72, C75, C79, C85, C90, C91, C96: 100nF, Capacitor_SMD:C_0805_2012Metric
- removed C105, C108, C117, C120, C123, C126, C129, C133, C134, C24, C25, C30, C31, C32, C33, C34, C39, C40, C45, C48, C51, C52, C60, C62, C65, C66, C68, C70, C71, C74, C77, C82, C83, C87, C88, C93, C94: 10uF, Capacitor_SMD:C_0805_2012Metric
- removed C11, C84: 12pF, Capacitor_SMD:C_0805_2012Metric
- removed C12, C13: C, Capacitor_SMD:C_0805_2012Metric
- removed C136, C137, C138, C139, C23, C26, C28, C29, C5, C56, C57, C58: DNP, Capacitor_SMD:C_0805_2012Metric
- removed C140: 10nF, Capacitor_SMD:C_0805_2012Metric
- removed C15, C16, C18, C54: 2.2uF, Capacitor_SMD:C_0805_2012Metric
- removed C2, C8: C 360 pF, Capacitor_SMD:C_0805_2012Metric
- removed C21, C22: 22pF, Capacitor_SMD:C_0805_2012Metric
- removed C3, C59: C 2.0 - 6.0 pF, Capacitor_SMD:C_0805_2012Metric
- removed C4, C9: C 390 pF, Capacitor_SMD:C_0805_2012Metric
- removed C6, C7: C 2.0 - 10.0 pF, Capacitor_SMD:C_0805_2012Metric
- removed C97: 330pF, Capacitor_SMD:C_0805_2012Metric
- removed C98: 150nF, Capacitor_SMD:C_0805_2012Metric
- removed D1: BAV199DW, Package_TO_SOT_SMD:SOT-363_SC-70-6
- removed D11, D12, D13, D14: 1N4001, Diode_THT:D_DO-41_SOD81_P10.16mm_Horizontal
- removed D15, D16, D17, D18, D19, D3, D4, D5: LED, LED_SMD:LED_0805_2012Metric
- removed K3, K4, K6, K7: TQ2-L2-5V, TQ2:RELAY_TQ2_2C_PAN
- removed R1, R12, R120, R121, R122, R124, R125, R126, R127, R141, R142, R143, R144, R145, R146, R148, R149, R150, R152, R157, R158, R16, R166, R167, R168, R169, R170, R171, R180, R181, R2, R37, R41, R45, R73, R75, R77, R78, R79, R80, R81, R82, R94: 33R, Resistor_SMD:R_0805_2012Metric
- removed R10, R14: R 49.9k, Resistor_SMD:R_0805_2012Metric
- removed R11, R15, R3, R8: R 953k, Resistor_SMD:R_0805_2012Metric
- removed R119, R123, R128, R129, R130, R131, R132, R133, R134, R135, R136, R137, R138, R139, R140, R147, R151, R153, R154, R155, R156, R162, R163, R164, R165, R172, R173, R174, R175, R176, R177, R178, R179, R189, R190, R191, R192, R74: 10kR, Resistor_SMD:R_0805_2012Metric
- removed R13, R9: R 9.53 kΩ, Resistor_SMD:R_0805_2012Metric
- removed R17, R199, R32, R36, R4, R43, R5, R7: 25R, Resistor_SMD:R_0805_2012Metric
- removed R18, R198: 33 R, Resistor_SMD:R_0805_2012Metric
- removed R183, R64, R86, R88, R90, R92: 220R, Resistor_SMD:R_0805_2012Metric
- removed R188, R20, R23, R33, R34, R38, R39, R53, R85, R87, R89, R91, R93: 10k, Resistor_SMD:R_0805_2012Metric
- removed R19, R35: R, Resistor_SMD:R_0805_2012Metric
- removed R200, R44: 49.9 R, Resistor_SMD:R_0805_2012Metric
- removed R21, R22, R24, R25, R26, R27, R6, R69: 499R, Resistor_SMD:R_0805_2012Metric
- removed R28, R29, R30, R31: 100 R, Resistor_SMD:R_0805_2012Metric
- removed R40, R47, R48, R51: 16k, Resistor_SMD:R_0805_2012Metric
- removed R42, R49: 8k, Resistor_SMD:R_0805_2012Metric
- removed R46, R54, R56, R58, R59, R70, R71, R72, R83, R84: DNP, Resistor_SMD:R_0805_2012Metric
- removed R50, R63, R65, R67: 120, Resistor_SMD:R_0805_2012Metric
- removed R52: 1k, Resistor_SMD:R_0805_2012Metric
- removed R55, R57: 0R, Resistor_SMD:R_0805_2012Metric
- removed R60: 360, Resistor_SMD:R_0805_2012Metric
- removed R61, R62: 1k2, Resistor_SMD:R_0805_2012Metric
- removed R66: 560, Resistor_SMD:R_0805_2012Metric
- removed R68: 200, Resistor_SMD:R_0805_2012Metric
- removed R76: 600, Resistor_SMD:R_0805_2012Metric
- removed TP1, TP10, TP11, TP12, TP13, TP14, TP15, TP16, TP17, TP18, TP19, TP2, TP20, TP21, TP22, TP23, TP24, TP25, TP26, TP27, TP3, TP4, TP5, TP6, TP7, TP8, TP9: TestPoint, Connector_PinHeader_2.54mm:PinHeader_1x01_P2.54mm_Vertical
- removed U15, U18: AP1117-ADJ, Package_TO_SOT_SMD:SOT-223-3_TabPin2
- removed U3, U5: AD8337BCPZ-REEL-ND, footprints:CP_8_2_ADI
- removed Y1: XLL735080.000000I, KiCad:XLL735080000000I
- added K10: G2RL-2, Relay_THT:Relay_DPDT_Omron_G2RL-2, F.Cu at (202.6, -76.1)
- added K9: G2RL-2, Relay_THT:Relay_DPDT_Omron_G2RL-2, F.Cu at (264.5, -39.0)
- added Q1: 2N7002, Package_TO_SOT_SMD:SOT-23, F.Cu at (211.0, -120.6)
- added Q2: DMP3099L, Package_TO_SOT_SMD:SOT-23, F.Cu at (211.0, -116.0)
- added Q3: DMP3099L, Package_TO_SOT_SMD:SOT-23, F.Cu at (211.0, -111.3)
- added R109: 33R, Resistor_SMD:R_0805_2012Metric, F.Cu at (125.5, 104.4)
- added R110: 33R, Resistor_SMD:R_0805_2012Metric, F.Cu at (125.5, 103.0)
- added R111: 33R, Resistor_SMD:R_0805_2012Metric, F.Cu at (125.5, 101.6)
- added R112: 33R, Resistor_SMD:R_0805_2012Metric, F.Cu at (125.5, 100.2)
- added R113: 33R, Resistor_SMD:R_0805_2012Metric, F.Cu at (125.5, 98.8)
- added R114: 33R, Resistor_SMD:R_0805_2012Metric, F.Cu at (125.5, 97.4)
- added R115: 33R, Resistor_SMD:R_0805_2012Metric, F.Cu at (125.2, 92.0)
- added R116: 33R, Resistor_SMD:R_0805_2012Metric, F.Cu at (125.2, 90.5)
- added R117: 33R, Resistor_SMD:R_0805_2012Metric, F.Cu at (125.2, 89.2)
- added R118: 33R, Resistor_SMD:R_0805_2012Metric, F.Cu at (125.2, 88.0)
- added TR1: Wuerth_749013011A, Transformer_SMD:Transformer_Ethernet_Wuerth_749013011A, F.Cu at (79.0, 179.0)
- added U12: SN75160BDW, Package_SO:SOIC-20W_7.5x12.8mm_P1.27mm, F.Cu at (86.7, 108.3)
- added U13: SN75160BDW, Package_SO:SOIC-20W_7.5x12.8mm_P1.27mm, F.Cu at (86.8, 157.2)
- added U16: DAC80504, Package_DFN_QFN:Texas_RTE0016D_WQFN-16-1EP_3x3mm_P0.5mm_EP0.8x0.8mm_ThermalVias, F.Cu at (74.6, -79.5)
- added U17: CYPD3177-24LQ, Package_DFN_QFN:QFN-24-1EP_4x4mm_P0.5mm_EP2.75x2.75mm, F.Cu at (108.7, -78.5)
- added U19: LM2596S-ADJ, Package_TO_SOT_SMD:TO-263-5_TabPin3, F.Cu at (201.5, -116.8)
- added U20: INA180A3, Package_TO_SOT_SMD:SOT-23-5, F.Cu at (193.4, -83.5)
- added U22: LM2596S-5, Package_TO_SOT_SMD:TO-263-5_TabPin3, F.Cu at (201.5, -92.1)
- added U23: AP1117-ADJ, Package_TO_SOT_SMD:SOT-223-3_TabPin2, F.Cu at (220.3, -118.8)
- added U24: AP1117-ADJ, Package_TO_SOT_SMD:SOT-223-3_TabPin2, F.Cu at (220.3, -110.5)
- added U25: AP1117-ADJ, Package_TO_SOT_SMD:SOT-223-3_TabPin2, F.Cu at (220.3, -102.2)
- added U26: AP1117-ADJ, Package_TO_SOT_SMD:SOT-223-3_TabPin2, F.Cu at (220.3, -93.8)
- added U27: AP1117-ADJ, Package_TO_SOT_SMD:SOT-223-3_TabPin2, F.Cu at (220.3, -85.5)
- added U28: STM32H723ZGIx, Package_BGA:UFBGA-144_7x7mm_Layout12x12_P0.5mm, F.Cu at (77.9, 191.2)
- added U29: LAN8742A, Package_DFN_QFN:VQFN-24-1EP_4x4mm_P0.5mm_EP2.5x2.5mm_ThermalVias, F.Cu at (76.0, 199.3)
- added U4: LMH6551MA, Package_SO:SOIC-8_3.9x4.9mm_P1.27mm, F.Cu at (44.1, -78.8)
- added U6: LTC2299xUP, Package_DFN_QFN:QFN-64-1EP_9x9mm_P0.5mm_EP7.15x7.15mm, F.Cu at (112.0, 77.6)
- added U7: LMH6551MA, Package_SO:SOIC-8_3.9x4.9mm_P1.27mm, F.Cu at (44.1, -72.2)
- D10, D6, D7: value 1N4001 -> 1N5822; footprint Diode_THT:D_DO-41_SOD81_P10.16mm_Horizontal -> Diode_THT:D_DO-201AD_P15.24mm_Horizontal
- D2: value BAV199DW -> 1N5822; footprint Package_TO_SOT_SMD:SOT-363_SC-70-6 -> Diode_THT:D_DO-201AD_P15.24mm_Horizontal
- D8, D9: value 1N4001 -> 1N5400; footprint Diode_THT:D_DO-41_SOD81_P10.16mm_Horizontal -> Diode_THT:D_DO-201AD_P15.24mm_Horizontal
- K8: value TQ2-L2-5V -> G2RL-2; footprint TQ2:RELAY_TQ2_2C_PAN -> Relay_THT:Relay_DPDT_Omron_G2RL-2
- R100, R101, R96, R98: value 10k -> 33R
- R102: value 220 -> 33R
- R103: value 120 -> 33R
- R104: value 1k2 -> 33R
- R105: value 800 -> 33R
- R106: value 600 -> 33R
- R107, R108: value 300 -> 33R
- R95, R97, R99: value 220R -> 33R
- U11, U14: value LM337_SOT223 -> SN75160BDW; footprint Package_TO_SOT_SMD:SOT-223-3_TabPin2 -> Package_SO:SOIC-20W_7.5x12.8mm_P1.27mm
- U2: value AP1117-ADJ -> LTC6754xSC6; footprint Package_TO_SOT_SMD:SOT-223-3_TabPin2 -> Package_TO_SOT_SMD:SOT-363_SC-70-6
- U21: value LTC2299xUP -> LM2596S-5; footprint Package_DFN_QFN:QFN-64-1EP_9x9mm_P0.5mm_EP7.15x7.15mm -> Package_TO_SOT_SMD:TO-263-5_TabPin3
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Connections:
- D10 pad 1: +5V_EXT -> Net-(D10-K)
- D10 pad 2: CH1_ATTEN_B -> +15V
- D2 pad 1: -5V -> Net-(D2-K)
- D2 pad 2: +5V -> GND
- D6 pad 1: +5V_EXT -> Net-(D6-K)
- D6 pad 2: TRIGG_1 -> +15V
- D7 pad 1: +5V_EXT -> Net-(D7-K)
- D7 pad 2: TRIGG_2 -> -5V
- D8 pad 1: +5V_EXT -> Net-(D8-K)
- D8 pad 2: TRIGGER_AC_DC -> -5V
- D9 pad 1: +5V_EXT -> +15V
- D9 pad 2: CH1_ATTEN_A -> Net-(D9-A)
- R100 pad 1: Net-(Q13-G) -> Net-(U11-B6)
- R100 pad 2: GND -> ADC_A_5
- R101 pad 1: unconnected-(R101-Pad1) -> Net-(U11-B7)
- R101 pad 2: unconnected-(R101-Pad2) -> ADC_A_6
- R102 pad 1: GND -> Net-(U11-B8)
- R102 pad 2: Net-(U11-ADJ) -> ADC_A_7
- R103 pad 1: Net-(U11-ADJ) -> Net-(U12-B1)
- R103 pad 2: -3V5 -> ADC_A_8
- R104 pad 2: GND -> ADC_A_9
- R105 pad 2: GND -> ADC_A_10
- R106 pad 2: -5V -> ADC_A_11
- R107 pad 2: GND -> ADC_B_0
- R108 pad 2: -3V5 -> ADC_B_1
- R95 pad 1: Net-(Q11-G) -> Net-(U11-B1)
- R95 pad 2: CH2_ATTEN_B_MCU -> ADC_A_0
- R96 pad 1: Net-(Q11-G) -> Net-(U11-B2)
- R96 pad 2: GND -> ADC_A_1
- R97 pad 1: Net-(Q12-G) -> Net-(U11-B3)
- R97 pad 2: AC_DC_CH1_MCU -> ADC_A_2
- R98 pad 1: Net-(Q12-G) -> Net-(U11-B4)
- R98 pad 2: GND -> ADC_A_3
- R99 pad 1: Net-(Q13-G) -> Net-(U11-B5)
- R99 pad 2: AC_DC_CH2_MCU -> ADC_A_4
- U1 pad 4: Net-(U1--VS) -> -5V
- U1 pad 6: Net-(U1-OUTPUT) -> Net-(U1-NEG)
- U1 pad 7: Net-(U1-+VS) -> +5V
- U10 pad JP1_10: GPIO_23 -> unconnected-(U10A-GPIO_07-PadJP1_10)
- U10 pad JP1_11: Net-(U10A-GPIO-0_VCC_SYS) -> unconnected-(U10A-GPIO-0_VCC_SYS-PadJP1_11)
- U10 pad JP1_12: GND -> Net-(U10A-GPIO-0_GND-PadJP1_12)
- U10 pad JP1_13: OE_A -> unconnected-(U10A-GPIO_08-PadJP1_13)
- U10 pad JP1_15: OE_B -> unconnected-(U10A-GPIO_010-PadJP1_15)
- U10 pad JP1_17: GPIO_6 -> unconnected-(U10A-GPIO_012-PadJP1_17)
- U10 pad JP1_18: QSPI_CS/GPIO_0 -> unconnected-(U10A-GPIO_013-PadJP1_18)
- U10 pad JP1_19: GPIO_7 -> unconnected-(U10A-GPIO_014-PadJP1_19)
- U10 pad JP1_20: QSPI_CLK/GPIO_1 -> unconnected-(U10A-GPIO_015-PadJP1_20)
- U10 pad JP1_21: GPIO_8 -> unconnected-(U10A-GPIO_016-PadJP1_21)
- U10 pad JP1_22: QSPI_IO0/GPIO_2 -> unconnected-(U10A-GPIO_017-PadJP1_22)
- U10 pad JP1_23: GPIO_9 -> unconnected-(U10A-GPIO_018-PadJP1_23)
- U10 pad JP1_24: QSPI_IO1/GPIO_3 -> unconnected-(U10A-GPIO_019-PadJP1_24)
- U10 pad JP1_25: GPIO_10 -> unconnected-(U10A-GPIO_020-PadJP1_25)
- U10 pad JP1_26: QSPI_IO2/GPIO_4 -> unconnected-(U10A-GPIO_021-PadJP1_26)
- U10 pad JP1_27: GPIO_11 -> unconnected-(U10A-GPIO_022-PadJP1_27)
- U10 pad JP1_28: QSPI_IO3/GPIO_5 -> unconnected-(U10A-GPIO_023-PadJP1_28)
- U10 pad JP1_29: Net-(U10A-GPIO-0_VCC3P3) -> unconnected-(U10A-GPIO-0_VCC3P3-PadJP1_29)
- U10 pad JP1_30: GND -> Net-(U10A-GPIO-0_GND-PadJP1_12)
- U10 pad JP1_31: Net-(U10A-GPIO_024) -> unconnected-(U10A-GPIO_024-PadJP1_31)
- U10 pad JP1_33: Net-(U10A-GPIO_026) -> unconnected-(U10A-GPIO_026-PadJP1_33)
- U10 pad JP1_4: GPIO_20 -> unconnected-(U10A-GPIO_01-PadJP1_4)
- U10 pad JP1_5: CLIPPING -> unconnected-(U10A-GPIO_02-PadJP1_5)
- U10 pad JP1_6: GPIO_21 -> unconnected-(U10A-GPIO_03-PadJP1_6)
- U10 pad JP1_7: USART_1_RX -> unconnected-(U10A-GPIO_04-PadJP1_7)
- U10 pad JP1_8: GPIO_22 -> unconnected-(U10A-GPIO_05-PadJP1_8)
- U10 pad JP1_9: USART_1_TX -> unconnected-(U10A-GPIO_06-PadJP1_9)
- U10 pad JP2_1: CLOCK_80MHz -> ADC_B_0
- U10 pad JP2_11: Net-(U10B-GPIO-1_VCC_SYS) -> unconnected-(U10B-GPIO-1_VCC_SYS-PadJP2_11)
- U10 pad JP2_12: GND -> Net-(U10B-GPIO-1_GND-PadJP2_12)
- U10 pad JP2_13: ADC_B_3 -> ADC_B_5
- U10 pad JP2_15: ADC_B_4 -> ADC_B_6
- U10 pad JP2_17: ADC_B_5 -> ADC_B_7
- U10 pad JP2_19: ADC_B_6 -> ADC_B_8
- U10 pad JP2_21: ADC_B_7 -> ADC_B_9
- U10 pad JP2_23: ADC_B_8 -> ADC_B_10
- U10 pad JP2_25: ADC_B_9 -> ADC_B_11
- U10 pad JP2_27: ADC_B_10 -> unconnected-(U10B-GPIO_122-PadJP2_27)
- U10 pad JP2_29: Net-(U10B-GPIO-1_VCC3P3) -> unconnected-(U10B-GPIO-1_VCC3P3-PadJP2_29)
- U10 pad JP2_3: unconnected-(U10B-GPIO_1_IN1-PadJP2_3) -> ADC_B_1
- U10 pad JP2_30: GND -> Net-(U10B-GPIO-1_GND-PadJP2_12)
- U10 pad JP2_31: ADC_B_11 -> unconnected-(U10B-GPIO_124-PadJP2_31)
- U10 pad JP2_33: ADC_B_10 -> unconnected-(U10B-GPIO_126-PadJP2_33)
- U10 pad JP2_35: ADC_B_11 -> unconnected-(U10B-GPIO_128-PadJP2_35)
- U10 pad JP2_37: ADC_A_13 -> unconnected-(U10B-GPIO_130-PadJP2_37)
- U10 pad JP2_39: ADC_A_12 -> unconnected-(U10B-GPIO_132-PadJP2_39)
- U10 pad JP2_5: ADC_B_0 -> ADC_B_2
- U10 pad JP2_7: ADC_B_1 -> ADC_B_3
- U10 pad JP2_9: ADC_B_2 -> ADC_B_4
- U11 pad 1: Net-(U11-ADJ) -> unconnected-(U11-TE-Pad1)
- U11 pad 2: Net-(U11-VI) -> Net-(U11-B1)
- U11 pad 3: -3V5 -> Net-(U11-B2)
- U14 pad 1: Net-(U14-ADJ) -> unconnected-(U14-TE-Pad1)
- U14 pad 3: -5V -> Net-(U14-B2)
- U2 pad 1: Net-(U2-ADJ) -> AN_TRIGGER_P
- U2 pad 2: +5V -> GND
- U21 pad 1: CH1_CH+ -> Net-(D6-K)
- U21 pad 2: CH1_CH- -> +5V
- U21 pad 4: GND -> unconnected-(U21-FB-Pad4)
- U21 pad 5: GND -> Net-(U21-~{ON}/OFF)
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Other:
- board size 159 x 149.3 mm -> 160 x 100 mm

Commit message: Add all footprints
Parts:
- removed K10, K8, K9: G2RL-2, Relay_THT:Relay_DPDT_Omron_G2RL-2
- removed TR1: Wuerth_749013011A, Transformer_SMD:Transformer_Ethernet_Wuerth_749013011A
- removed the U11 at (86.5, 125.0)
- removed U19: LM2596S-ADJ, Package_TO_SOT_SMD:TO-263-5_TabPin3
- removed the U2 at (74.1, -72.8)
- removed U20: INA180A3, Package_TO_SOT_SMD:SOT-23-5
- removed U21, U22: LM2596S-5, Package_TO_SOT_SMD:TO-263-5_TabPin3
- removed U23, U24, U25, U26, U27: AP1117-ADJ, Package_TO_SOT_SMD:SOT-223-3_TabPin2
- removed U28: STM32H723ZGIx, Package_BGA:UFBGA-144_7x7mm_Layout12x12_P0.5mm
- removed U29: LAN8742A, Package_DFN_QFN:VQFN-24-1EP_4x4mm_P0.5mm_EP2.5x2.5mm_ThermalVias
- added C1: DNP, Capacitor_SMD:C_0805_2012Metric, F.Cu at (143.8, 58.0)
- added C10: DNP, Capacitor_SMD:C_0805_2012Metric, F.Cu at (84.8, 104.9)
- added C100: 10nF, Capacitor_SMD:C_0805_2012Metric, F.Cu at (288.6, -64.9)
- added C101: 10uF, Capacitor_SMD:C_0805_2012Metric, F.Cu at (284.0, -129.6)
- added C102: 10uF, Capacitor_SMD:C_0805_2012Metric, F.Cu at (284.0, -123.6)
- added C103: 10uF, Capacitor_SMD:C_0805_2012Metric, F.Cu at (288.4, -123.6)
- added C104: 10uF, Capacitor_SMD:C_0805_2012Metric, F.Cu at (284.0, -120.6)
- added C105: 10uF, Capacitor_SMD:C_0805_2012Metric, F.Cu at (288.4, -132.6)
- added C106: 100nF, Capacitor_SMD:C_0805_2012Metric, F.Cu at (288.4, -120.6)
- added C107: 100nF, Capacitor_SMD:C_0805_2012Metric, F.Cu at (288.4, -135.7)
- added C108: 10uF, Capacitor_SMD:C_0805_2012Metric, F.Cu at (288.4, -129.6)
- added C109: 100nF, Capacitor_SMD:C_0805_2012Metric, F.Cu at (288.4, -126.6)
- added C11: C 2.0 - 6.0 pF, Capacitor_SMD:C_Trimmer_Murata_TZB4-A, F.Cu at (146.0, 79.0)
- added C110: 100nF, Capacitor_SMD:C_0805_2012Metric, F.Cu at (297.3, -138.7)
- added C111: 10uF, Capacitor_SMD:C_0805_2012Metric, F.Cu at (292.9, -120.6)
- added C112: 10uF, Capacitor_SMD:C_0805_2012Metric, F.Cu at (297.3, -132.6)
- added C113: 10uF, Capacitor_SMD:C_0805_2012Metric, F.Cu at (297.3, -135.7)
- added C114: 100nF, Capacitor_SMD:C_0805_2012Metric, F.Cu at (292.9, -123.6)
- added C115: 100nF, Capacitor_SMD:C_0805_2012Metric, F.Cu at (297.3, -129.6)
- added C116: 10uF, Capacitor_SMD:C_0805_2012Metric, F.Cu at (284.0, -126.6)
- added C117: 10uF, Capacitor_SMD:C_0805_2012Metric, F.Cu at (284.0, -138.7)
- added C118: 10uF, Capacitor_SMD:C_0805_2012Metric, F.Cu at (292.9, -138.7)
- added C119: 10uF, Capacitor_SMD:C_0805_2012Metric, F.Cu at (284.0, -135.7)
- added C12: C 2.0 - 6.0 pF, Capacitor_SMD:C_Trimmer_Murata_TZB4-A, F.Cu at (84.8, 107.9)
- added C120: 100nF, Capacitor_SMD:C_0805_2012Metric, F.Cu at (292.9, -135.7)
- added C121: 100nF, Capacitor_SMD:C_0805_2012Metric, F.Cu at (284.0, -132.6)
- added C122: 100nF, Capacitor_SMD:C_0805_2012Metric, F.Cu at (292.9, -132.6)
- added C123: 100nF, Capacitor_SMD:C_0805_2012Metric, F.Cu at (288.4, -138.7)
- added C124: 10uF, Capacitor_SMD:C_0805_2012Metric, F.Cu at (292.9, -126.6)
- added C125: 10uF, Capacitor_SMD:C_0805_2012Metric, F.Cu at (292.9, -129.6)
- added C126: 1uF, Capacitor_SMD:C_0805_2012Metric, F.Cu at (279.5, -91.8)
- added C127: 0.1uF, Capacitor_SMD:C_0805_2012Metric, F.Cu at (279.5, -88.8)
- added C128: 100pF, Capacitor_SMD:C_0805_2012Metric, F.Cu at (284.0, -100.8)
- added C129: 150nF, Capacitor_SMD:C_0805_2012Metric, F.Cu at (279.5, -94.8)
- added C13: 22nF, Capacitor_SMD:C_0805_2012Metric, F.Cu at (206.0, -123.0)
- added C130: 330pF, Capacitor_SMD:C_0805_2012Metric, F.Cu at (279.5, -97.8)
- added C131: 100pF, Capacitor_SMD:C_0805_2012Metric, F.Cu at (279.5, -100.8)
- added C132: 100pF, Capacitor_SMD:C_0805_2012Metric, F.Cu at (288.4, -97.8)
- added C133: 100pF, Capacitor_SMD:C_0805_2012Metric, F.Cu at (284.0, -91.8)
- added C134: 0.1uF, Capacitor_SMD:C_0805_2012Metric, F.Cu at (284.0, -88.8)
- added C135: 0.1uF, Capacitor_SMD:C_0805_2012Metric, F.Cu at (288.4, -94.8)
- added C136: 0.1uF, Capacitor_SMD:C_0805_2012Metric, F.Cu at (284.0, -94.8)
- added C137: 1uF, Capacitor_SMD:C_0805_2012Metric, F.Cu at (288.4, -100.8)
- added C138: 1uF, Capacitor_SMD:C_0805_2012Metric, F.Cu at (288.4, -91.8)
- added C139: 1uF, Capacitor_SMD:C_0805_2012Metric, F.Cu at (284.0, -97.8)
- added C14: 22nF, Capacitor_SMD:C_0805_2012Metric, F.Cu at (206.0, -95.9)
- added C15: 100nF, Capacitor_SMD:C_0805_2012Metric, F.Cu at (232.7, -105.0)
- added C16: 100nF, Capacitor_SMD:C_0805_2012Metric, F.Cu at (210.4, -114.0)
- added C17: 1uF, Capacitor_SMD:C_0805_2012Metric, F.Cu at (232.7, -101.9)
- added C18: 1uF, Capacitor_SMD:C_0805_2012Metric, F.Cu at (210.4, -111.0)
- added C19: 10uF, Capacitor_SMD:C_0805_2012Metric, F.Cu at (232.7, -98.9)
- added C2: DNP, Capacitor_SMD:C_0805_2012Metric, F.Cu at (58.4, 99.0)
- added C20: 10uF, Capacitor_SMD:C_0805_2012Metric, F.Cu at (232.7, -108.0)
- added C21: 100nF, Capacitor_SMD:C_0805_2012Metric, F.Cu at (228.2, -117.0)
- added C22: 100nF, Capacitor_SMD:C_0805_2012Metric, F.Cu at (223.8, -92.9)
- added C23: 1uF, Capacitor_SMD:C_0805_2012Metric, F.Cu at (228.2, -114.0)
- added C24: 1uF, Capacitor_SMD:C_0805_2012Metric, F.Cu at (228.2, -123.0)
- added C25: 100nF, Capacitor_SMD:C_0805_2012Metric, F.Cu at (223.8, -101.9)
- added C26: 100nF, Capacitor_SMD:C_0805_2012Metric, F.Cu at (223.8, -111.0)
- added C27: 10uF, Capacitor_SMD:C_0805_2012Metric, F.Cu at (228.2, -111.0)
- added C28: 10uF, Capacitor_SMD:C_0805_2012Metric, F.Cu at (228.2, -120.0)
- added C29: 1uF, Capacitor_SMD:C_0805_2012Metric, F.Cu at (223.8, -98.9)
- added C3: C 2.0 - 10.0 pF, Capacitor_SMD:C_Trimmer_Murata_TZB4-A, F.Cu at (143.8, 60.0)
- added C30: 1uF, Capacitor_SMD:C_0805_2012Metric, F.Cu at (223.8, -108.0)
- added C31: 10uF, Capacitor_SMD:C_0805_2012Metric, F.Cu at (223.8, -95.9)
- added C32: 10uF, Capacitor_SMD:C_0805_2012Metric, F.Cu at (223.8, -105.0)
- added C33: 22nF, Capacitor_SMD:C_0805_2012Metric, F.Cu at (232.7, -123.0)
- added C34: 100nF, Capacitor_SMD:C_0805_2012Metric, F.Cu at (228.2, -101.9)
- added C35: 100nF, Capacitor_SMD:C_0805_2012Metric, F.Cu at (228.2, -108.0)
- added C36: 1uF, Capacitor_SMD:C_0805_2012Metric, F.Cu at (228.2, -98.9)
- added C37: 1uF, Capacitor_SMD:C_0805_2012Metric, F.Cu at (228.2, -105.0)
- added C38: 10uF, Capacitor_SMD:C_0805_2012Metric, F.Cu at (223.8, -123.0)
- added C39: 10uF, Capacitor_SMD:C_0805_2012Metric, F.Cu at (219.3, -108.0)
- added C4: C 360 pF, Capacitor_SMD:C_0805_2012Metric, F.Cu at (149.0, 56.0)
- added C40: 10uF, Capacitor_SMD:C_0805_2012Metric, F.Cu at (223.8, -120.0)
- added C41: 10uF, Capacitor_SMD:C_0805_2012Metric, F.Cu at (228.2, -95.9)
- added C42: 10uF, Capacitor_SMD:C_0805_2012Metric, F.Cu at (228.2, -92.9)
- added C43: 1uF, Capacitor_SMD:C_0805_2012Metric, F.Cu at (219.3, -92.9)
- added C44: 10uF, Capacitor_SMD:C_0805_2012Metric, F.Cu at (219.3, -105.0)
- added C45: 1uF, Capacitor_SMD:C_0805_2012Metric, F.Cu at (219.3, -111.0)
- added C46: 1uF, Capacitor_SMD:C_0805_2012Metric, F.Cu at (223.8, -117.0)
- added C47: 1uF, Capacitor_SMD:C_0805_2012Metric, F.Cu at (219.3, -101.9)
- added C48: 100nF, Capacitor_SMD:C_0805_2012Metric, F.Cu at (219.3, -95.9)
- added C49: 100nF, Capacitor_SMD:C_0805_2012Metric, F.Cu at (219.3, -114.0)
- added C5: C 2.0 - 10.0 pF, Capacitor_SMD:C_Trimmer_Murata_TZB4-A, F.Cu at (58.4, 105.0)
- added C50: 100nF, Capacitor_SMD:C_0805_2012Metric, F.Cu at (223.8, -114.0)
- added C51: 100nF, Capacitor_SMD:C_0805_2012Metric, F.Cu at (219.3, -98.9)
- added C52: DNP, Capacitor_SMD:C_0805_2012Metric, F.Cu at (210.4, -120.0)
- added C53: DNP, Capacitor_SMD:C_0805_2012Metric, F.Cu at (210.4, -123.0)
- added C54: 100nF, Capacitor_SMD:C_0805_2012Metric, F.Cu at (214.9, -117.0)
- added C55: 100nF, Capacitor_SMD:C_0805_2012Metric, F.Cu at (214.9, -108.0)
- added C56: DNP, Capacitor_SMD:C_0805_2012Metric, F.Cu at (232.7, -117.0)
- added C57: DNP, Capacitor_SMD:C_0805_2012Metric, F.Cu at (232.7, -120.0)
- added C58: 100nF, Capacitor_SMD:C_0805_2012Metric, F.Cu at (210.4, -117.0)
- added C59: 100nF, Capacitor_SMD:C_0805_2012Metric, F.Cu at (214.9, -98.9)
- added C6: C 360 pF, Capacitor_SMD:C_0805_2012Metric, F.Cu at (135.0, 103.0)
- added C60: DNP, Capacitor_SMD:C_0805_2012Metric, F.Cu at (232.7, -111.0)
- added C61: DNP, Capacitor_SMD:C_0805_2012Metric, F.Cu at (232.7, -114.0)
- added C62: 1uF, Capacitor_SMD:C_0805_2012Metric, F.Cu at (214.9, -114.0)
- added C63: 1uF, Capacitor_SMD:C_0805_2012Metric, F.Cu at (214.9, -105.0)
- added C64: 1uF, Capacitor_SMD:C_0805_2012Metric, F.Cu at (214.9, -95.9)
- added C65: 1uF, Capacitor_SMD:C_0805_2012Metric, F.Cu at (214.9, -92.9)
- added C66: 10uF, Capacitor_SMD:C_0805_2012Metric, F.Cu at (214.9, -111.0)
- added C67: 10uF, Capacitor_SMD:C_0805_2012Metric, F.Cu at (214.9, -101.9)
- added C68: 10uF, Capacitor_SMD:C_0805_2012Metric, F.Cu at (219.3, -123.0)
- added C69: 10uF, Capacitor_SMD:C_0805_2012Metric, F.Cu at (219.3, -120.0)
- added C7: C 390 pF, Capacitor_SMD:C_0805_2012Metric, F.Cu at (136.0, 74.0)
- added C70: 12pF, Capacitor_SMD:C_0805_2012Metric, F.Cu at (206.0, -92.9)
- added C71: 12pF, Capacitor_SMD:C_0805_2012Metric, F.Cu at (219.3, -117.0)
- added C72: DNP, Capacitor_SMD:C_0805_2012Metric, F.Cu at (210.4, -105.0)
- added C73: DNP, Capacitor_SMD:C_0805_2012Metric, F.Cu at (210.4, -108.0)
- added C74: DNP, Capacitor_SMD:C_0805_2012Metric, F.Cu at (210.4, -101.9)
- added C75: DNP, Capacitor_SMD:C_0805_2012Metric, F.Cu at (210.4, -98.9)
- added C76: 10uF, Capacitor_SMD:C_0805_2012Metric, F.Cu at (257.2, -59.2)
- added C77: 10uF, Capacitor_SMD:C_0805_2012Metric, F.Cu at (252.7, -56.2)
- added C78: 10uF, Capacitor_SMD:C_0805_2012Metric, F.Cu at (257.2, -56.2)
- added C79: 10uF, Capacitor_SMD:C_0805_2012Metric, F.Cu at (257.2, -74.2)
- added C8: DNP, Capacitor_SMD:C_0805_2012Metric, F.Cu at (142.0, 79.0)
- added C80: 1uF, Capacitor_SMD:C_0805_2012Metric, F.Cu at (261.6, -74.2)
- added C81: 1uF, Capacitor_SMD:C_0805_2012Metric, F.Cu at (257.2, -71.2)
- added C82: 2.2uF, Capacitor_SMD:C_0805_2012Metric, F.Cu at (252.7, -71.2)
- added C83: 2.2uF, Capacitor_SMD:C_0805_2012Metric, F.Cu at (252.7, -74.2)
- added C84: 1uF, Capacitor_SMD:C_0805_2012Metric, F.Cu at (261.6, -71.2)
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- renumbered U9 to U11, U8 to U2, U1 to U3
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Connections:
- D10 pad 1: Net-(D10-K) -> +5V_EXT
- D10 pad 2: +15V -> AC_DC_CH1
- D2 pad 1: Net-(D2-K) -> -5V
- D2 pad 2: GND -> +5V
- D6 pad 1: Net-(D6-K) -> +5V_EXT
- D6 pad 2: +15V -> CH1_ATTEN_A
- D7 pad 1: Net-(D7-K) -> +5V_EXT
- D7 pad 2: -5V -> CH1_ATTEN_B
- D8 pad 1: Net-(D8-K) -> +5V_EXT
- D8 pad 2: -5V -> CH2_ATTEN_A
- D9 pad 1: +15V -> +5V_EXT
- D9 pad 2: Net-(D9-A) -> CH2_ATTEN_B
- Q1 pad 1: USB_PD_FAULT -> Net-(Q1-G)
- Q1 pad 3: Net-(Q1-D) -> TRIGG_1
- Q2 pad 2: Net-(Q2-S) -> GND
- Q2 pad 3: Net-(Q2-D) -> TRIGG_2
- Q3 pad 1: Net-(Q2-G) -> Net-(Q3-G)
- Q3 pad 2: Net-(Q2-S) -> GND
- Q3 pad 3: Net-(Q3-D) -> TRIGGER_AC_DC
- R100 pad 1: Net-(U11-B6) -> GPIO_PD5
- R100 pad 2: ADC_A_5 -> Net-(U11D-D53/USART_B_TX)
- R101 pad 1: Net-(U11-B7) -> GPIO_PD4
- R101 pad 2: ADC_A_6 -> Net-(U11D-D54/USART_B_RTS)
- R102 pad 1: Net-(U11-B8) -> GPIO_PD3
- R102 pad 2: ADC_A_7 -> Net-(U11D-D55/USART_B_CTS)
- R103 pad 1: Net-(U12-B1) -> GPIO_PE4
- R103 pad 2: ADC_A_8 -> Net-(U11D-D57/SAI_A_FS)
- R104 pad 1: Net-(U12-B2) -> GPIO_PE5
- R104 pad 2: ADC_A_9 -> Net-(U11D-D58/SAI_A_SCK)
- R105 pad 1: Net-(U12-B3) -> GPIO_PE6
- R105 pad 2: ADC_A_10 -> Net-(U11D-D59/SAI_A_SD)
- R106 pad 1: Net-(U12-B4) -> USART_1_RX
- R106 pad 2: ADC_A_11 -> Net-(U11F-D0/USART_A_RX)
- R107 pad 1: Net-(U13-B1) -> USART_1_TX
- R107 pad 2: ADC_B_0 -> Net-(U11F-D1/USART_A_TX)
- R108 pad 1: Net-(U13-B2) -> GPIO_PE9
- R108 pad 2: ADC_B_1 -> Net-(U11F-D6/TIMER_A_PWM1)
- R109 pad 1: Net-(U13-B3) -> GPIO_PE11
- R109 pad 2: ADC_B_2 -> Net-(U11F-D5/TIMER_A_PWM2)
- R110 pad 1: Net-(U13-B4) -> GPIO_PE13
- R110 pad 2: ADC_B_3 -> Net-(U11F-D3/TIMER_A_PWM3)
- R111 pad 1: Net-(U13-B5) -> GPIO_PE15
- R111 pad 2: ADC_B_4 -> Net-(U11F-D37/TIMER_A_BKIN1)
- R112 pad 1: Net-(U13-B6) -> GPIO_PE12
- R112 pad 2: ADC_B_5 -> Net-(U11F-D39/TIMER_A_PWM3N)
- R113 pad 1: Net-(U13-B7) -> GPIO_PE10
- R113 pad 2: ADC_B_6 -> Net-(U11F-D40/TIMER_A_PWM2N)
- R114 pad 1: Net-(U13-B8) -> GPIO_PE7
- R114 pad 2: ADC_B_7 -> Net-(U11F-D41/TIMER_A_ETR)
- R115 pad 1: Net-(U14-B1) -> GPIO_PE8
- R115 pad 2: ADC_B_8 -> Net-(U11F-D42/TIMER_A_PWM1N)
- R116 pad 1: Net-(U14-B2) -> Net-(Q4-G)
- R116 pad 2: ADC_B_9 -> CH1_ATTEN_A_MCU
- R117 pad 1: Net-(U14-B3) -> Net-(Q4-G)
- R117 pad 2: ADC_B_10 -> GND
- R118 pad 1: Net-(U14-B4) -> Net-(Q5-G)
- R118 pad 2: ADC_B_11 -> CH1_ATTEN_B_MCU
- R95 pad 1: Net-(U11-B1) -> GPIO_PE6
- R95 pad 2: ADC_A_0 -> +3V3
- R96 pad 1: Net-(U11-B2) -> USART_1_TX
- R96 pad 2: ADC_A_1 -> +3V3
- R97 pad 1: Net-(U11-B3) -> +3V3
- R97 pad 2: ADC_A_2 -> GPIO_PE8
- R98 pad 1: Net-(U11-B4) -> GPIO_PD7
- R98 pad 2: ADC_A_3 -> Net-(U11D-D51/USART_B_SCLK)
- R99 pad 1: Net-(U11-B5) -> GPIO_PD6
- R99 pad 2: ADC_A_4 -> Net-(U11D-D52/USART_B_RX)
- U10 pad JP1_10: unconnected-(U10A-GPIO_07-PadJP1_10) -> GPIO_23
- U10 pad JP1_11: unconnected-(U10A-GPIO-0_VCC_SYS-PadJP1_11) -> Net-(U10A-GPIO-0_VCC_SYS)
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Other:
- board size 160 x 100 mm -> 150 x 150 mm
- copper layers 2 -> 4

Commit message: Fix footprints and allign components placements
Parts:
- removed D10, D11: 1N4001, Diode_THT:D_DO-41_SOD81_P10.16mm_Horizontal
- removed Q5, Q7: 2N7002, Package_TO_SOT_SMD:SOT-23
- removed R100, R101, R102, R103, R104, R105, R106, R107, R108, R109, R110, R111, R112, R113, R114, R115, R135, R136, R137, R138, R139, R140, R141, R142, R143, R144, R145, R146, R147, R148, R98, R99: 33R, Resistor_SMD:R_0805_2012Metric
- removed R118, R150: 220R, Resistor_SMD:R_0805_2012Metric
- removed R119, R151: 10k, Resistor_SMD:R_0805_2012Metric
- removed R120, R121, R122, R123, R124, R125, R126, R127, R128, R129, R130, R131, R132, R133, R71, R80, R81, R82, R83, R84, R85, R86, R87, R88, R89, R90, R91, R92, R94, R95, R97: 10kR, Resistor_SMD:R_0805_2012Metric
- added C140: 100pF, Capacitor_SMD:C_0805_2012Metric, F.Cu at (405.8, -89.1)
- added C141: 100pF, Capacitor_SMD:C_0805_2012Metric, F.Cu at (405.8, -86.1)
- added C142: 10uF, Capacitor_SMD:C_0805_2012Metric, F.Cu at (416.6, -64.7)
- added C143: 10uF, Capacitor_SMD:C_0805_2012Metric, F.Cu at (416.6, -61.7)
- added C144: 100nF, Capacitor_SMD:C_0805_2012Metric, F.Cu at (416.6, -58.7)
- added C145: 100nF, Capacitor_SMD:C_0805_2012Metric, F.Cu at (416.6, -55.7)
- added C146: 10uF, Capacitor_SMD:C_0805_2012Metric, F.Cu at (416.6, -52.7)
- added C147: 10uF, Capacitor_SMD:C_0805_2012Metric, F.Cu at (421.1, -64.7)
- added C148: 10uF, Capacitor_SMD:C_0805_2012Metric, F.Cu at (421.1, -61.7)
- added C149: 100nF, Capacitor_SMD:C_0805_2012Metric, F.Cu at (421.1, -58.7)
- added C150: 100nF, Capacitor_SMD:C_0805_2012Metric, F.Cu at (421.1, -55.7)
- added C151: 10uF, Capacitor_SMD:C_0805_2012Metric, F.Cu at (421.1, -52.7)
- added J10: Conn_01x02_Pin, TerminalBlock:TerminalBlock_MaiXu_MX126-5.0-02P_1x02_P5.00mm, F.Cu at (418.4, -103.7)
- added J11: Conn_01x02_Pin, TerminalBlock:TerminalBlock_MaiXu_MX126-5.0-02P_1x02_P5.00mm, F.Cu at (418.4, -93.6)
- added J12: Conn_01x02_Pin, TerminalBlock:TerminalBlock_MaiXu_MX126-5.0-02P_1x02_P5.00mm, F.Cu at (418.4, -83.5)
- added J14: Conn_01x02_Pin, TerminalBlock:TerminalBlock_MaiXu_MX126-5.0-02P_1x02_P5.00mm, F.Cu at (418.4, -73.3)
- added J8: Conn_01x03_Pin, TerminalBlock:TerminalBlock_MaiXu_MX126-5.0-03P_1x03_P5.00mm, F.Cu at (431.0, -103.7)
- added J9: Conn_01x03_Pin, TerminalBlock:TerminalBlock_MaiXu_MX126-5.0-03P_1x03_P5.00mm, F.Cu at (431.0, -93.6)
- added K6: TQ2-5V, TQ2-5V:TQ2, F.Cu at (154.0, 115.0)
- added K7: TQ2-5V, TQ2-5V:TQ2, F.Cu at (166.0, 115.0)
- added L59: 0.68uH, 0.8Ohm, Inductor_SMD:L_0805_2012Metric, F.Cu at (425.6, -52.6)
- added L60: LCBB-601, Inductor_SMD:L_0805_2012Metric, F.Cu at (425.6, -49.9)
- added L61: 0.68uH, 0.8Ohm, Inductor_SMD:L_0805_2012Metric, F.Cu at (425.6, -47.1)
- added L62: LCBB-601, Inductor_SMD:L_0805_2012Metric, F.Cu at (425.6, -44.4)
- added U18: AZ1117-ADJ, Package_TO_SOT_SMD:SOT-89-3, F.Cu at (426.7, -63.1)
- added U19: AZ1117-ADJ, Package_TO_SOT_SMD:SOT-89-3, F.Cu at (426.7, -57.0)
- C11, C12: value C 2.0 - 6.0 pF -> 2.0-6.0pF
- C3, C5: value C 2.0 - 10.0 pF -> 2.0-10.0pF
- C4, C6: value C 360 pF -> 360pF
- C7, C9: value C 390 pF -> 390pF
- D12, D13, D14: footprint Diode_THT:D_DO-41_SOD81_P10.16mm_Horizontal -> LED_SMD:LED_0805_2012Metric
- D3, D4, D5: value 1N4001 -> 1N4148W; footprint LED_SMD:LED_0805_2012Metric -> Diode_SMD:D_SOD-123
- D6, D7, D8, D9: value 1N4001 -> 1N4148W; footprint Diode_THT:D_DO-41_SOD81_P10.16mm_Horizontal -> Diode_SMD:D_SOD-123
- K1, K2, K3, K4, K5: value TQ2-L2-5V -> TQ2-5V; footprint TQ2:RELAY_TQ2_2C_PAN -> TQ2-5V:TQ2
- R1, R2: value R 953k -> 990k
- R10, R8: value R 953k -> 953k
- R14, R18: value 10k -> 120
- R16, R19: value 10k -> 200
- R31, R32: value 10k -> 2M
- R5, R6: value R 9.53 kΩ -> 10k
- R56: value DNP -> 10kR
- R57: value DNP -> 10R
- R66: value 10kR -> 10R
- R67, R70: value 10kR -> 10k
- R68, R69: value 10kR -> 20k
- R7, R9: value R 49.9k -> 49.9k
- U2, U3: footprint OPA656U:SOIC127P599X175-8N -> OPA656:SOIC127P599X175-8N
- U4: footprint AD813ARZ:R_8_ADI-L -> AD8611ARZ:R_8_ADI-L
- U7, U8: footprint AD813ARZ:R_8_ADI-L -> AD8138ARZ:R_8_ADI-L
- moved C2 404.0 mm to (405.8, -107.2)
- moved C9 398.8 mm to (405.8, -95.2)
- moved C5 393.7 mm to (407.9, -76.3)
- moved C10 376.6 mm to (405.8, -92.2)
- moved C12 366.5 mm to (407.9, -65.2)
- moved R2 346.5 mm to (405.8, -58.0)
- moved R10 343.1 mm to (410.2, -55.1)
- moved R9 343.1 mm to (410.2, -58.0)
- moved R6 342.7 mm to (405.8, -52.1)
- moved C6 339.2 mm to (405.8, -101.2), turned to 0 degrees
- moved C7 320.1 mm to (405.8, -98.2), turned to 0 degrees
- moved R8 310.0 mm to (410.2, -61.0), turned to 0 degrees
- moved C4 302.7 mm to (405.8, -104.2)
- moved C11 301.6 mm to (407.9, -70.8), turned to 0 degrees
- moved C3 299.7 mm to (407.9, -81.9)
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Connections:
- net CH1_ATTEN_A_MCU renamed CH1_ATTEN_MCU
- net CH2_ATTEN_A_MCU renamed CH2_ATTEN_MCU
- C52 pad 1: +1V5 -> +1V5_VOCM_CH1
- C53 pad 1: +1V5 -> +1V5_VOCM_CH2
- C76 pad 1: Net-(C76-Pad1) -> +VDD_FILTERED
- C78 pad 1: Net-(C76-Pad1) -> +VDD_FILTERED
- C80 pad 1: Net-(C76-Pad1) -> +VDD_FILTERED
- C82 pad 1: +1V5 -> +1V5_VOCM_CH1
- C83 pad 1: +1V5 -> +1V5_VOCM_CH2
- C84 pad 1: Net-(C76-Pad1) -> +VDD_FILTERED
- C88 pad 1: Net-(C76-Pad1) -> +VDD_FILTERED
- C92 pad 1: Net-(C76-Pad1) -> +VDD_FILTERED
- D6 pad 2: CH1_ATTEN_A -> CH1_ATTEN
- D7 pad 2: CH1_ATTEN_B -> CH2_ATTEN
- D8 pad 2: CH2_ATTEN_A -> AC_DC_CH1
- D9 pad 2: CH2_ATTEN_B -> AC_DC_CH2
- J4 pad 3: +1V5 -> +1V5_VOCM_CH2
- J5 pad 3: +1V5 -> +1V5_VOCM_CH1
- K1 pad 10: +5V_EXT -> CH1_ATTEN
- K1 pad 5: CH1_ATTEN_A -> (no net)
- K1 pad 6: CH1_ATTEN_B -> (no net)
- K2 pad 10: +5V_EXT -> CH2_ATTEN
- K2 pad 5: CH2_ATTEN_A -> (no net)
- K2 pad 6: CH2_ATTEN_B -> (no net)
- K3 pad 10: +5V_EXT -> AC_DC_CH1
- K3 pad 2: unconnected-(K3-Pad2) -> Net-(D2A-K3A4)
- K3 pad 3: Net-(C14-Pad1) -> Net-(C13-Pad1)
- K3 pad 4: Net-(D1A-K3A4) -> unconnected-(K3-Pad4)
- K3 pad 5: AC_DC_CH2 -> (no net)
- K3 pad 6: AC_DC_CH1 -> (no net)
- K3 pad 7: Net-(D2A-K3A4) -> unconnected-(K3-Pad7)
- K3 pad 8: Net-(C13-Pad1) -> unconnected-(K3-Pad8)
- K4 pad 10: +5V_EXT -> AC_DC_CH2
- K4 pad 2: AN_TRIGGER_CH1 -> Net-(D1A-K3A4)
- K4 pad 3: Net-(K4-Pad3) -> Net-(C14-Pad1)
- K4 pad 4: AN_TRIGGER_CH2 -> unconnected-(K4-Pad4)
- K4 pad 5: TRIGG_1 -> (no net)
- K4 pad 6: TRIGG_2 -> (no net)
- K4 pad 7: EXT_TRIGGER_LEVEL -> unconnected-(K4-Pad7)
- K4 pad 8: Net-(C33-Pad1) -> unconnected-(K4-Pad8)
- K4 pad 9: Net-(K4-Pad3) -> unconnected-(K4-Pad9)
- K5 pad 10: unconnected-(K5-Pad10) -> TRIGG_1
- K5 pad 2: unconnected-(K5-Pad2) -> AN_TRIGGER_CH1
- K5 pad 3: Net-(C33-Pad1) -> Net-(K5-Pad3)
- K5 pad 4: Net-(C33-Pad2) -> AN_TRIGGER_CH2
- K5 pad 5: TRIGGER_AC_DC -> (no net)
- K5 pad 6: unconnected-(K5-Pad6) -> (no net)
- L33 pad 1: +3V3 -> +3V3A
- L34 pad 1: +3V3 -> +3V3A
- L35 pad 2: Net-(C76-Pad1) -> +VDD_FILTERED
- L39 pad 1: +3V3 -> +3V3DRV
- L40 pad 1: +3V3 -> +3V3DRV
- Q4 pad 3: CH1_ATTEN_A -> CH1_ATTEN
- Q6 pad 3: CH2_ATTEN_A -> CH2_ATTEN
- R14 pad 1: Net-(U2-POS) -> +3V3A
- R14 pad 2: Net-(D1A-K3A4) -> Net-(U18-ADJ)
- R15 pad 2: Net-(U1B--) -> Net-(C141-Pad2)
- R16 pad 1: Net-(U2-POS) -> Net-(U18-ADJ)
- R17 pad 2: Net-(U1A--) -> Net-(C140-Pad2)
- R18 pad 1: Net-(U3-POS) -> +3V3DRV
- R18 pad 2: Net-(D2A-K3A4) -> Net-(U19-ADJ)
- R19 pad 1: Net-(U3-POS) -> Net-(U19-ADJ)
- R56 pad 1: CLK_FPGA_PLL_50MHz -> DAC_ALM
- R56 pad 2: CLOCK_80MHz -> +3V3
- R57 pad 1: CLK_FPGA_PLL_50MHz -> Net-(C140-Pad2)
- R57 pad 2: CLOCK_80MHz -> Net-(U1A--)
- R60 pad 2: +5V -> +5V_EXT
- R62 pad 2: +5V -> +5V_EXT
- R66 pad 1: +3V3 -> Net-(C141-Pad2)
- R66 pad 2: GPIO_PD15 -> Net-(U1B--)
- R67 pad 1: +3V3 -> +VDD_FILTERED
- R67 pad 2: SPI_1_CS -> Net-(R67-Pad2)
- R68 pad 1: +3V3 -> Net-(R67-Pad2)
- R68 pad 2: SPI_1_MOSI -> Net-(J11-Pin_2)
- R69 pad 1: +3V3 -> +VDD_FILTERED
- R69 pad 2: SPI_1_MISO -> Net-(R69-Pad2)
- R70 pad 1: +3V3 -> Net-(R69-Pad2)
- R70 pad 2: SPI_1_SCK -> Net-(J10-Pin_2)
- R76 pad 2: +5V -> +5V_EXT
- TP7 pad 1: Net-(U1A--) -> Net-(C140-Pad2)
- TP8 pad 1: Net-(U1B--) -> Net-(C141-Pad2)
- U11 pad CN10_10: Net-(U11F-D3/TIMER_A_PWM3) -> GPIO_PE13
- U11 pad CN10_13: Net-(U11F-D26/QSPI_CS) -> QSPI_CS
- U11 pad CN10_14: Net-(U11F-D1/USART_A_TX) -> USART_1_TX
- U11 pad CN10_15: Net-(U11F-D27/QSPI_CLK) -> QSPI_CLK
- U11 pad CN10_16: Net-(U11F-D0/USART_A_RX) -> USART_1_RX
- U11 pad CN10_18: Net-(U11F-D42/TIMER_A_PWM1N) -> GPIO_PE8
- U11 pad CN10_19: Net-(U11F-D28/QSPI_BK1_IO3) -> QSPI_IO3/GPIO_PD13
- U11 pad CN10_20: Net-(U11F-D41/TIMER_A_ETR) -> GPIO_PE7
- U11 pad CN10_21: Net-(U11F-D29/QSPI_BK1_IO1) -> QSPI_IO1/GPIO_PD12
- U11 pad CN10_23: Net-(U11F-D30/QSPI_BK1_IO0) -> QSPI_IO0/GPIO_PD11
- U11 pad CN10_24: Net-(U11F-D40/TIMER_A_PWM2N) -> GPIO_PE10
- U11 pad CN10_25: Net-(U11F-D31/QSPI_BK1_IO2) -> QSPI_IO2/GPIO_PE2
- U11 pad CN10_26: Net-(U11F-D39/TIMER_A_PWM3N) -> GPIO_PE12
- U11 pad CN10_29: Net-(U11F-D32/TIMER_C_PWM1) -> GPIO_4
- U11 pad CN10_30: Net-(U11F-D37/TIMER_A_BKIN1) -> GPIO_PE15
- U11 pad CN10_31: Net-(U11F-D33/TIMER_D_PWM1) -> GPIO_1
- U11 pad CN10_32: Net-(U11F-D36/TIMER_C_PWM2) -> GPIO_3
- U11 pad CN10_33: Net-(U11F-D34/TIMER_B_ETR) -> GPIO_PE0
- U11 pad CN10_34: Net-(U11F-D35/TIMER_C_PWM3) -> GPIO_2
- U11 pad CN10_4: Net-(U11F-D6/TIMER_A_PWM1) -> GPIO_PE9
- U11 pad CN10_6: Net-(U11F-D5/TIMER_A_PWM2) -> GPIO_PE11
- U11 pad CN10_8: Net-(U11F-D4/IO) -> GPIO_0
- U11 pad CN7_13: CH1_ATTEN_B_MCU -> unconnected-(U11E-D22/I2S_B_SD/SPI_B_MOSI-PadCN7_13)
- U11 pad CN7_17: CH2_ATTEN_B_MCU -> unconnected-(U11E-D24/SPI_B_NSS-PadCN7_17)
- U11 pad CN9_1: unconnected-(U11D-A0/ADC12_INP15-PadCN9_1) -> DAC_TEMP
- U11 pad CN9_10: Net-(U11D-D55/USART_B_CTS) -> GPIO_PD3
- U11 pad CN9_16: Net-(U11D-D57/SAI_A_FS) -> GPIO_PE4
- U11 pad CN9_18: Net-(U11D-D58/SAI_A_SCK) -> GPIO_PE5
- U11 pad CN9_19: DAC_TEMP -> GPIO_PD0
- U11 pad CN9_2: Net-(U11D-D51/USART_B_SCLK) -> GPIO_PD7
- U11 pad CN9_20: Net-(U11D-D59/SAI_A_SD) -> GPIO_PE6
- U11 pad CN9_21: unconnected-(U11D-D68/I2C_B_SDA-PadCN9_21) -> GPIO_PD1
- U11 pad CN9_25: Net-(U11D-D67/CAN_RX) -> unconnected-(U11D-D67/CAN_RX-PadCN9_25)
- U11 pad CN9_27: Net-(U11D-D66/CAN_TX) -> unconnected-(U11D-D66/CAN_TX-PadCN9_27)
- U11 pad CN9_4: Net-(U11D-D52/USART_B_RX) -> GPIO_PD6
- U11 pad CN9_6: Net-(U11D-D53/USART_B_TX) -> GPIO_PD5
- U11 pad CN9_8: Net-(U11D-D54/USART_B_RTS) -> GPIO_PD4
- U2 pad 3: Net-(U2-POS) -> Net-(D1A-K3A4)
- U3 pad 3: Net-(U3-POS) -> Net-(D2A-K3A4)
- U5 pad 2: Net-(U5-INPN) -> GND
- U6 pad 2: Net-(U6-INPN) -> GND
- U7 pad 2: +1V5 -> +1V5_VOCM_CH1
- U8 pad 2: +1V5 -> +1V5_VOCM_CH2
- U9 pad 11: Net-(U9-REFLB-Pad11) -> GND
- U9 pad 12: Net-(U9-REFLB-Pad11) -> GND
- U9 pad 13: Net-(U9-REFHB-Pad13) -> GND
- U9 pad 14: Net-(U9-REFHB-Pad13) -> GND
- U9 pad 18: Net-(C76-Pad1) -> +VDD_FILTERED
- U9 pad 20: +1V5 -> +1V5_VOCM_CH2
- U9 pad 60: GND -> Net-(J10-Pin_1)
- U9 pad 61: +1V5 -> +1V5_VOCM_CH1
- U9 pad 63: Net-(C76-Pad1) -> +VDD_FILTERED
- U9 pad 8: CLOCK_80MHz -> Net-(J8-Pin_2)
- U9 pad 9: CLOCK_80MHz -> Net-(J9-Pin_2)

Commit message: Route AFE - attenuators
Parts:
- moved D7 374.3 mm to (153.2, 85.0), turned to -90 degrees
- moved D9 371.8 mm to (157.4, 92.0), turned to -90 degrees
- moved C2 330.8 mm to (139.9, 89.6)
- moved C9 329.2 mm to (140.2, 99.4)
- moved C10 327.8 mm to (144.4, 105.7), turned to -90 degrees
- moved C12 319.9 mm to (137.4, 105.6), turned to 180 degrees
- moved C7 317.4 mm to (139.5, 74.6)
- moved C6 316.8 mm to (148.6, 83.8)
- moved R9 313.7 mm to (140.2, 101.8)
- moved C5 311.1 mm to (141.8, 85.0)
- moved TP2 309.8 mm to (132.6, 100.4)
- moved C11 309.0 mm to (137.4, 78.8), turned to 180 degrees
- moved R10 308.2 mm to (147.2, 105.6), turned to -90 degrees
- moved R2 305.4 mm to (139.9, 92.2)
- moved C4 303.4 mm to (148.6, 56.8)
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Routing:
- net Net-(C1-Pad2): track 0.00 -> 26.3 mm
- net Net-(C14-Pad1): track 0.00 -> 23.9 mm
- net Net-(C11-Pad1): track 0.00 -> 23.8 mm
- net Net-(C13-Pad1): track 0.00 -> 23.6 mm
- net Net-(C2-Pad2): track 0.00 -> 23.1 mm
- net Net-(C10-Pad1): track 0.00 -> 23.0 mm
- net GND: track 0.00 -> 15.9 mm, vias 0 -> 10
- net Net-(C1-Pad1): track 0.00 -> 15.2 mm
- net Net-(C2-Pad1): track 0.00 -> 14.9 mm
- net Net-(K2-Pad3): track 0.00 -> 14.6 mm
- net Net-(K1-Pad3): track 0.00 -> 14.2 mm
- net Net-(D1A-K3A4): track 0.00 -> 12.7 mm
- net Net-(C7-Pad1): track 0.00 -> 10.0 mm
- net Net-(C9-Pad1): track 0.00 -> 9.70 mm
- net Net-(J1-In): track 0.00 -> 9.20 mm
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- added copper zone on In2.Cu, net GND

Commit message: Route up to symetric amplifier in CH1
Parts:
- moved C141 299.8 mm to (158.2, 83.0), turned to 90 degrees
- moved C140 283.9 mm to (172.8, 73.0), turned to -90 degrees
- moved R66 281.3 mm to (159.3, 78.2)
- moved R57 272.0 mm to (169.2, 74.0), turned to 180 degrees
- moved TP8 227.1 mm to (157.6, 87.7)
- moved L1 220.0 mm to (153.3, 77.4), turned to 90 degrees
- moved L3 218.7 mm to (151.3, 77.5), turned to 90 degrees
- moved R53 214.3 mm to (196.7, 90.3), turned to 180 degrees
- moved D1 205.1 mm to (171.4, 87.4), turned to -90 degrees
- moved L2 201.0 mm to (177.2, 80.8), turned to 180 degrees
- moved R52 197.9 mm to (196.6, 95.1), turned to 180 degrees
- moved R15 197.8 mm to (156.0, 80.3), turned to 90 degrees
- moved R17 196.8 mm to (176.0, 74.0), turned to 180 degrees
- moved C16 196.5 mm to (169.1, 78.2), turned to 90 degrees
- moved TP7 195.6 mm to (179.8, 74.8)
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Routing:
- net GND: track 15.9 -> 47.2 mm, vias 10 -> 32
- net Net-(U3-NEG): track 0.00 -> 20.5 mm, vias 0 -> 2
- net Net-(D2A-K3A4): track 8.19 -> 26.8 mm
- net CH1_CH-: track 0.00 -> 16.0 mm
- net Net-(C141-Pad2): track 0.00 -> 13.0 mm
- net Net-(U8-+OUT): track 0.00 -> 12.3 mm
- net Net-(U3--VS): track 0.00 -> 12.3 mm
- net Net-(U1C-V-): track 0.00 -> 11.8 mm
- net Net-(U5-INPP): track 0.00 -> 11.3 mm
- net Net-(U5-GAIN): track 0.00 -> 11.1 mm
- net Net-(U1C-V+): track 0.00 -> 10.9 mm
- net Net-(U3-+VS): track 0.00 -> 10.7 mm
- net Net-(U5-VPOS): track 0.00 -> 10.7 mm
- net Net-(C140-Pad2): track 0.00 -> 10.4 mm
- net Net-(U3-OUTPUT): track 0.00 -> 10.2 mm
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- added copper zone on In1.Cu, net +5V_EXT
Other:
- board text added: "CH1"
- board text added: "CH2"
- board text added: "TRIG"
