File: fpga.kicad_sch (KiCad schematic)
At the start: 11 parts, among them U10 P0082_BOTTOMMOUNT, Y1 XLL735080.000000I

Commit message: Place all componenets
Parts:
- removed R58: 33R, Resistor_SMD:R_0805_2012Metric, symbol Device:R
- renumbered C100 to C102, R71 to R65
Connections:
- net AN_TRIGGER_N: now also U10.JP2_7 (GPIO_14); no longer U10.JP2_5 (GPIO_12)
- net AN_TRIGGER_P: now also U10.JP2_5 (GPIO_12); no longer U10.JP2_3 (GPIO_1_IN1)
- no-connect marks 19 -> 20
Changed lines of the file:
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@@
 	)
 	(no_connect
-		(at 80.01 128.27)
-	)
-	(no_connect
 		(at 80.01 46.99)
 	)
@@
 	)
 	(no_connect
+		(at 80.01 85.09)
+	)
+	(no_connect
 		(at 125.73 138.43)
 	)
@@
 		(at 125.73 125.73)
 	)
+	(no_connect
+		(at 80.01 123.19)
+	)
 	(bus_entry
 		(at 181.61 106.68)
@@
 	(wire
 		(pts
-			(xy 68.58 125.73) (xy 80.01 125.73)
-		)
-		(stroke
-			(width 0)
-			(type default)
-		)
-	)
-	(wire
-		(pts
 			(xy 127 175.26) (xy 127 179.07)
 		)
@@
 	(wire
 		(pts
+			(xy 68.58 128.27) (xy 80.01 128.27)
+		)
+		(stroke
+			(width 0)
+			(type default)
+		)
+	)
+	(wire
+		(pts
 			(xy 57.15 95.25) (xy 80.01 95.25)
 		)
@@
 		)
 	)
+	(wire
+		(pts
+			(xy 68.58 125.73) (xy 80.01 125.73)
+		)
+		(stroke
+			(width 0)
+			(type default)
+		)
+	)
 	(bus
 		(pts
@@
 	(wire
 		(pts
-			(xy 68.58 123.19) (xy 80.01 123.19)
-		)
-		(stroke
-			(width 0)
-			(type default)
-		)
-	)
-	(wire
-		(pts
 			(xy 68.58 120.65) (xy 80.01 120.65)
 		)
@@
 	(wire
 		(pts
-			(xy 60.96 85.09) (xy 57.15 85.09)
-		)
-		(stroke
-			(width 0)
-			(type default)
-		)
-	)
-	(wire
-		(pts
 			(xy 60.96 87.63) (xy 57.15 87.63)
 		)
@@
 		)
 	)
-	(wire
-		(pts
-			(xy 68.58 85.09) (xy 80.01 85.09)
-		)
-		(stroke
-			(width 0)
-			(type default)
-		)
-	)
 	(bus
 		(pts
@@
 	(global_label "AN_TRIGGER_N"
 		(shape input)
-		(at 68.58 125.73 180)
+		(at 68.58 128.27 180)
 		(fields_autoplaced yes)
 		(effects
@@
 		)
 		(property "Intersheetrefs" "${INTERSHEET_REFS}"
-			(at 52.1086 125.73 0)
+			(at 52.1086 128.27 0)
 			(effects
 				(font
@@
 	(global_label "AN_TRIGGER_P"
 		(shape input)
-		(at 68.58 123.19 180)
+		(at 68.58 125.73 180)
 		(fields_autoplaced yes)
 		(effects
@@
 		)
 		(property "Intersheetrefs" "${INTERSHEET_REFS}"
-			(at 52.1691 123.19 0)
+			(at 52.1691 125.73 0)
 			(effects
 				(font
@@
 		)
 	)
-	(global_label "CLK_FPGA_PLL_50MHz"
-		(shape input)
-		(at 57.15 85.09 180)
-		(fields_autoplaced yes)
-		(effects
-			(font
-				(size 1.27 1.27)
-			)
-			(justify right)
-		)
-		(property "Intersheetrefs" "${INTERSHEET_REFS}"
-			(at 33.4215 85.09 0)
-			(effects
-				(font
-					(size 1.27 1.27)
-				)
-				(justify right)
-				(hide yes)
-			)
-		)
-	)
 	(global_label "GPIO_23"
 		(shape input)
@@
 		(dnp no)
 		(fields_autoplaced yes)
-		(property "Reference" "#PWR0143"
+		(property "Reference" "#PWR0145"
 			(at 163.83 41.91 0)
 			(effects
@@
 			(project "DigitalOsciloscope"
 				(path "/553deb7b-4100-40fe-99d2-0c7b4b56aad2/3a7288c4-cf21-495b-9b8e-7b87b52ff1d8"
-					(reference "#PWR0143")
+					(reference "#PWR0145")
 					(unit 1)
 				)
@@
 		(dnp no)
 		(fields_autoplaced yes)
-		(property "Reference" "#PWR0148"
+		(property "Reference" "#PWR0150"
 			(at 256.54 72.39 0)
 			(effects
@@
 			(project ""
 				(path "/553deb7b-4100-40fe-99d2-0c7b4b56aad2/3a7288c4-cf21-495b-9b8e-7b87b52ff1d8"
-					(reference "#PWR0148")
+					(reference "#PWR0150")
 					(unit 1)
 				)
@@
 		(dnp no)
 		(fields_autoplaced yes)
-		(property "Reference" "#PWR0144"
+		(property "Reference" "#PWR0146"
 			(at 163.83 115.57 0)
 			(effects
@@
 			(project ""
 				(path "/553deb7b-4100-40fe-99d2-0c7b4b56aad2/3a7288c4-cf21-495b-9b8e-7b87b52ff1d8"
-					(reference "#PWR0144")
-					(unit 1)
-				)
-			)
-		)
-	)
-	(symbol
-		(lib_id "Device:R")
-		(at 64.77 85.09 90)
-		(unit 1)
-		(exclude_from_sim no)
-		(in_bom yes)
-		(on_board yes)
-		(dnp no)
-		(property "Reference" "R58"
-			(at 70.866 83.82 90)
-			(effects
-				(font
-					(size 1.27 1.27)
-				)
-			)
-		)
-		(property "Value" "33R"
-			(at 75.692 83.82 90)
-			(effects
-				(font
-					(size 1.27 1.27)
-				)
-			)
-		)
-		(property "Footprint" "Resistor_SMD:R_0805_2012Metric"
-			(at 64.77 86.868 90)
-			(effects
-				(font
-					(size 1.27 1.27)
-				)
-				(hide yes)
-			)
-		)
-		(property "Datasheet" "~"
-			(at 64.77 85.09 0)
-			(effects
-				(font
-					(size 1.27 1.27)
-				)
-				(hide yes)
-			)
-		)
-		(property "Description" "Resistor"
-			(at 64.77 85.09 0)
-			(effects
-				(font
-					(size 1.27 1.27)
-				)
-				(hide yes)
-			)
-		)
-		(pin "1"
-		)
-		(pin "2"
-		)
-		(instances
-			(project "DigitalOsciloscope"
-				(path "/553deb7b-4100-40fe-99d2-0c7b4b56aad2/3a7288c4-cf21-495b-9b8e-7b87b52ff1d8"
-					(reference "R58")
+					(reference "#PWR0146")
 					(unit 1)
 				)
@@
 		(dnp no)
 		(fields_autoplaced yes)
-		(property "Reference" "#PWR0145"
+		(property "Reference" "#PWR0147"
 			(at 176.53 58.42 0)
 			(effects
@@
 			(project "DigitalOsciloscope"
 				(path "/553deb7b-4100-40fe-99d2-0c7b4b56aad2/3a7288c4-cf21-495b-9b8e-7b87b52ff1d8"
-					(reference "#PWR0145")
+					(reference "#PWR0147")
 					(unit 1)
 				)
@@
 		(dnp no)
 		(fields_autoplaced yes)
-		(property "Reference" "#FLG024"
+		(property "Reference" "#FLG025"
 			(at 134.62 111.125 0)
 			(effects
@@
 			(project "DigitalOsciloscope"
 				(path "/553deb7b-4100-40fe-99d2-0c7b4b56aad2/3a7288c4-cf21-495b-9b8e-7b87b52ff1d8"
-					(reference "#FLG024")
+					(reference "#FLG025")
 					(unit 1)
 				)
@@
 		(on_board yes)
 		(dnp no)
-		(property "Reference" "R71"
+		(property "Reference" "R65"
 			(at 226.314 64.77 90)
 			(effects
@@
 			(project ""
 				(path "/553deb7b-4100-40fe-99d2-0c7b4b56aad2/3a7288c4-cf21-495b-9b8e-7b87b52ff1d8"
-					(reference "R71")
+					(reference "R65")
 					(unit 1)
 				)
@@
 		(dnp no)
 		(fields_autoplaced yes)
-		(property "Reference" "#PWR0140"
+		(property "Reference" "#PWR0142"
 			(at 127 185.42 0)
 			(effects
@@
 			(project ""
 				(path "/553deb7b-4100-40fe-99d2-0c7b4b56aad2/3a7288c4-cf21-495b-9b8e-7b87b52ff1d8"
-					(reference "#PWR0140")
+					(reference "#PWR0142")
 					(unit 1)
 				)
@@
 		(on_board yes)
 		(dnp no)
-		(property "Reference" "#FLG023"
+		(property "Reference" "#FLG024"
 			(at 134.62 43.815 0)
 			(effects
@@
 			(project "DigitalOsciloscope"
 				(path "/553deb7b-4100-40fe-99d2-0c7b4b56aad2/3a7288c4-cf21-495b-9b8e-7b87b52ff1d8"
-					(reference "#FLG023")
+					(reference "#FLG024")
 					(unit 1)
 				)
@@
 		(dnp no)
 		(fields_autoplaced yes)
-		(property "Reference" "#FLG025"
+		(property "Reference" "#FLG026"
 			(at 134.62 117.475 0)
 			(effects
@@
 			(project "DigitalOsciloscope"
 				(path "/553deb7b-4100-40fe-99d2-0c7b4b56aad2/3a7288c4-cf21-495b-9b8e-7b87b52ff1d8"
-					(reference "#FLG025")
+					(reference "#FLG026")
 					(unit 1)
 				)
@@
 		(dnp no)
 		(fields_autoplaced yes)
-		(property "Reference" "#PWR0146"
+		(property "Reference" "#PWR0148"
 			(at 187.96 69.85 0)
 			(effects
@@
 			(project "DigitalOsciloscope"
 				(path "/553deb7b-4100-40fe-99d2-0c7b4b56aad2/3a7288c4-cf21-495b-9b8e-7b87b52ff1d8"
-					(reference "#PWR0146")
+					(reference "#PWR0148")
 					(unit 1)
 				)
@@
 		(dnp no)
 		(fields_autoplaced yes)
-		(property "Reference" "#PWR0139"
+		(property "Reference" "#PWR0141"
 			(at 127 109.22 0)
 			(effects
@@
 			(project "DigitalOsciloscope"
 				(path "/553deb7b-4100-40fe-99d2-0c7b4b56aad2/3a7288c4-cf21-495b-9b8e-7b87b52ff1d8"
-					(reference "#PWR0139")
+					(reference "#PWR0141")
 					(unit 1)
 				)
@@
 		(dnp no)
 		(fields_autoplaced yes)
-		(property "Reference" "#PWR0147"
+		(property "Reference" "#PWR0149"
 			(at 256.54 58.42 0)
 			(effects
@@
 			(project "DigitalOsciloscope"
 				(path "/553deb7b-4100-40fe-99d2-0c7b4b56aad2/3a7288c4-cf21-495b-9b8e-7b87b52ff1d8"
-					(reference "#PWR0147")
+					(reference "#PWR0149")
 					(unit 1)
 				)
@@
 		(dnp no)
 		(fields_autoplaced yes)
-		(property "Reference" "#PWR0141"
+		(property "Reference" "#PWR0144"
 			(at 156.21 115.57 0)
 			(effects
@@
 			(project "DigitalOsciloscope"
 				(path "/553deb7b-4100-40fe-99d2-0c7b4b56aad2/3a7288c4-cf21-495b-9b8e-7b87b52ff1d8"
-					(reference "#PWR0141")
+					(reference "#PWR0144")
 					(unit 1)
 				)
@@
 		(dnp no)
 		(fields_autoplaced yes)
-		(property "Reference" "#FLG022"
+		(property "Reference" "#FLG023"
 			(at 134.62 37.465 0)
 			(effects
@@
 			(project ""
 				(path "/553deb7b-4100-40fe-99d2-0c7b4b56aad2/3a7288c4-cf21-495b-9b8e-7b87b52ff1d8"
-					(reference "#FLG022")
+					(reference "#FLG023")
 					(unit 1)
 				)
@@
 		(dnp no)
 		(fields_autoplaced yes)
-		(property "Reference" "C100"
+		(property "Reference" "C102"
 			(at 260.35 60.9599 0)
 			(effects
@@
 			(project ""
 				(path "/553deb7b-4100-40fe-99d2-0c7b4b56aad2/3a7288c4-cf21-495b-9b8e-7b87b52ff1d8"
-					(reference "C100")
+					(reference "C102")
 					(unit 1)
 				)
@@
 		(dnp no)
 		(fields_autoplaced yes)
-		(property "Reference" "#PWR0107"
+		(property "Reference" "#PWR0143"
 			(at 156.21 41.91 0)
 			(effects
@@
 			(project ""
 				(path "/553deb7b-4100-40fe-99d2-0c7b4b56aad2/3a7288c4-cf21-495b-9b8e-7b87b52ff1d8"
-					(reference "#PWR0107")
+					(reference "#PWR0143")
 					(unit 1)
 				)

Commit message: Save before second attempt of routing ADC to FPGA
Connections:
- net ADC_A_0: now also U10.JP2_35 (GPIO_128); no longer U10.JP1_22 (GPIO_017)
- net ADC_A_1: now also U10.JP2_33 (GPIO_126); no longer U10.JP1_21 (GPIO_016)
- net ADC_A_10: now also U10.JP2_9 (GPIO_16); no longer U10.JP1_10 (GPIO_07)
- net ADC_A_11: now also U10.JP2_7 (GPIO_14); no longer U10.JP1_9 (GPIO_06)
- net ADC_A_12: now also U10.JP2_5 (GPIO_12); no longer U10.JP1_8 (GPIO_05)
- net ADC_A_13: now also U10.JP2_3 (GPIO_1_IN1); no longer U10.JP1_7 (GPIO_04)
- net ADC_A_2: now also U10.JP2_27 (GPIO_122); no longer U10.JP1_20 (GPIO_015)
- net ADC_A_3: now also U10.JP2_25 (GPIO_120); no longer U10.JP1_19 (GPIO_014)
- net ADC_A_4: now also U10.JP2_23 (GPIO_118); no longer U10.JP1_18 (GPIO_013)
- net ADC_A_5: now also U10.JP2_21 (GPIO_116); no longer U10.JP1_17 (GPIO_012)
- net ADC_A_6: now also U10.JP2_19 (GPIO_114); no longer U10.JP1_16 (GPIO_011)
- net ADC_A_7: now also U10.JP2_17 (GPIO_112); no longer U10.JP1_15 (GPIO_010)
- net ADC_A_8: now also U10.JP2_15 (GPIO_110); no longer U10.JP1_14 (GPIO_09)
- net ADC_A_9: now also U10.JP2_13 (GPIO_18); no longer U10.JP1_13 (GPIO_08)
- net ADC_B_0: now also U10.JP1_5 (GPIO_02); no longer U10.JP1_40 (GPIO_033)
- net ADC_B_1: now also U10.JP1_7 (GPIO_04); no longer U10.JP1_39 (GPIO_032)
- net ADC_B_10: now also U10.JP1_31 (GPIO_024); no longer U10.JP1_26 (GPIO_021)
- net ADC_B_11: now also U10.JP1_35 (GPIO_028); no longer U10.JP1_25 (GPIO_020)
- net ADC_B_12: now also U10.JP1_37 (GPIO_030); no longer U10.JP1_24 (GPIO_019)
- net ADC_B_13: now also U10.JP1_39 (GPIO_032); no longer U10.JP1_23 (GPIO_018)
- net ADC_B_2: now also U10.JP1_9 (GPIO_06); no longer U10.JP1_38 (GPIO_031)
- net ADC_B_3: now also U10.JP1_13 (GPIO_08); no longer U10.JP1_37 (GPIO_030)
- net ADC_B_4: now also U10.JP1_15 (GPIO_010); no longer U10.JP1_36 (GPIO_029)
- net ADC_B_5: now also U10.JP1_17 (GPIO_012); no longer U10.JP1_35 (GPIO_028)
- net ADC_B_6: now also U10.JP1_19 (GPIO_014); no longer U10.JP1_34 (GPIO_027)
- net ADC_B_7: now also U10.JP1_21 (GPIO_016); no longer U10.JP1_32 (GPIO_025)
- net ADC_B_8: now also U10.JP1_25 (GPIO_020); no longer U10.JP1_28 (GPIO_023)
- net AN_TRIGGER_N: now also U10.JP1_38 (GPIO_031); no longer U10.JP2_7 (GPIO_14)
- net AN_TRIGGER_P: now also U10.JP1_40 (GPIO_033); no longer U10.JP2_5 (GPIO_12)
- net CLIPPING: now also U10.JP2_4 (GPIO_11); no longer U10.JP2_15 (GPIO_110)
- net GPIO_10: now also U10.JP2_8 (GPIO_15); no longer U10.JP2_35 (GPIO_128)
- net GPIO_11: now also U10.JP2_6 (GPIO_13); no longer U10.JP2_37 (GPIO_130)
- net GPIO_6: now also U10.JP2_18 (GPIO_113); no longer U10.JP2_25 (GPIO_120)
- net GPIO_7: now also U10.JP2_16 (GPIO_111); no longer U10.JP2_27 (GPIO_122)
- net GPIO_8: now also U10.JP2_14 (GPIO_19); no longer U10.JP2_31 (GPIO_124)
- net GPIO_9: now also U10.JP2_10 (GPIO_17); no longer U10.JP2_33 (GPIO_126)
- net OE_A: now also U10.JP1_28 (GPIO_023); no longer U10.JP2_21 (GPIO_116)
- net OE_B: now also U10.JP1_26 (GPIO_021); no longer U10.JP2_23 (GPIO_118)
- net OVERFLOW: now also U10.JP2_2 (GPIO_10); no longer U10.JP2_39 (GPIO_132)
- net USART_1_RX: now also U10.JP1_36 (GPIO_029); no longer U10.JP2_17 (GPIO_112)
- net USART_1_TX: now also U10.JP1_34 (GPIO_027); no longer U10.JP2_19 (GPIO_114)
- no-connect marks 20 -> 5

Commit message: Done routing FGPA ADC data lines
Connections:
- net ADC_A_0: now also U10.JP2_3 (GPIO_1_IN1); no longer U10.JP2_35 (GPIO_128)
- net ADC_A_1: now also U10.JP2_5 (GPIO_12); no longer U10.JP2_33 (GPIO_126)
- net ADC_A_10: now also U10.JP2_25 (GPIO_120); no longer U10.JP2_9 (GPIO_16)
- net ADC_A_11: now also U10.JP2_27 (GPIO_122); no longer U10.JP2_7 (GPIO_14)
- net ADC_A_12: now also U10.JP2_31 (GPIO_124); no longer U10.JP2_5 (GPIO_12)
- net ADC_A_13: now also U10.JP2_33 (GPIO_126); no longer U10.JP2_3 (GPIO_1_IN1)
- net ADC_A_2: now also U10.JP2_7 (GPIO_14); no longer U10.JP2_27 (GPIO_122)
- net ADC_A_3: now also U10.JP2_9 (GPIO_16); no longer U10.JP2_25 (GPIO_120)
- net ADC_A_4: now also U10.JP2_13 (GPIO_18); no longer U10.JP2_23 (GPIO_118)
- net ADC_A_5: now also U10.JP2_15 (GPIO_110); no longer U10.JP2_21 (GPIO_116)
- net ADC_A_6: now also U10.JP2_17 (GPIO_112); no longer U10.JP2_19 (GPIO_114)
- net ADC_A_7: now also U10.JP2_19 (GPIO_114); no longer U10.JP2_17 (GPIO_112)
- net ADC_A_8: now also U10.JP2_21 (GPIO_116); no longer U10.JP2_15 (GPIO_110)
- net ADC_A_9: now also U10.JP2_23 (GPIO_118); no longer U10.JP2_13 (GPIO_18)
- no-connect marks 5 -> 18

Commit message: Save work before routing FPGA to STM32
Connections:
- net OE_A: now also U10.JP2_39 (GPIO_132); no longer U10.JP1_28 (GPIO_023)
- net OE_B: now also U10.JP1_18 (GPIO_013); no longer U10.JP1_26 (GPIO_021)
- net OVERFLOW: now also U10.JP2_37 (GPIO_130); no longer U10.JP2_2 (GPIO_10)
- no-connect marks 18 -> 15
Changed lines of the file:
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@@
 	)
 	(no_connect
-		(at 80.01 166.37)
-	)
-	(no_connect
 		(at 80.01 100.33)
 	)
@@
 	)
 	(no_connect
-		(at 125.73 67.31)
-	)
-	(no_connect
 		(at 125.73 72.39)
 	)
@@
 	)
 	(no_connect
-		(at 80.01 168.91)
-	)
-	(no_connect
 		(at 80.01 163.83)
 	)
@@
 	(wire
 		(pts
-			(xy 130.81 80.01) (xy 125.73 80.01)
-		)
-		(stroke
-			(width 0)
-			(type default)
-		)
-	)
-	(wire
-		(pts
 			(xy 130.81 123.19) (xy 125.73 123.19)
 		)
@@
 	(wire
 		(pts
+			(xy 68.58 168.91) (xy 80.01 168.91)
+		)
+		(stroke
+			(width 0)
+			(type default)
+		)
+	)
+	(wire
+		(pts
 			(xy 234.95 110.49) (xy 264.16 110.49)
 		)
@@
 	(wire
 		(pts
+			(xy 68.58 166.37) (xy 80.01 166.37)
+		)
+		(stroke
+			(width 0)
+			(type default)
+		)
+	)
+	(wire
+		(pts
 			(xy 55.88 67.31) (xy 80.01 67.31)
 		)
@@
 		)
 	)
+	(wire
+		(pts
+			(xy 130.81 67.31) (xy 125.73 67.31)
+		)
+		(stroke
+			(width 0)
+			(type default)
+		)
+	)
 	(bus
 		(pts
@@
 	(wire
 		(pts
-			(xy 130.81 77.47) (xy 125.73 77.47)
-		)
-		(stroke
-			(width 0)
-			(type default)
-		)
-	)
-	(wire
-		(pts
 			(xy 186.69 57.15) (xy 189.23 57.15)
 		)
@@
 		)
 	)
+	(global_label "OE_B"
+		(shape input)
+		(at 130.81 67.31 0)
+		(fields_autoplaced yes)
+		(effects
+			(font
+				(size 1.27 1.27)
+			)
+			(justify left)
+		)
+		(property "Intersheetrefs" "${INTERSHEET_REFS}"
+			(at 138.5123 67.31 0)
+			(effects
+				(font
+					(size 1.27 1.27)
+				)
+				(justify left)
+				(hide yes)
+			)
+		)
+	)
 	(global_label "ADC_B_1"
 		(shape input)
@@
 		)
 	)
+	(global_label "OE_A"
+		(shape input)
+		(at 68.58 168.91 180)
+		(fields_autoplaced yes)
+		(effects
+			(font
+				(size 1.27 1.27)
+			)
+			(justify right)
+		)
+		(property "Intersheetrefs" "${INTERSHEET_REFS}"
+			(at 61.0591 168.91 0)
+			(effects
+				(font
+					(size 1.27 1.27)
+				)
+				(justify right)
+				(hide yes)
+			)
+		)
+	)
 	(global_label "ADC_A_6"
 		(shape output)
@@
 		)
 	)
-	(global_label "OE_B"
-		(shape input)
-		(at 130.81 77.47 0)
-		(fields_autoplaced yes)
-		(effects
-			(font
-				(size 1.27 1.27)
-			)
-			(justify left)
-		)
-		(property "Intersheetrefs" "${INTERSHEET_REFS}"
-			(at 138.5123 77.47 0)
-			(effects
-				(font
-					(size 1.27 1.27)
-				)
-				(justify left)
-				(hide yes)
-			)
-		)
-	)
 	(global_label "ADC_B_5"
 		(shape input)
@@
 		)
 	)
-	(global_label "OE_A"
-		(shape input)
-		(at 130.81 80.01 0)
-		(fields_autoplaced yes)
-		(effects
-			(font
-				(size 1.27 1.27)
-			)
-			(justify left)
-		)
-		(property "Intersheetrefs" "${INTERSHEET_REFS}"
-			(at 138.3309 80.01 0)
-			(effects
-				(font
-					(size 1.27 1.27)
-				)
-				(justify left)
-				(hide yes)
-			)
-		)
-	)
 	(global_label "QSPI_IO3{slash}GPIO_5"
 		(shape input)
@@
 		)
 	)
-	(global_label "OVERFLOW"
+	(global_label "GPIO_23"
 		(shape input)
-		(at 130.81 120.65 0)
+		(at 130.81 151.13 0)
 		(fields_autoplaced yes)
 		(effects
@@
 		)
 		(property "Intersheetrefs" "${INTERSHEET_REFS}"
-			(at 143.5319 120.65 0)
+			(at 141.6571 151.13 0)
 			(effects
 				(font
@@
 		)
 	)
-	(global_label "GPIO_23"
+	(global_label "GPIO_10"
 		(shape input)
-		(at 130.81 151.13 0)
+		(at 130.81 128.27 0)
 		(fields_autoplaced yes)
 		(effects
@@
 		)
 		(property "Intersheetrefs" "${INTERSHEET_REFS}"
-			(at 141.6571 151.13 0)
+			(at 141.6571 128.27 0)
 			(effects
 				(font
@@
 		)
 	)
-	(global_label "GPIO_10"
-		(shape input)
-		(at 130.81 128.27 0)
+	(global_label "ADC_B_13"
+		(shape output)
+		(at 264.16 113.03 0)
 		(fields_autoplaced yes)
 		(effects
@@
 		)
 		(property "Intersheetrefs" "${INTERSHEET_REFS}"
-			(at 141.6571 128.27 0)
+			(at 276.398 113.03 0)
 			(effects
 				(font
@@
 		)
 	)
-	(global_label "ADC_B_13"
+	(global_label "ADC_A_2"
 		(shape output)
-		(at 264.16 113.03 0)
+		(at 213.36 86.36 0)
 		(fields_autoplaced yes)
 		(effects
@@
 		)
 		(property "Intersheetrefs" "${INTERSHEET_REFS}"
-			(at 276.398 113.03 0)
+			(at 224.2071 86.36 0)
 			(effects
 				(font
@@
 		)
 	)
-	(global_label "ADC_A_2"
-		(shape output)
-		(at 213.36 86.36 0)
+	(global_label "OVERFLOW"
+		(shape input)
+		(at 68.58 166.37 180)
 		(fields_autoplaced yes)
 		(effects
@@
 				(size 1.27 1.27)
 			)
-			(justify left)
+			(justify right)
 		)
 		(property "Intersheetrefs" "${INTERSHEET_REFS}"
-			(at 224.2071 86.36 0)
+			(at 55.8581 166.37 0)
 			(effects
 				(font
 					(size 1.27 1.27)
 				)
-				(justify left)
+				(justify right)
 				(hide yes)
 			)

Commit message: Save work before trying to allign FPGA MCU traces
Connections:
- net CLIPPING: now also U10.JP1_14 (GPIO_09); no longer U10.JP2_4 (GPIO_11)
- net GPIO_PD2: now reaches U10.JP1_16 (GPIO_011)
- net GPIO_PD15: now reaches U10.JP1_20 (GPIO_015)
- net GPIO_PE9: now reaches U10.JP1_22 (GPIO_017)
- net GPIO_PE11: now reaches U10.JP1_24 (GPIO_019)
- net GPIO_PE13: now reaches U10.JP1_26 (GPIO_021)
- net GPIO_PE8: now reaches U10.JP1_28 (GPIO_023)
- net GPIO_PE7: now reaches U10.JP1_32 (GPIO_025)
- net GPIO_PD1: now reaches U10.JP2_2 (GPIO_10)
- net GPIO_10 renamed GPIO_PE5
- net GPIO_11 renamed GPIO_PE6
- net GPIO_20 renamed GPIO_PD6
- net GPIO_21 renamed GPIO_PD7
- net GPIO_22 renamed GPIO_PE0
- net GPIO_23 renamed GPIO_PE15
- net GPIO_6 renamed GPIO_PD5
- net GPIO_7 renamed GPIO_PD4
- net GPIO_8 renamed GPIO_PD3
- net GPIO_9 renamed GPIO_PE4
- net QSPI_CLK/GPIO_1 renamed GPIO_PE12
- net QSPI_CS/GPIO_0 renamed QSPI_IO2/GPIO_PE2
- net QSPI_IO0/GPIO_2 renamed QSPI_IO0/GPIO_PD11
- net QSPI_IO1/GPIO_3 renamed GPIO_PE10
- net QSPI_IO2/GPIO_4 renamed QSPI_IO1/GPIO_PD12
- net QSPI_IO3/GPIO_5 renamed QSPI_IO3/GPIO_PD13
- new net GPIO_PD0: U10.JP2_4 (GPIO_11)
- no-connect marks 15 -> 10

Commit message: Everything is routed
Connections:
- net READY: now reaches U10.JP2_35 (GPIO_128)
- no-connect marks 10 -> 9
Changed lines of the file:
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@@
-	)
-	(no_connect
-		(at 80.01 163.83)
 	)
 	(no_connect
@@
 		(pts
 			(xy 163.83 38.1) (xy 163.83 41.91)
+		)
+		(stroke
+			(width 0)
+			(type default)
+		)
+	)
+	(wire
+		(pts
+			(xy 68.58 163.83) (xy 80.01 163.83)
 		)
 		(stroke
@@
 			(effects
 				(font
+					(size 1.27 1.27)
+				)
+				(justify right)
+				(hide yes)
+			)
+		)
+	)
+	(global_label "READY"
+		(shape input)
+		(at 68.58 163.83 180)
+		(fields_autoplaced yes)
+		(effects
+			(font
+				(size 1.27 1.27)
+			)
+			(justify right)
+		)
+		(property "Intersheetrefs" "${INTERSHEET_REFS}"
+			(at 59.7286 163.83 0)
+			(effects
+				(font

Commit message: Place most of the components in cart
Connections:
- no-connect marks 9 -> 10
Changed lines of the file:
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@@
+	)
+	(no_connect
+		(at 80.01 74.93)
 	)
 	(no_connect
