File: fpga.kicad_sch (KiCad schematic)
At the start: 10 parts, among them U10 P0082_BOTTOMMOUNT, Y1 XLL735080.000000I

Commit message: Finish channel 1 rework
Parts:
- renumbered C102 to C101, R59 to R58, R60 to R59, R61 to R60, R62 to R61, R63 to R62, R64 to R63, R65 to R64
Connections:
- no-connect marks 10 -> 9
Other:
- note removed: "TODO: ledy FPGA"
Changed lines of the file:
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@@
 	(generator_version "9.0")
 	(paper "A4")
-	(text "TODO: ledy FPGA"
-		(exclude_from_sim no)
-		(at 50.0772 22.4014 0)
-		(effects
-			(font
-				(size 1.27 1.27)
-			)
-		)
-	)
 	(junction
 		(at 127 175.26)
@@
 	)
 	(no_connect
-		(at 80.01 100.33)
-	)
-	(no_connect
 		(at 80.01 74.93)
 	)
@@
 		(on_board yes)
 		(dnp no)
-		(property "Reference" "R59"
+		(property "Reference" "R58"
 			(at 70.866 86.36 90)
 			(effects
@@
 			(project "DigitalOsciloscope"
 				(path "/553deb7b-4100-40fe-99d2-0c7b4b56aad2/3a7288c4-cf21-495b-9b8e-7b87b52ff1d8"
-					(reference "R59")
+					(reference "R58")
 					(unit 1)
 				)
@@
 		(pin "JP1_31"
 		)
-		(pin "S3"
-		)
 		(pin "JP1_33"
 		)
@@
 		(pin "JP2_11"
 		)
-		(pin "S4"
-		)
 		(pin "JP2_8"
 		)
@@
 		(pin "JP2_14"
 		)
-		(pin "S1"
-		)
 		(pin "JP2_1"
 		)
@@
 		(pin "JP2_33"
 		)
-		(pin "S2"
-		)
 		(pin "JP2_31"
 		)
@@
 		(dnp no)
 		(fields_autoplaced yes)
-		(property "Reference" "#PWR0145"
+		(property "Reference" "#PWR0144"
 			(at 163.83 41.91 0)
 			(effects
@@
 			(project "DigitalOsciloscope"
 				(path "/553deb7b-4100-40fe-99d2-0c7b4b56aad2/3a7288c4-cf21-495b-9b8e-7b87b52ff1d8"
-					(reference "#PWR0145")
+					(reference "#PWR0144")
 					(unit 1)
 				)
@@
 		(dnp no)
 		(fields_autoplaced yes)
-		(property "Reference" "#PWR0150"
+		(property "Reference" "#PWR0149"
 			(at 256.54 72.39 0)
 			(effects
@@
 			(project ""
 				(path "/553deb7b-4100-40fe-99d2-0c7b4b56aad2/3a7288c4-cf21-495b-9b8e-7b87b52ff1d8"
-					(reference "#PWR0150")
+					(reference "#PWR0149")
 					(unit 1)
 				)
@@
 		(dnp no)
 		(fields_autoplaced yes)
-		(property "Reference" "#PWR0146"
+		(property "Reference" "#PWR0145"
 			(at 163.83 115.57 0)
 			(effects
@@
 			(project ""
 				(path "/553deb7b-4100-40fe-99d2-0c7b4b56aad2/3a7288c4-cf21-495b-9b8e-7b87b52ff1d8"
-					(reference "#PWR0146")
+					(reference "#PWR0145")
 					(unit 1)
 				)
@@
 		(dnp no)
 		(fields_autoplaced yes)
-		(property "Reference" "#PWR0147"
+		(property "Reference" "#PWR0146"
 			(at 176.53 58.42 0)
 			(effects
@@
 			(project "DigitalOsciloscope"
 				(path "/553deb7b-4100-40fe-99d2-0c7b4b56aad2/3a7288c4-cf21-495b-9b8e-7b87b52ff1d8"
-					(reference "#PWR0147")
+					(reference "#PWR0146")
 					(unit 1)
 				)
@@
 		(dnp yes)
 		(fields_autoplaced yes)
-		(property "Reference" "R64"
+		(property "Reference" "R63"
 			(at 182.88 50.8 90)
 			(effects
@@
 			(project ""
 				(path "/553deb7b-4100-40fe-99d2-0c7b4b56aad2/3a7288c4-cf21-495b-9b8e-7b87b52ff1d8"
-					(reference "R64")
+					(reference "R63")
 					(unit 1)
 				)
@@
 		(on_board yes)
 		(dnp no)
-		(property "Reference" "R65"
+		(property "Reference" "R64"
 			(at 226.314 64.77 90)
 			(effects
@@
 			(project ""
 				(path "/553deb7b-4100-40fe-99d2-0c7b4b56aad2/3a7288c4-cf21-495b-9b8e-7b87b52ff1d8"
-					(reference "R65")
+					(reference "R64")
 					(unit 1)
 				)
@@
 		(dnp no)
 		(fields_autoplaced yes)
-		(property "Reference" "#PWR0142"
+		(property "Reference" "#PWR0141"
 			(at 127 185.42 0)
 			(effects
@@
 			(project ""
 				(path "/553deb7b-4100-40fe-99d2-0c7b4b56aad2/3a7288c4-cf21-495b-9b8e-7b87b52ff1d8"
-					(reference "#PWR0142")
+					(reference "#PWR0141")
 					(unit 1)
 				)
@@
 		(dnp no)
 		(fields_autoplaced yes)
-		(property "Reference" "#PWR0148"
+		(property "Reference" "#PWR0147"
 			(at 187.96 69.85 0)
 			(effects
@@
 			(project "DigitalOsciloscope"
 				(path "/553deb7b-4100-40fe-99d2-0c7b4b56aad2/3a7288c4-cf21-495b-9b8e-7b87b52ff1d8"
-					(reference "#PWR0148")
+					(reference "#PWR0147")
 					(unit 1)
 				)
@@
 		(dnp no)
 		(fields_autoplaced yes)
-		(property "Reference" "#PWR0141"
+		(property "Reference" "#PWR0140"
 			(at 127 109.22 0)
 			(effects
@@
 			(project "DigitalOsciloscope"
 				(path "/553deb7b-4100-40fe-99d2-0c7b4b56aad2/3a7288c4-cf21-495b-9b8e-7b87b52ff1d8"
-					(reference "#PWR0141")
+					(reference "#PWR0140")
 					(unit 1)
 				)
@@
 		(on_board yes)
 		(dnp no)
-		(property "Reference" "R60"
+		(property "Reference" "R59"
 			(at 148.336 38.1 90)
 			(effects
@@
 			(project "DigitalOsciloscope"
 				(path "/553deb7b-4100-40fe-99d2-0c7b4b56aad2/3a7288c4-cf21-495b-9b8e-7b87b52ff1d8"
-					(reference "R60")
+					(reference "R59")
 					(unit 1)
 				)
@@
 		(dnp no)
 		(fields_autoplaced yes)
-		(property "Reference" "#PWR0149"
+		(property "Reference" "#PWR0148"
 			(at 256.54 58.42 0)
 			(effects
@@
 			(project "DigitalOsciloscope"
 				(path "/553deb7b-4100-40fe-99d2-0c7b4b56aad2/3a7288c4-cf21-495b-9b8e-7b87b52ff1d8"
-					(reference "#PWR0149")
+					(reference "#PWR0148")
 					(unit 1)
 				)
@@
 		(dnp no)
 		(fields_autoplaced yes)
-		(property "Reference" "#PWR0144"
+		(property "Reference" "#PWR0143"
 			(at 156.21 115.57 0)
 			(effects
@@
 			(project "DigitalOsciloscope"
 				(path "/553deb7b-4100-40fe-99d2-0c7b4b56aad2/3a7288c4-cf21-495b-9b8e-7b87b52ff1d8"
-					(reference "#PWR0144")
+					(reference "#PWR0143")
 					(unit 1)
 				)
@@
 		(on_board yes)
 		(dnp no)
-		(property "Reference" "R62"
+		(property "Reference" "R61"
 			(at 148.336 111.76 90)
 			(effects
@@
 			(project "DigitalOsciloscope"
 				(path "/553deb7b-4100-40fe-99d2-0c7b4b56aad2/3a7288c4-cf21-495b-9b8e-7b87b52ff1d8"
-					(reference "R62")
+					(reference "R61")
 					(unit 1)
 				)
@@
 		(pin "JP1_31"
 		)
-		(pin "S3"
-		)
 		(pin "JP1_33"
 		)
@@
 		(pin "JP2_11"
 		)
-		(pin "S4"
-		)
 		(pin "JP2_8"
 		)
@@
 		(pin "JP2_14"
 		)
-		(pin "S1"
-		)
 		(pin "JP2_1"
 		)
@@
 		(pin "JP2_33"
 		)
-		(pin "S2"
-		)
 		(pin "JP2_31"
 		)
@@
 		(on_board yes)
 		(dnp yes)
-		(property "Reference" "R61"
+		(property "Reference" "R60"
 			(at 148.336 40.64 90)
 			(effects
@@
 			(project "DigitalOsciloscope"
 				(path "/553deb7b-4100-40fe-99d2-0c7b4b56aad2/3a7288c4-cf21-495b-9b8e-7b87b52ff1d8"
-					(reference "R61")
+					(reference "R60")
 					(unit 1)
 				)
@@
 		(on_board yes)
 		(dnp yes)
-		(property "Reference" "R63"
+		(property "Reference" "R62"
 			(at 148.336 114.3 90)
 			(effects
@@
 			(project "DigitalOsciloscope"
 				(path "/553deb7b-4100-40fe-99d2-0c7b4b56aad2/3a7288c4-cf21-495b-9b8e-7b87b52ff1d8"
-					(reference "R63")
+					(reference "R62")
 					(unit 1)
 				)
@@
 		(dnp no)
 		(fields_autoplaced yes)
-		(property "Reference" "C102"
+		(property "Reference" "C101"
 			(at 260.35 60.9599 0)
 			(effects
@@
 			(project ""
 				(path "/553deb7b-4100-40fe-99d2-0c7b4b56aad2/3a7288c4-cf21-495b-9b8e-7b87b52ff1d8"
-					(reference "C102")
+					(reference "C101")
 					(unit 1)
 				)
@@
 		(dnp no)
 		(fields_autoplaced yes)
-		(property "Reference" "#PWR0143"
+		(property "Reference" "#PWR0142"
 			(at 156.21 41.91 0)
 			(effects
@@
 			(project ""
 				(path "/553deb7b-4100-40fe-99d2-0c7b4b56aad2/3a7288c4-cf21-495b-9b8e-7b87b52ff1d8"
-					(reference "#PWR0143")
+					(reference "#PWR0142")
 					(unit 1)
 				)
