File: _autosave-analog_inputs_sch.kicad_sch (KiCad schematic)
At the start: 189 parts, among them J1 Conn_Coaxial, J2 Conn_Coaxial, K1 TX2SA-5V, K2 TX2SA-5V, K3 TX2SA-5V, K4 TX2SA-5V, K5 TX2SA-5V, K6 TX2SA-5V, U1 AD8611ARZ, U2 TL072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

Commit message: Trying to add symetry
Parts:
- removed TP5: TestPoint, TestPoint:TestPoint_Pad_D1.0mm, symbol Connector:TestPoint
Changed lines of the file:
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@@
 	)
 	(junction
-		(at 311.15 516.89)
-		(diameter 0)
-		(color 0 0 0 0)
-	)
-	(junction
 		(at 759.46 341.63)
 		(diameter 0)
@@
 	(wire
 		(pts
-			(xy 311.15 516.89) (xy 323.85 516.89)
-		)
-		(stroke
-			(width 0)
-			(type default)
-		)
-	)
-	(wire
-		(pts
 			(xy 77.47 156.21) (xy 77.47 162.56)
 		)
@@
 	(wire
 		(pts
-			(xy 308.61 516.89) (xy 311.15 516.89)
+			(xy 308.61 516.89) (xy 323.85 516.89)
 		)
 		(stroke
@@
 					(unit 1)
 				)
-			)
-		)
-	)
-	(symbol
-		(lib_id "Connector:TestPoint")
-		(at 311.15 516.89 0)
-		(unit 1)
-		(exclude_from_sim no)
-		(in_bom yes)
-		(on_board yes)
-		(dnp no)
-		(fields_autoplaced yes)
-		(property "Reference" "TP5"
-			(at 313.69 512.3179 0)
-			(effects
-				(font
-					(size 1.27 1.27)
-				)
-				(justify left)
-			)
-		)
-		(property "Value" "TestPoint"
-			(at 313.69 514.8579 0)
-			(effects
-				(font
-					(size 1.27 1.27)
-				)
-				(justify left)
-			)
-		)
-		(property "Footprint" "TestPoint:TestPoint_Pad_D1.0mm"
-			(at 316.23 516.89 0)
-			(effects
-				(font
-					(size 1.27 1.27)
-				)
-				(hide yes)
-			)
-		)
-		(property "Datasheet" "~"
-			(at 316.23 516.89 0)
-			(effects
-				(font
-					(size 1.27 1.27)
-				)
-				(hide yes)
-			)
-		)
-		(property "Description" "test point"
-			(at 311.15 516.89 0)
-			(effects
-				(font
-					(size 1.27 1.27)
-				)
-				(hide yes)
-			)
-		)
-		(pin "1"
-		)
-		(instances
-			(project "DigitalOsciloscope"
-				(path "/553deb7b-4100-40fe-99d2-0c7b4b56aad2/c6e88111-c18e-4095-b1d8-9b944099aec3"
-					(reference "TP5")
-					(unit 1)
-				)
